File: PH60/PH60.kicad_sch (KiCad schematic)
At the start: 42 parts, among them U1 nRF52840, U2 BQ24075RGT, U3 XC6220B331MR, Y1 32MHz, Y2 32.768kHz

Commit message: Remodel whole system to nrfmicro
Parts:
- removed C1, C14, C15, C2: 12pF, 0805:0805C, symbol Device:C
- removed C10, C11, C16, C22, C23, C25, C9: 4.7uF, 0805:0805C, symbol Device:C
- removed C12: 4.7nF, 0805:0805C, symbol Device:C
- removed C13, C20, C21: 1uF, 0805:0805C, symbol Device:C
- removed C17, C18, C19, C6: 100nF, 0805:0805C, symbol Device:C
- removed C24: 10uF, 0805:0805C, symbol Device:C
- removed C3, C4, C5: C, 0805:0805C, symbol Device:C
- removed C7: 100pF, 0805:0805C, symbol Device:C
- removed C8: 820pF, 0805:0805C, symbol Device:C
- removed D1: LED, 0805:0805D, symbol Device:LED
- removed JP1: Charge Boost, 0805:0805R, symbol Jumper:Jumper_2_Open
- removed L1: 3.9nH, 0805:0805R, symbol Device:L
- removed L2, L3: 10uH, 0805:0805R, symbol Device:L
- removed L4: 15nH, 0805:0805R, symbol Device:L
- removed R1: 0, 0805:0805R, symbol Device:R
- removed R4: 10k, 0805:0805R, symbol Device:R
- removed R5: 2k, 0805:0805R, symbol Device:R
- removed U1: nRF52840, Package_DFN_QFN:Nordic_AQFN-73-1EP_7x7mm_P0.5mm, symbol MCU_Nordic:nRF52840
- removed U2: BQ24075RGT, Package_DFN_QFN:VQFN-16-1EP_3x3mm_P0.5mm_EP1.6x1.6mm, symbol Battery_Management:BQ24075RGT
- removed U3: XC6220B331MR, Package_TO_SOT_SMD:SOT-23-5, symbol Regulator_Linear:XC6220B331MR
- removed Y1: 32MHz, Crystal:Crystal_SMD_2016-4Pin_2.0x1.6mm, symbol Device:Crystal_GND2
- removed Y2: 32.768kHz, Crystal:Crystal_SMD_3225-4Pin_3.2x2.5mm, symbol Device:Crystal
- added D63: 1N5819, Diode_SMD:D_SOD-323F, symbol nrfmicro-rescue:MBR0520
- added D64: BLUE, LED_SMD:LED_0603_1608Metric, symbol Device:LED
- added D65: RED, LED_SMD:LED_0603_1608Metric, symbol Device:LED
- added J1: USB-C USB 2.0 MC-372, nrfmicro:USB-C_C168688, symbol nrfmicro:USB_C_Receptacle_USB2.0
- added J2: Conn_01x04, Connector_JST:JST_GH_SM04B-GHS-TB_1x04-1MP_P1.25mm_Horizontal, symbol Connector_Generic:Conn_01x04
- added J3: Conn_01x02, Connector_Molex:Molex_PicoBlade_53261-0271_1x02-1MP_P1.25mm_Horizontal, symbol Connector_Generic:Conn_01x02
- added J4: Conn_01x04, nrfmicro:connector_usb, symbol Connector_Generic:Conn_01x04
- added JP1: SolderJumper_2_Open, nrfmicro:Jumper_SMD, symbol Jumper:SolderJumper_2_Open
- added Q1, Q2: AO3407, Package_TO_SOT_SMD:SOT-23, symbol nrfmicro-rescue:BSS83P
- added R1: 100K, Resistor_SMD:R_0603_1608Metric, symbol nrfmicro-rescue:R
- added R4, R8: 1K, Resistor_SMD:R_0603_1608Metric, symbol nrfmicro-rescue:R
- added R5: RPROG, Resistor_SMD:R_0603_1608Metric, symbol nrfmicro-rescue:R
- added R7, R9: 2M, Resistor_SMD:R_0603_1608Metric, symbol Device:R
- added U1: E73-2G4M08S1C, nrfmicro:E73-2G4M08S1C-52840, symbol nrfmicro:E73-2G4M08S1C-52840
- added U2: AP2112K-3.3, Package_TO_SOT_SMD:SOT-23-5, symbol Regulator_Linear:AP2112K-3.3
- added U3: TP4054, Package_TO_SOT_SMD:SOT-23-5, symbol Battery_Management:MCP73832-2-OT
- added U4: ProMicro, nrfmicro:pro_micro, symbol nrfmicro-rescue:ProMicro
- added X1: 32768kHz, Crystal:Crystal_SMD_3215-2Pin_3.2x1.5mm, symbol Device:Crystal_Small
- R2, R3: value 10k -> 5.1K; footprint 0805:0805R -> Resistor_SMD:R_0603_1608Metric
- R6: value 10M -> 820K; footprint 0805:0805R -> Resistor_SMD:R_0603_1608Metric
Connections:
- net GND: now also R2.2, R3.2, J1.A1 (GND), J1.S1 (SHIELD), J2.2 (Pin_2), J3.2 (Pin_2), J4.1 (Pin_1), R1.2, R4.2, R5.2, R7.2, R9.2, U1.21 (GND), U1.24 (GND), U1.5 (GND), U2.2 (GND), U3.2 (VSS), U4.15 (GND), U4.16 (GND), U4.2 (GND); no longer R2.1
- net col_0: now also U1.16 (P0.08), U4.14 (PD2)
- net col_1: now also U1.14 (P0.06), U4.13 (PD3)
- net col_10: now also JP1.2 (B), U1.1 (P1.11), U4.12 (PB6)
- net col_11: now also U1.4 (P0.28/AIN4), U4.11 (PB2)
- net col_12: now also U1.3 (P0.03/AIN1), U4.10 (PB3)
- net col_13: now also U1.6 (P1.13), U4.9 (PB1)
- net col_2: now also U1.28 (P0.15), U4.17 (PD1)
- net col_3: now also U1.30 (P0.17), U4.18 (PD0)
- net col_4: now also U1.32 (P0.20), U4.19 (PD4)
- net col_5: now also U1.33 (P0.13), U4.20 (PC6)
- net col_6: now also U1.35 (P0.24), U4.21 (PD7)
- net col_7: now also U1.41 (P0.09/NFC1), U4.22 (PE6)
- net col_8: now also U1.43 (P0.10/NFC2), U4.23 (PB4)
- net col_9: now also U1.42 (P1.06), U4.24 (PB5)
- net row_0: now also U1.7 (P0.02/AIN0), U4.8 (PF7)
- net row_1: now also U1.8 (P0.29/AIN5), U4.7 (PF6)
- net row_2: now also U1.9 (P0.31/AIN7), U4.6 (PF5)
- net row_3: now also U1.10 (P0.30/AIN6), U4.5 (PF4)
- net row_4: now also U1.20 (P0.12)
- net power_pin renamed BATTERY_PIN
- net BATTERY_PIN: now also R7.1, U1.18 (P0.04/AIN2)
- net vddh renamed CC1
- net CC1: now also J1.A5 (CC1); no longer R6.1
- new net: D63.1 (K), Q1.2 (S), U2.1 (VIN), U2.3 (EN)
- new net: D64.1 (K), R4.1
- new net: D65.1 (K), R8.1
- new net: R8.2, U3.1 (STAT)
- new net: R5.1, U3.5 (PROG)
- new net BLUE_LED: D64.2 (A), U1.2 (P1.10)
- new net CC2: J1.B5 (CC2), R2.1
- new net DATA+: J1.A6 (D+), J1.B6 (D+), J4.2 (Pin_2), U1.31 (USB_D+)
- new net DATA-: J1.A7 (D-), J1.B7 (D-), J4.3 (Pin_3), U1.29 (USB_D-)
- new net DCCH: U1.25 (DCCH)
- new net EXT_VCC: Q2.3 (D), U4.4 (VCC)
- new net P0.00: U1.11 (P0.00/XL1), X1.2
- new net P0.01: U1.13 (P0.01/XL2), X1.1
- new net P0.07: U1.22 (P0.07)
- new net P0.22: U1.34 (P0.22)
- new net P0.26: U1.12 (P0.26)
- new net P1.00: U1.36 (P1.00)
- new net P1.02: U1.38 (P1.02)
- new net P1.04: JP1.1 (A), U1.40 (P1.04)
- new net POWER_PIN: Q2.1 (G), R9.1, U1.17 (P1.09)
- new net PROG: U1.15 (P0.05/AIN3)
- new net RESET: U1.26 (P0.18/RESET), U4.3 (RST)
- new net SWC: J2.4 (Pin_4), U1.39 (SWDCLK)
- new net SWD: J2.3 (Pin_3), U1.37 (SWDIO)
- new net VBAT: J3.1 (Pin_1), Q1.3 (D), R6.1, U3.3 (VBAT), U4.1 (RAW)
- new net VBUS: D63.2 (A), D65.2 (A), J1.A4 (VBUS), J4.4 (Pin_4), Q1.1 (G), R1.1, U1.27 (VBUS), U3.4 (VDD)
- new net nRF_VDD: J2.1 (Pin_1), Q2.2 (S), U1.19 (VDD), U1.23 (VDDH), U2.5 (VOUT)
- no-connect marks 24 -> 4
Other:
- note added: "1.4.x"
- note added: "Battery monitor"
- note added: "E73-2G4M08S1C pins: P0.02 P0.03 P0.04 P0.05 P0.06 P0.07 P0.08 P0.09 P0.10 P0.12 P0.13 P0.15 P0.17 P0.18 P0.20 P0.22 P0.24 P0.26 P0.28 P0.29 P0.30 P0.31 P1.00 P1.02 P1.04 P1.06 P1.09 P1.10 P1.11 P1.13"
- note added: "Feather pins: P1.15 LED1 x P1.10 LED2 P0.15 BTN1 P0.19 BTN2 x P0.16 NEOPIXEL x P0.08 RX P0.06 TX P1.02 DFU P0.18 RESET"
- note added: "Jan 3, 2021"
- note added: "LiPo Charging"
- note added: "Power and Filtering"
- note added: "RProg = 1000/iBat iBat in amps RProg iBAT 10k 100mA 5k 200mA 2.5k 400mA 2k 500mA 1.25k 800mA"
- note added: "nrfmicro"
- note removed: "Controller"
- note removed: "Power Management"
- note removed: "VCC Regulator and Cut Off"
