File: PH60/PH60.kicad_pcb (KiCad board)
At the start: 2 copper layers, 166 parts, among them U1 nRF52840, U2 BQ24075RGT, U3 XC6220B331MR, Y1 32MHz, Y2 32.768kHz

Commit message: UPDATE PCB
Parts:
- moved R3 191.9 mm to (384.2, 198.9), turned to 0 degrees
- moved U3 174.9 mm to (253.2, 217.8)
- moved D1 134.5 mm to (388.8, 199.1)
- moved C17 133.4 mm to (264.3, 220.7), turned to -90 degrees
- moved C23 131.1 mm to (397.1, 198.4), turned to -90 degrees
- moved L1 130.0 mm to (233.1, 211.3), turned to 0 degrees
- moved JP1 130.0 mm to (394.8, 190.9), turned to 0 degrees
- moved C25 130.0 mm to (253.6, 212.0), turned to 90 degrees
- moved C18 129.3 mm to (267.6, 220.7), turned to -90 degrees
- moved C3 129.2 mm to (234.5, 215.4), turned to 90 degrees
- moved C9 129.0 mm to (278.8, 219.9), turned to 0 degrees
- moved C4 127.6 mm to (231.1, 215.4), turned to 90 degrees
- moved C5 126.3 mm to (227.8, 215.4), turned to 90 degrees
- moved C19 125.3 mm to (270.9, 220.7), turned to -90 degrees
- moved C21 125.0 mm to (389.9, 190.8), turned to 0 degrees
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Routing:
- net Net-(D9-A): track 0.00 -> 9.05 mm
- net Net-(D8-A): track 0.00 -> 9.05 mm
- net Net-(D7-A): track 0.00 -> 9.05 mm
- net Net-(D6-A): track 0.00 -> 9.05 mm
- net Net-(D57-A): track 0.00 -> 9.05 mm
- net Net-(D55-A): track 0.00 -> 9.05 mm
- net Net-(D54-A): track 0.00 -> 9.05 mm
- net Net-(D53-A): track 0.00 -> 9.05 mm
- net Net-(D52-A): track 0.00 -> 9.05 mm
- net Net-(D51-A): track 0.00 -> 9.05 mm
- net Net-(D50-A): track 0.00 -> 9.05 mm
- net Net-(D5-A): track 0.00 -> 9.05 mm
- net Net-(D49-A): track 0.00 -> 9.05 mm
- net Net-(D48-A): track 0.00 -> 9.05 mm
- net Net-(D47-A): track 0.00 -> 9.05 mm
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Other:
- board outline added: 285.7 x 95.2 mm

Commit message: Remodel whole system to nrfmicro
Parts:
- removed C1, C14, C15, C2: 12pF, 0805:0805C
- removed C10, C11, C16, C22, C23, C25, C9: 4.7uF, 0805:0805C
- removed C12: 4.7nF, 0805:0805C
- removed C13, C20, C21: 1uF, 0805:0805C
- removed C17, C18, C19, C6: 100nF, 0805:0805C
- removed C24: 10uF, 0805:0805C
- removed C3, C4, C5: C, 0805:0805C
- removed C7: 100pF, 0805:0805C
- removed C8: 820pF, 0805:0805C
- removed D68, D69, D70, D71: DIODE, 0805:0805D
- removed L1: 3.9nH, 0805:0805R
- removed L2, L3: 10uH, 0805:0805R
- removed L4: 15nH, 0805:0805R
- removed S63: MX1A, Button_Switch_Keyboard:SW_Cherry_MX_6.25u_PCB
- removed S67, S68, S69, S70: MX1A, Button_Switch_Keyboard:SW_Cherry_MX_1.25u_PCB
- removed Y1: 32MHz, Crystal:Crystal_SMD_2016-4Pin_2.0x1.6mm
- removed Y2: 32.768kHz, Crystal:Crystal_SMD_3225-4Pin_3.2x2.5mm
- added D42: DIODE, Diode_SMD:D_0805_2012Metric_Pad1.15x1.40mm_HandSolder, B.Cu at (45.6, 98.3)
- added D56: DIODE, Diode_SMD:D_0805_2012Metric_Pad1.15x1.40mm_HandSolder, B.Cu at (69.4, 117.3)
- added D61: DIODE, Diode_SMD:D_0805_2012Metric_Pad1.15x1.40mm_HandSolder, B.Cu at (283.7, 117.3)
- added D62: DIODE, Diode_SMD:D_0805_2012Metric_Pad1.15x1.40mm_HandSolder, B.Cu at (307.5, 117.3)
- added D63: 1N5819, Diode_SMD:D_SOD-323F, B.Cu at (206.7, 121.2)
- added D65: RED, LED_SMD:LED_0603_1608Metric, B.Cu at (218.3, 120.6)
- added J1: USB-C USB 2.0 MC-372, nrfmicro:USB-C_C168688, B.Cu at (304.1, 94.3)
- added J2: Conn_01x04, Connector_JST:JST_GH_SM04B-GHS-TB_1x04-1MP_P1.25mm_Horizontal, B.Cu at (205.1, 109.8)
- added J3: Conn_01x02, Connector_Molex:Molex_PicoBlade_53261-0271_1x02-1MP_P1.25mm_Horizontal, B.Cu at (291.5, 53.8)
- added J4: Conn_01x04, nrfmicro:connector_usb, B.Cu at (219.2, 105.8)
- added Q1: AO3407, Package_TO_SOT_SMD:SOT-23, B.Cu at (205.7, 116.5)
- added Q2: AO3407, Package_TO_SOT_SMD:SOT-23, B.Cu at (193.3, 116.2)
- added R7: 2M, Resistor_SMD:R_0603_1608Metric, B.Cu at (198.2, 110.3)
- added R8: 1K, Resistor_SMD:R_0603_1608Metric, B.Cu at (212.8, 115.9)
- added R9: 2M, Resistor_SMD:R_0603_1608Metric, B.Cu at (197.2, 115.2)
- added S53: MX1A, PCM_Switch_Keyboard_Hotswap_Kailh:SW_Hotswap_Kailh_MX_1.00u, F.Cu at (252.4, 95.2)
- added S54: MX1A, PCM_Switch_Keyboard_Hotswap_Kailh:SW_Hotswap_Kailh_MX_2.75u, F.Cu at (288.1, 95.2)
- added S60: MX1A, PCM_Switch_Keyboard_Hotswap_Kailh:SW_Hotswap_Kailh_MX_1.25u, F.Cu at (254.8, 114.3)
- added S61: MX1A, PCM_Switch_Keyboard_Hotswap_Kailh:SW_Hotswap_Kailh_MX_1.25u, F.Cu at (278.6, 114.3)
- added S62: MX1A, PCM_Switch_Keyboard_Hotswap_Kailh:SW_Hotswap_Kailh_MX_1.25u, F.Cu at (302.4, 114.3)
- added X1: 32768kHz, Crystal:Crystal_SMD_3215-2Pin_3.2x1.5mm, B.Cu at (193.1, 110.3)
- D1: value LED -> DIODE; footprint 0805:0805D -> Diode_SMD:D_0805_2012Metric_Pad1.15x1.40mm_HandSolder
- D10, D11, D12, D13, D14, D15, D16, D17, D18, D19, D2, D20, D21, D22, D23, D24, D25, D26, D27, D28, D29, D3, D30, D31, D32, D33, D34, D35, D36, D37, D38, D39, D4, D40, D41, D43, D44, D45, D46, D47, D48, D49, D5, D50, D51, D52, D53, D54, D55, D57, D58, D59, D6, D60, D7, D8, D9: footprint 0805:0805D -> Diode_SMD:D_0805_2012Metric_Pad1.15x1.40mm_HandSolder
- D64: value DIODE -> BLUE; footprint 0805:0805D -> LED_SMD:LED_0603_1608Metric
- JP1: value Charge Boost -> SolderJumper_2_Open; footprint 0805:0805R -> nrfmicro:Jumper_SMD
- R1: value 0 -> 100K; footprint 0805:0805R -> Resistor_SMD:R_0603_1608Metric
- R2, R3: value 10k -> 5.1K; footprint 0805:0805R -> Resistor_SMD:R_0603_1608Metric
- R4: value 10k -> 1K; footprint 0805:0805R -> Resistor_SMD:R_0603_1608Metric
- R5: value 2k -> RPROG; footprint 0805:0805R -> Resistor_SMD:R_0603_1608Metric
- R6: value 10M -> 820K; footprint 0805:0805R -> Resistor_SMD:R_0603_1608Metric
- S1, S10, S11, S12, S13, S16, S17, S18, S19, S2, S20, S21, S22, S23, S24, S25, S26, S27, S3, S31, S32, S33, S34, S35, S36, S37, S38, S39, S4, S40, S41, S43, S44, S45, S46, S47, S48, S49, S5, S50, S51, S52, S6, S7, S8, S9: footprint Button_Switch_Keyboard:SW_Cherry_MX_1.00u_PCB -> PCM_Switch_Keyboard_Hotswap_Kailh:SW_Hotswap_Kailh_MX_1.00u
- S14: footprint Button_Switch_Keyboard:SW_Cherry_MX_2.00u_PCB -> PCM_Switch_Keyboard_Hotswap_Kailh:SW_Hotswap_Kailh_MX_2.00u
- S15: footprint Button_Switch_Keyboard:SW_Cherry_MX_1.50u_PCB -> PCM_Switch_Keyboard_Hotswap_Kailh:SW_Hotswap_Kailh_MX_1.50u
- S28: footprint Button_Switch_Keyboard:SW_Cherry_MX_ISOEnter_PCB -> PCM_Switch_Keyboard_Hotswap_Kailh:SW_Hotswap_Kailh_MX_ISOEnter
- S29: footprint Button_Switch_Keyboard:SW_Cherry_MX_1.75u_PCB -> PCM_Switch_Keyboard_Hotswap_Kailh:SW_Hotswap_Kailh_MX_1.75u
- S30: footprint Button_Switch_Keyboard:SW_Cherry_MX_1.25u_PCB -> PCM_Switch_Keyboard_Hotswap_Kailh:SW_Hotswap_Kailh_MX_1.00u
- S42, S55: footprint Button_Switch_Keyboard:SW_Cherry_MX_1.00u_PCB -> PCM_Switch_Keyboard_Hotswap_Kailh:SW_Hotswap_Kailh_MX_1.25u
- S56: footprint Button_Switch_Keyboard:SW_Cherry_MX_2.75u_PCB -> PCM_Switch_Keyboard_Hotswap_Kailh:SW_Hotswap_Kailh_MX_1.25u
- S57, S59: footprint Button_Switch_Keyboard:SW_Cherry_MX_1.25u_PCB -> PCM_Switch_Keyboard_Hotswap_Kailh:SW_Hotswap_Kailh_MX_1.25u
- S58: footprint Button_Switch_Keyboard:SW_Cherry_MX_1.25u_PCB -> PCM_Switch_Keyboard_Hotswap_Kailh:SW_Hotswap_Kailh_MX_6.25u
- U1: value nRF52840 -> E73-2G4M08S1C; footprint Package_DFN_QFN:Nordic_AQFN-73-1EP_7x7mm_P0.5mm -> nrfmicro:E73-2G4M08S1C-52840
- U2: value BQ24075RGT -> AP2112K-3.3; footprint Package_DFN_QFN:VQFN-16-1EP_3x3mm_P0.5mm_EP1.6x1.6mm -> Package_TO_SOT_SMD:SOT-23-5
- U3: value XC6220B331MR -> TP4054
- moved D1 380.0 mm to (43.2, 41.1), turned to 90 degrees
- moved D29 351.8 mm to (50.3, 79.2), turned to 90 degrees
- moved D15 344.8 mm to (47.9, 60.2), turned to 90 degrees
- moved S55 332.8 mm to (40.5, 114.3)
- moved S56 320.4 mm to (64.3, 114.3)
- moved D43 312.6 mm to (67.0, 98.3), turned to 90 degrees
- moved D55 305.7 mm to (45.6, 117.3), turned to 90 degrees
- moved D57 294.2 mm to (93.2, 117.3), turned to 90 degrees
- moved JP1 240.0 mm to (170.0, 106.9), turned to 90 degrees
- moved S42 225.0 mm to (40.5, 95.2)
- moved R4 224.6 mm to (184.2, 105.0), turned to 0 degrees
- moved S43 224.4 mm to (61.9, 95.2)
- moved U2 207.3 mm to (199.5, 120.6)
- moved S45 206.5 mm to (100.0, 95.2)
- moved S44 205.7 mm to (81.0, 95.2)
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Connections:
- D1 pad 1: Net-(D1-K) -> row_0
- D10 pad 1: Net-(D10-A) -> row_0
- D10 pad 2: row_0 -> Net-(D10-A)
- D11 pad 1: Net-(D11-A) -> row_0
- D11 pad 2: row_0 -> Net-(D11-A)
- D12 pad 1: Net-(D12-A) -> row_0
- D12 pad 2: row_0 -> Net-(D12-A)
- D13 pad 1: Net-(D13-A) -> row_0
- D13 pad 2: row_0 -> Net-(D13-A)
- D14 pad 1: Net-(D14-A) -> row_0
- D14 pad 2: row_0 -> Net-(D14-A)
- D15 pad 1: Net-(D15-A) -> row_1
- D15 pad 2: row_0 -> Net-(D15-A)
- D16 pad 1: Net-(D16-A) -> row_1
- D16 pad 2: row_1 -> Net-(D16-A)
- D17 pad 1: Net-(D17-A) -> row_1
- D17 pad 2: row_1 -> Net-(D17-A)
- D18 pad 1: Net-(D18-A) -> row_1
- D18 pad 2: row_1 -> Net-(D18-A)
- D19 pad 1: Net-(D19-A) -> row_1
- D19 pad 2: row_1 -> Net-(D19-A)
- D2 pad 1: Net-(D2-A) -> row_0
- D2 pad 2: row_0 -> Net-(D2-A)
- D20 pad 1: Net-(D20-A) -> row_1
- D20 pad 2: row_1 -> Net-(D20-A)
- D21 pad 1: Net-(D21-A) -> row_1
- D21 pad 2: row_1 -> Net-(D21-A)
- D22 pad 1: Net-(D22-A) -> row_1
- D22 pad 2: row_1 -> Net-(D22-A)
- D23 pad 1: Net-(D23-A) -> row_1
- D23 pad 2: row_1 -> Net-(D23-A)
- D24 pad 1: Net-(D24-A) -> row_1
- D24 pad 2: row_1 -> Net-(D24-A)
- D25 pad 1: Net-(D25-A) -> row_1
- D25 pad 2: row_1 -> Net-(D25-A)
- D26 pad 1: Net-(D26-A) -> row_1
- D26 pad 2: row_1 -> Net-(D26-A)
- D27 pad 1: Net-(D27-A) -> row_1
- D27 pad 2: row_1 -> Net-(D27-A)
- D28 pad 1: Net-(D28-A) -> row_1
- D28 pad 2: row_1 -> Net-(D28-A)
- D29 pad 1: Net-(D29-A) -> row_2
- D29 pad 2: row_1 -> Net-(D29-A)
- D3 pad 1: Net-(D3-A) -> row_0
- D3 pad 2: row_0 -> Net-(D3-A)
- D30 pad 1: Net-(D30-A) -> row_2
- D30 pad 2: row_2 -> Net-(D30-A)
- D31 pad 1: Net-(D31-A) -> row_2
- D31 pad 2: row_2 -> Net-(D31-A)
- D32 pad 1: Net-(D32-A) -> row_2
- D32 pad 2: row_2 -> Net-(D32-A)
- D33 pad 1: Net-(D33-A) -> row_2
- D33 pad 2: row_2 -> Net-(D33-A)
- D34 pad 1: Net-(D34-A) -> row_2
- D34 pad 2: row_2 -> Net-(D34-A)
- D35 pad 1: Net-(D35-A) -> row_2
- D35 pad 2: row_2 -> Net-(D35-A)
- D36 pad 1: Net-(D36-A) -> row_2
- D36 pad 2: row_2 -> Net-(D36-A)
- D37 pad 1: Net-(D37-A) -> row_2
- D37 pad 2: row_2 -> Net-(D37-A)
- D38 pad 1: Net-(D38-A) -> row_2
- D38 pad 2: row_2 -> Net-(D38-A)
- D39 pad 1: Net-(D39-A) -> row_2
- D39 pad 2: row_2 -> Net-(D39-A)
- D4 pad 1: Net-(D4-A) -> row_0
- D4 pad 2: row_0 -> Net-(D4-A)
- D40 pad 1: Net-(D40-A) -> row_2
- D40 pad 2: row_2 -> Net-(D40-A)
- D41 pad 1: Net-(D41-A) -> row_2
- D41 pad 2: row_2 -> Net-(D41-A)
- D43 pad 1: Net-(D43-A) -> row_3
- D43 pad 2: row_2 -> Net-(D43-A)
- D44 pad 1: Net-(D44-A) -> row_3
- D44 pad 2: row_3 -> Net-(D44-A)
- D45 pad 1: Net-(D45-A) -> row_3
- D45 pad 2: row_3 -> Net-(D45-A)
- D46 pad 1: Net-(D46-A) -> row_3
- D46 pad 2: row_3 -> Net-(D46-A)
- D47 pad 1: Net-(D47-A) -> row_3
- D47 pad 2: row_3 -> Net-(D47-A)
- D48 pad 1: Net-(D48-A) -> row_3
- D48 pad 2: row_3 -> Net-(D48-A)
- D49 pad 1: Net-(D49-A) -> row_3
- D49 pad 2: row_3 -> Net-(D49-A)
- D5 pad 1: Net-(D5-A) -> row_0
- D5 pad 2: row_0 -> Net-(D5-A)
- D50 pad 1: Net-(D50-A) -> row_3
- D50 pad 2: row_3 -> Net-(D50-A)
- D51 pad 1: Net-(D51-A) -> row_3
- D51 pad 2: row_3 -> Net-(D51-A)
- D52 pad 1: Net-(D52-A) -> row_3
- D52 pad 2: row_3 -> Net-(D52-A)
- D53 pad 1: Net-(D53-A) -> row_3
- D53 pad 2: row_3 -> Net-(D53-A)
- D54 pad 1: Net-(D54-A) -> row_3
- D54 pad 2: row_3 -> Net-(D54-A)
- D55 pad 1: Net-(D55-A) -> row_4
- D55 pad 2: row_3 -> Net-(D55-A)
- D57 pad 1: Net-(D57-A) -> row_4
- D57 pad 2: row_3 -> Net-(D57-A)
- D58 pad 1: Net-(D58-A) -> row_4
- D58 pad 2: row_4 -> Net-(D58-A)
- D59 pad 1: Net-(D59-A) -> row_4
- D59 pad 2: row_4 -> Net-(D59-A)
- D6 pad 1: Net-(D6-A) -> row_0
- D6 pad 2: row_0 -> Net-(D6-A)
- D60 pad 1: Net-(D60-A) -> row_4
- D60 pad 2: row_4 -> Net-(D60-A)
- D64 pad 1: Net-(D64-A) -> Net-(D64-K)
- D64 pad 2: row_4 -> BLUE_LED
- D7 pad 1: Net-(D7-A) -> row_0
- D7 pad 2: row_0 -> Net-(D7-A)
- D8 pad 1: Net-(D8-A) -> row_0
- D8 pad 2: row_0 -> Net-(D8-A)
- D9 pad 1: Net-(D9-A) -> row_0
- D9 pad 2: row_0 -> Net-(D9-A)
- JP1 pad 1: Net-(JP1-A) -> /P1.04
- JP1 pad 2: Net-(JP1-B) -> col_10
- R1 pad 1: antenna -> VBUS
- R1 pad 2: Net-(C4-Pad2) -> GND
- R2 pad 1: GND -> CC2
- R2 pad 2: Net-(U2-TS) -> GND
- R3 pad 1: vddh -> CC1
- R3 pad 2: Net-(D1-A) -> GND
- R4 pad 1: GND -> Net-(D64-K)
- R4 pad 2: Net-(JP1-A) -> GND
- R5 pad 1: GND -> Net-(U3-PROG)
- R5 pad 2: Net-(JP1-B) -> GND
- R6 pad 1: vddh -> VBAT
- R6 pad 2: power_pin -> BATTERY_PIN
- S1 pad 1: Net-(D2-A) -> Net-(D1-A)
- S10 pad 1: Net-(D11-A) -> Net-(D10-A)
- S11 pad 1: Net-(D12-A) -> Net-(D11-A)
- S12 pad 1: Net-(D13-A) -> Net-(D12-A)
- S13 pad 1: Net-(D14-A) -> Net-(D13-A)
- S14 pad 1: Net-(D15-A) -> Net-(D14-A)
- S15 pad 1: Net-(D16-A) -> Net-(D15-A)
- S16 pad 1: Net-(D17-A) -> Net-(D16-A)
- S17 pad 1: Net-(D18-A) -> Net-(D17-A)
- S18 pad 1: Net-(D19-A) -> Net-(D18-A)
- S19 pad 1: Net-(D20-A) -> Net-(D19-A)
- S2 pad 1: Net-(D3-A) -> Net-(D2-A)
- S20 pad 1: Net-(D21-A) -> Net-(D20-A)
- S21 pad 1: Net-(D22-A) -> Net-(D21-A)
- S22 pad 1: Net-(D23-A) -> Net-(D22-A)
- S23 pad 1: Net-(D24-A) -> Net-(D23-A)
- S24 pad 1: Net-(D25-A) -> Net-(D24-A)
- S25 pad 1: Net-(D26-A) -> Net-(D25-A)
- S26 pad 1: Net-(D27-A) -> Net-(D26-A)
- S27 pad 1: Net-(D28-A) -> Net-(D27-A)
- S28 pad 1: Net-(D29-A) -> Net-(D28-A)
- S29 pad 1: Net-(D30-A) -> Net-(D29-A)
- S3 pad 1: Net-(D4-A) -> Net-(D3-A)
- S30 pad 1: Net-(D44-A) -> Net-(D30-A)
- S30 pad 2: col_0 -> col_1
- S31 pad 2: col_1 -> col_2
- S32 pad 1: Net-(D45-A) -> Net-(D32-A)
- S32 pad 2: col_1 -> col_3
- S33 pad 1: Net-(D32-A) -> Net-(D33-A)
- S33 pad 2: col_2 -> col_4
- S34 pad 1: Net-(D46-A) -> Net-(D34-A)
- S34 pad 2: col_2 -> col_5
- S35 pad 1: Net-(D33-A) -> Net-(D35-A)
- S35 pad 2: col_3 -> col_6
- S36 pad 1: Net-(D47-A) -> Net-(D36-A)
- S36 pad 2: col_3 -> col_7
- S37 pad 1: Net-(D34-A) -> Net-(D37-A)
- S37 pad 2: col_4 -> col_8
- S38 pad 1: Net-(D48-A) -> Net-(D38-A)
- S38 pad 2: col_4 -> col_9
- S39 pad 1: Net-(D35-A) -> Net-(D39-A)
- S39 pad 2: col_5 -> col_10
- S4 pad 1: Net-(D5-A) -> Net-(D4-A)
- S40 pad 1: Net-(D49-A) -> Net-(D40-A)
- S40 pad 2: col_5 -> col_11
- S41 pad 1: Net-(D36-A) -> Net-(D41-A)
- S41 pad 2: col_6 -> col_13
- S42 pad 1: Net-(D50-A) -> Net-(D42-A)
- S42 pad 2: col_6 -> col_0
- S43 pad 1: Net-(D37-A) -> Net-(D43-A)
- S43 pad 2: col_7 -> col_1
- S44 pad 1: Net-(D51-A) -> Net-(D44-A)
- S44 pad 2: col_7 -> col_2
- S45 pad 1: Net-(D38-A) -> Net-(D45-A)
- S45 pad 2: col_8 -> col_3
- S46 pad 1: Net-(D52-A) -> Net-(D46-A)
- S46 pad 2: col_8 -> col_4
- S47 pad 1: Net-(D39-A) -> Net-(D47-A)
- S47 pad 2: col_9 -> col_5
- S48 pad 1: Net-(D53-A) -> Net-(D48-A)
- S48 pad 2: col_9 -> col_6
- S49 pad 1: Net-(D40-A) -> Net-(D49-A)
- S49 pad 2: col_10 -> col_7
- S5 pad 1: Net-(D6-A) -> Net-(D5-A)
- S50 pad 1: Net-(D54-A) -> Net-(D50-A)
- S50 pad 2: col_10 -> col_8
- S51 pad 1: Net-(D41-A) -> Net-(D51-A)
- S51 pad 2: col_11 -> col_9
- S52 pad 1: Net-(D55-A) -> Net-(D52-A)
- S52 pad 2: col_11 -> col_10
- S55 pad 1: Net-(D43-A) -> Net-(D55-A)
- S55 pad 2: col_13 -> col_0
- S56 pad 1: Net-(D57-A) -> Net-(D56-A)
- S56 pad 2: col_13 -> col_1
- S57 pad 1: Net-(D58-A) -> Net-(D57-A)
- S57 pad 2: col_0 -> col_2
- S58 pad 1: Net-(D59-A) -> Net-(D58-A)
- S58 pad 2: col_1 -> col_6
- S59 pad 1: Net-(D60-A) -> Net-(D59-A)
- S59 pad 2: col_2 -> col_9
- S6 pad 1: Net-(D7-A) -> Net-(D6-A)
- S7 pad 1: Net-(D8-A) -> Net-(D7-A)
- S8 pad 1: Net-(D9-A) -> Net-(D8-A)
- S9 pad 1: Net-(D10-A) -> Net-(D9-A)
- U2 pad 1: Net-(U2-TS) -> Net-(D63-K)
- U2 pad 2: vbat -> GND
- U2 pad 3: vbat -> Net-(D63-K)
- U2 pad 4: GND -> unconnected-(U2-NC-Pad4)
- U2 pad 5: GND -> nRF_VDD
- U3 pad 1: vddh -> Net-(U3-STAT)
- U3 pad 3: power_pin -> VBAT
- U3 pad 4: unconnected-(U3-NC-Pad4) -> VBUS
- U3 pad 5: ext_vcc -> Net-(U3-PROG)
Routing:
- net Net-(D9-A): track 9.05 -> 0.00 mm
- net Net-(D8-A): track 9.05 -> 0.00 mm
- net Net-(D7-A): track 9.05 -> 0.00 mm
- net Net-(D6-A): track 9.05 -> 0.00 mm
- net Net-(D57-A): track 9.05 -> 0.00 mm
- net Net-(D55-A): track 9.05 -> 0.00 mm
- net Net-(D54-A): track 9.05 -> 0.00 mm
- net Net-(D53-A): track 9.05 -> 0.00 mm
- net Net-(D52-A): track 9.05 -> 0.00 mm
- net Net-(D51-A): track 9.05 -> 0.00 mm
- net Net-(D50-A): track 9.05 -> 0.00 mm
- net Net-(D5-A): track 9.05 -> 0.00 mm
- net Net-(D49-A): track 9.05 -> 0.00 mm
- net Net-(D48-A): track 9.05 -> 0.00 mm
- net Net-(D47-A): track 9.05 -> 0.00 mm
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Other:
- board outline removed

Commit message: PCB Updates
Parts:
- removed J1: USB-C USB 2.0 MC-372, nrfmicro:USB-C_C168688
- removed J4: Conn_01x04, nrfmicro:connector_usb
- removed JP1: SolderJumper_2_Open, nrfmicro:Jumper_SMD
- removed R2, R3: 5.1K, Resistor_SMD:R_0603_1608Metric
- J2: footprint Connector_JST:JST_GH_SM04B-GHS-TB_1x04-1MP_P1.25mm_Horizontal -> Connector_FFC-FPC:Molex_200528-0040_1x04-1MP_P1.00mm_Horizontal
- moved J2 70.2 mm to (135.0, 114.0)
- moved R5 10.3 mm to (211.1, 120.4), turned to -90 degrees
- moved D65 9.27 mm to (220.0, 111.5)
- moved R8 8.14 mm to (214.3, 107.9)
- moved R6 6.28 mm to (201.7, 109.1)
- moved R9 6.20 mm to (197.1, 109.0)
- moved D64 5.82 mm to (174.4, 104.5)
- moved R4 5.52 mm to (178.7, 104.5)
- moved U3 5.12 mm to (214.2, 115.3)
- moved R7 5.12 mm to (199.3, 105.3), turned to 180 degrees
- moved X1 4.53 mm to (189.9, 107.1)
- moved R1 3.44 mm to (188.9, 121.2)
- moved Q2 3.09 mm to (194.6, 113.4)
- moved Q1 2.54 mm to (205.0, 114.1)
- moved D63 1.39 mm to (206.0, 120.0)
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Other:
- board outline added: 285.8 x 95.2 mm
