File: PH60/_autosave-PH60.kicad_sch (KiCad schematic)
At the start: 23 parts, among them J1 USB-C USB 2.0 MC-372, J2 Conn_01x04, J3 Conn_01x02, Q1 AO3407, Q2 AO3407, U1 E73-2G4M08S1C, U2 AP2112K-3.3, U3 TP4054, U4 ProMicro, X1 32768kHz

Commit message: PCB Updates
Parts:
- removed J1: USB-C USB 2.0 MC-372, nrfmicro:USB-C_C168688, symbol nrfmicro:USB_C_Receptacle_USB2.0
- removed R2, R3: 5.1K, Resistor_SMD:R_0603_1608Metric, symbol Device:R
