File: PCB_Rev2/PH60_Rev2.kicad_pcb (KiCad board)
At the start: 4 copper layers, 285.7 x 95.2 mm, 151 parts, among them J2 Conn_01x02, J3 Conn_01x04, U1 NCP1117-3.3_SOT223, U2 W25Q128JVS, U3 RP2040, Y1 Crystal_GND24

Commit message: PCB Update
Finished the wiring of PCB
Parts:
- moved R3 67.5 mm to (137.0, 117.5), turned to 0 degrees
- moved R4 64.6 mm to (137.0, 118.4), turned to 0 degrees
- moved C7 59.2 mm to (170.3, 116.9), turned to 90 degrees
- moved J2 59.0 mm to (134.4, 107.1), turned to 0 degrees
- moved R1 58.3 mm to (132.3, 107.6)
- moved U2 57.4 mm to (126.7, 109.5)
- moved C5 49.4 mm to (126.7, 112.9), turned to 0 degrees
- moved R2 49.3 mm to (126.7, 106.2), turned to 0 degrees
- moved C4 45.9 mm to (171.3, 116.9), turned to 90 degrees
- moved C3 44.1 mm to (155.6, 118.5), turned to 90 degrees
- moved C2 43.1 mm to (150.4, 118.5)
- moved Y1 41.4 mm to (153.0, 118.5)
- moved R5 37.4 mm to (153.0, 120.7), turned to 180 degrees
- moved C1 35.7 mm to (182.1, 110.0), turned to 90 degrees
- moved U1 34.1 mm to (176.4, 110.0)
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Connections:
- C11 pad 2: Net-(C11-Pad2) -> GND
- C12 pad 2: Net-(C11-Pad2) -> GND
- C13 pad 2: Net-(C11-Pad2) -> GND
- C14 pad 2: Net-(C11-Pad2) -> GND
- C15 pad 2: Net-(C11-Pad2) -> GND
- C16 pad 2: Net-(C11-Pad2) -> GND
- C9 pad 2: Net-(C11-Pad2) -> GND
- U3 pad 56: unconnected-(U3-QSPI_SS-Pad56) -> /QSPI_SS
Routing:
- net +3V3: track 19.4 -> 192.6 mm, vias 2 -> 13
- net row_4: track 119.1 -> 266.8 mm
- net col_13: track 127.7 -> 270.5 mm, vias 0 -> 6
- net col_12: track 56.7 -> 196.7 mm, vias 0 -> 3
- net col_0: track 87.8 -> 196.1 mm, vias 0 -> 6
- net col_10: track 110.2 -> 209.4 mm, vias 8 -> 6
- net Net-(U3-USB_DP): track 89.5 -> 3.46 mm
- net col_11: track 149.6 -> 232.6 mm, vias 4 -> 6
- net Net-(U3-USB_DM): track 86.1 -> 3.69 mm
- net row_0: track 257.2 -> 336.5 mm, vias 0 -> 2
- net col_1: track 103.4 -> 180.9 mm
- net col_9: track 112.8 -> 186.9 mm, vias 8 -> 6
- net /QSPI_SD1: track 82.1 -> 12.6 mm
- net col_8: track 75.0 -> 140.6 mm, vias 6 -> 5
- net /QSPI_SD2: track 77.0 -> 12.2 mm
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- removed copper zone on In1.Cu, net +3V3
- removed copper zone on In2.Cu, net GND
Other:
- board size 285.7 x 95.2 mm -> 285.8 x 95.2 mm

Commit message: PCB Copper Filling
Routing:
- net +3V3: track 192.6 -> 196.3 mm
- net /QSPI_SS: track 13.2 -> 16.8 mm
- net GND: track 31.0 -> 32.9 mm, vias 8 -> 10
- added copper zone on B.Cu, net (none)
- added copper zone on In1.Cu, net (none)
- added copper zone on In2.Cu, net (none)
- added copper zone on F.Cu, net GND
Changed lines of the file:
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@@
 		(tags "capacitor")
 		(property "Reference" "C9"
-			(at 0 1.16 360)
+			(at 0 1.16 0)
 			(layer "B.SilkS")
 			(effects
@@
 		)
 		(property "Value" "100n"
-			(at 0 -1.16 360)
+			(at 0 -1.16 0)
 			(layer "B.Fab")
 			(effects
@@
 		)
 		(fp_text user "${REFERENCE}"
-			(at 0 0 360)
+			(at 0 0 0)
 			(layer "B.Fab")
 			(effects
@@
 		(net 2)
 	)
+	(via
+		(at 144.225 116.125)
+		(size 0.6)
+		(drill 0.3)
+		(layers "F.Cu" "B.Cu")
+		(net 2)
+	)
+	(via
+		(at 141.775 104.075)
+		(size 0.6)
+		(drill 0.3)
+		(layers "F.Cu" "B.Cu")
+		(net 2)
+	)
+	(segment
+		(start 141.775 105.075)
+		(end 142.695 105.075)
+		(width 0.2)
+		(layer "B.Cu")
+		(net 2)
+	)
 	(segment
 		(start 179.575 107.675)
@@
 	)
 	(segment
+		(start 144.225 116.1125)
+		(end 144.225 116.125)
+		(width 0.2)
+		(layer "B.Cu")
+		(net 2)
+	)
+	(segment
+		(start 141.775 105.075)
+		(end 141.775 104.075)
+		(width 0.2)
+		(layer "B.Cu")
+		(net 2)
+	)
+	(segment
 		(start 130.855 118.965)
 		(end 130.845 118.975)
@@
 	)
 	(segment
+		(start 126.175 106.175)
+		(end 124.52 106.175)
+		(width 0.2)
+		(layer "B.Cu")
+		(net 5)
+	)
+	(segment
 		(start 141.775 106.035)
 		(end 141.775 107.275)
@@
 	)
 	(segment
+		(start 124.52 106.175)
+		(end 123.075 107.62)
+		(width 0.2)
+		(layer "B.Cu")
+		(net 5)
+	)
+	(segment
 		(start 142.695 108.195)
 		(end 142.725 108.225)
@@
 	)
 	(segment
+		(start 128.83 106.175)
+		(end 130.275 107.62)
+		(width 0.2)
+		(layer "B.Cu")
+		(net 77)
+	)
+	(segment
 		(start 132.215 107.993924)
 		(end 132.711076 108.49)
@@
 	)
 	(segment
+		(start 127.195 106.175)
+		(end 128.83 106.175)
+		(width 0.2)
+		(layer "B.Cu")
+		(net 77)
+	)
+	(segment
 		(start 131.765 107.625)
 		(end 132.215 107.625)
@@
 		(net 99)
 	)
+	(zone
+		(net 2)
+		(net_name "GND")
+		(layer "F.Cu")
+		(hatch edge 0.5)
+		(connect_pads
+			(clearance 0.5)
+		)
+		(min_thickness 0.25)
+		(filled_areas_thickness no)
+		(fill
+			(thermal_gap 0.5)
+			(thermal_bridge_width 0.5)
+		)
+		(polygon
+			(pts
+				(xy 28.575 28.575) (xy 28.575 123.825) (xy 314.325 123.825) (xy 314.325 28.575)
+			)
+		)
+	)
+	(zone
+		(net 0)
+		(net_name "")
+		(layers "In1.Cu" "In2.Cu" "B.Cu")
+		(hatch edge 0.5)
+		(priority 1)
+		(connect_pads
+			(clearance 0.5)
+		)
+		(min_thickness 0.25)
+		(filled_areas_thickness no)
+		(fill
+			(thermal_gap 0.5)
+			(thermal_bridge_width 0.5)
+			(island_removal_mode 1)
+			(island_area_min 10)
+		)
+		(polygon
+			(pts
+				(xy 28.575 28.575) (xy 28.575 123.825) (xy 314.325 123.825) (xy 314.325 28.575)
+			)
+		)
+	)
 )
