File: PCB_Rev3/Multi/RGB.kicad_sch (KiCad schematic)
At the start: 62 parts

Commit message: muliti layout
Parts:
- C23: renamed from C22; now not fitted
- RGB1, RGB10, RGB11, RGB12, RGB13, RGB14, RGB15, RGB16, RGB17, RGB18, RGB19, RGB2, RGB20, RGB21, RGB22, RGB23, RGB24, RGB25, RGB26, RGB27, RGB28, RGB29, RGB3, RGB30, RGB31, RGB32, RGB33, RGB34, RGB35, RGB36, RGB37, RGB38, RGB39, RGB4, RGB40, RGB41, RGB42, RGB43, RGB44, RGB45, RGB46, RGB47, RGB48, RGB49, RGB5, RGB50, RGB51, RGB52, RGB53, RGB54, RGB55, RGB56, RGB57, RGB58, RGB59, RGB6, RGB60, RGB61, RGB7, RGB8, RGB9: now not fitted; now left out of the parts list
