File: PCB_Rev3/Multi/PH60_Rev3.kicad_sch (KiCad schematic)
At the start: 47 parts, among them J1 Conn_01x02_Pin, J2 Conn_01x02_Pin, J3 USB_C_Receptacle_USB2.0_16P, J4 Conn_01x04_Socket, U1 TP4057, U2 nRF52840, U4 TPS2116DRL, X1 32.768kHz, X2 Crystal_Generic

Commit message: 供电原理图审查
Connections:
- net BATT_STAT: now also U4.8 (ST)
Changed lines of the file:
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@@
+	(wire
+		(pts
+			(xy 80.01 191.77) (xy 76.2 191.77)
+		)
+		(stroke
+			(width 0)
+			(type default)
+		)
+	)
 	(wire
 		(pts
@@
 	(global_label "BATT_STAT"
 		(shape input)
-		(at 77.47 191.77 0)
+		(at 80.01 191.77 0)
 		(fields_autoplaced yes)
 		(effects
@@
 		)
 		(property "Intersheetrefs" "${INTERSHEET_REFS}"
-			(at 89.9499 191.77 0)
+			(at 92.4899 191.77 0)
 			(effects
 				(font

Commit message: Replace cap
Parts:
- C11, C9: footprint (none) -> Capacitor_SMD:C_0402_1005Metric
- J3: footprint Connector_USB:USB_C_Receptacle_GCT_USB4105-xx-A_16P_TopMnt_Horizontal -> Library:USB-C_16P_HandSolder
- R1, R2, R3: footprint (none) -> Resistor_SMD:R_0402_1005Metric
Connections:
- net CHRG is gone; now on net BATT_STAT: U2.A14 (P1.15)
- net VBUS_USB is gone; now on net VBUS: C11.1, D1.4 (VCC), J3.A4 (VBUS), J3.A9 (VBUS), J3.B4 (VBUS), J3.B9 (VBUS), J4.1 (Pin_1), R1.1, U1.4 (V_{CC}), U4.3 (VIN1), U4.5 (MODE)
- net VDDH is gone; now on net +BATT: C3.2, U2.Y2 (VDDH)
- net batt_level: no longer names the net of U2.B13 (AIN1/P0.03)
