File: PCB_Rev3/ISO60/PH60_Rev3.kicad_pcb (KiCad board)
At the start: 4 copper layers, 285.8 x 95.2 mm, 151 parts, among them J2 Conn_01x02, J3 Conn_01x04, U1 NCP1117-3.3_SOT223, U2 W25Q128JVS, U3 RP2040, Y1 Crystal_GND24

Commit message: Update PCB Rev3
Parts:
- removed J3: Conn_01x04, Connector_FFC-FPC:Molex_200528-0040_1x04-1MP_P1.00mm_Horizontal
- removed R2: DNF, Resistor_SMD:R_0402_1005Metric
- added J1: USB_C_Receptacle_USB2.0_16P, Connector_USB:USB_C_Receptacle_GCT_USB4105-xx-A_16P_TopMnt_Horizontal, B.Cu at (52.1, 41.6)
- added R6: 5K1, Resistor_SMD:R_0402_1005Metric, B.Cu at (182.9, 153.3)
- added R7: 5K1, Resistor_SMD:R_0402_1005Metric, B.Cu at (182.9, 155.3)
- C2, C3: value 15p -> 20p
- U1: value NCP1117-3.3_SOT223 -> TLV1117-33
- moved U1 49.9 mm to (165.0, 158.5)
- moved C4 49.5 mm to (122.5, 125.5), turned to 180 degrees
- moved C1 45.4 mm to (180.0, 155.3), turned to 180 degrees
- moved C11 43.9 mm to (131.0, 129.0), turned to -90 degrees
- moved C12 42.0 mm to (132.0, 129.0), turned to -90 degrees
- moved C16 40.5 mm to (105.5, 123.5), turned to 180 degrees
- moved C7 32.3 mm to (139.0, 125.0), turned to 0 degrees
- moved J2 20.9 mm to (116.5, 118.0), turned to 90 degrees
- moved U2 18.7 mm to (113.0, 122.2)
- moved C15 17.8 mm to (130.0, 118.0)
- moved R1 17.2 mm to (119.0, 118.5), turned to -90 degrees
- moved C10 13.4 mm to (126.0, 128.0)
- moved C8 13.3 mm to (126.0, 127.0)
- moved R4 13.3 mm to (126.0, 126.0)
- moved R3 13.3 mm to (126.0, 125.0)
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Routing:
- net row_0: track 336.6 -> 0.00 mm, vias 2 -> 0
- net row_1: track 328.6 -> 0.00 mm, vias 2 -> 0
- net row_2: track 288.2 -> 0.00 mm, vias 5 -> 0
- net row_3: track 279.1 -> 0.00 mm, vias 4 -> 0
- net col_13: track 270.5 -> 0.00 mm, vias 6 -> 0
- net row_4: track 265.3 -> 0.00 mm
- net col_11: track 232.6 -> 0.00 mm, vias 6 -> 0
- net col_10: track 209.4 -> 0.00 mm, vias 6 -> 0
- net col_12: track 196.7 -> 0.00 mm, vias 3 -> 0
- net col_0: track 196.1 -> 0.00 mm, vias 6 -> 0
- net col_9: track 186.9 -> 0.00 mm, vias 6 -> 0
- net col_1: track 180.9 -> 0.00 mm, vias 6 -> 0
- net +3V3: track 199.4 -> 29.0 mm, vias 13 -> 0
- net col_2: track 164.4 -> 0.00 mm, vias 6 -> 0
- net col_8: track 140.6 -> 0.00 mm, vias 5 -> 0
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- removed copper zone on B.Cu, net (none)
- removed copper zone on In2.Cu, net (none)
- removed copper zone on In1.Cu, net +3V3
- removed copper zone on F.Cu, net GND
Other:
- board outline removed

Commit message: modify routing
Parts:
- moved R6 167.0 mm to (52.7, 48.6)
- moved R7 167.0 mm to (52.7, 50.6)
- moved U1 41.1 mm to (185.0, 122.6)
- moved C1 34.6 mm to (191.0, 122.5), turned to 90 degrees
Connections:
- D28 pad 1: row_1 -> row_2
- S41 pad 2: col_13 -> col_12
- S59 pad 2: col_9 -> col_10
- S60 pad 2: col_10 -> col_11
- S61 pad 2: col_11 -> col_12
- U3 pad 26: /RUN -> unconnected-(U3-RUN-Pad26)
Routing:
- net row_0: track 0.00 -> 274.9 mm
- net row_2: track 0.00 -> 261.1 mm
- net row_3: track 0.00 -> 247.7 mm
- net row_1: track 0.00 -> 233.4 mm
- net row_4: track 0.00 -> 190.5 mm
- net col_2: track 0.00 -> 114.2 mm, vias 0 -> 5
- net col_12: track 0.00 -> 113.9 mm, vias 0 -> 4
- net col_1: track 0.00 -> 113.9 mm, vias 0 -> 5
- net col_13: track 0.00 -> 112.2 mm, vias 0 -> 4
- net col_0: track 0.00 -> 99.7 mm, vias 0 -> 5
- net col_6: track 0.00 -> 85.5 mm, vias 0 -> 4
- net col_4: track 0.00 -> 85.5 mm, vias 0 -> 4
- net col_5: track 0.00 -> 85.5 mm, vias 0 -> 4
- net col_9: track 0.00 -> 85.5 mm, vias 0 -> 4
- net col_8: track 0.00 -> 85.5 mm, vias 0 -> 4
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
Commit message: PCB Rev3 Layout
Parts:
- J2: footprint Connector_PinHeader_1.00mm:PinHeader_1x02_P1.00mm_Vertical -> Connector_PinHeader_2.54mm:PinHeader_1x02_P2.54mm_Vertical
- moved C1 85.3 mm to (105.8, 118.1), turned to 0 degrees
- moved U1 79.7 mm to (105.8, 113.1), turned to 90 degrees
- moved C16 31.1 mm to (136.5, 120.6)
- moved C5 20.8 mm to (137.5, 110.1), turned to 90 degrees
- moved C6 19.7 mm to (141.2, 117.3), turned to -90 degrees
- moved C14 19.3 mm to (116.8, 108.8), turned to 180 degrees
- moved C12 18.7 mm to (132.8, 110.3), turned to 90 degrees
- moved D27 17.5 mm to (271.1, 60.7)
- moved D54 17.5 mm to (283.1, 98.8)
- moved D20 17.5 mm to (137.8, 60.7)
- moved D21 17.5 mm to (156.8, 60.7)
- moved D23 17.5 mm to (194.9, 60.7)
- moved D25 17.5 mm to (233.0, 60.7)
- moved D26 17.5 mm to (252.1, 60.7)
- moved D10 17.5 mm to (204.5, 41.6)
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Routing:
- net col_13: track 112.2 -> 285.2 mm, vias 4 -> 5
- net /USB_D+: track 1.54 -> 167.3 mm, vias 1 -> 2
- net /USB_D-: track 1.33 -> 166.9 mm, vias 1 -> 2
- net col_12: track 113.9 -> 265.4 mm, vias 4 -> 5
- net col_11: track 85.5 -> 235.5 mm, vias 4 -> 6
- net VBUS: track 3.89 -> 140.7 mm, vias 0 -> 2
- net col_10: track 85.5 -> 213.6 mm, vias 4 -> 6
- net col_9: track 85.5 -> 173.2 mm, vias 4 -> 5
- net col_0: track 99.7 -> 185.6 mm, vias 5 -> 4
- net row_4: track 190.5 -> 267.7 mm
- net col_8: track 85.5 -> 154.7 mm, vias 4 -> 5
- net row_0: track 274.9 -> 343.9 mm, vias 0 -> 2
- net row_2: track 261.1 -> 329.3 mm, vias 0 -> 2
- net +3V3: track 29.0 -> 93.5 mm, vias 0 -> 6
- net row_1: track 233.4 -> 293.1 mm, vias 0 -> 2
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- added copper zone on B.Cu, net (none)
- added copper zone on F.Cu, net GND
Other:
- board outline added: 285.8 x 95.2 mm
- copper layers 4 -> 2

Commit message: Add RGB Lighting for PCB Rev3
Parts:
- added REF**: Stabilizer_Cherry_MX_2.00u, PCM_Mounting_Keyboard_Stabilizer:Stabilizer_Cherry_MX_2.00u, F.Cu at (302.4, 66.7)
- added REF**: Stabilizer_Cherry_MX_2.00u, PCM_Mounting_Keyboard_Stabilizer:Stabilizer_Cherry_MX_2.00u, F.Cu at (295.3, 38.1)
- added REF**: Stabilizer_Cherry_MX_2.00u, PCM_Mounting_Keyboard_Stabilizer:Stabilizer_Cherry_MX_2.00u, F.Cu at (288.1, 95.2)
- added REF**: Stabilizer_Cherry_MX_6.25u, PCM_Mounting_Keyboard_Stabilizer:Stabilizer_Cherry_MX_6.25u, F.Cu at (159.5, 114.3)
- added RGB1: WS2812B, RGB:ws2812B_6028, B.Cu at (38.1, 32.6)
- added RGB10: WS2812B, RGB:ws2812B_6028, B.Cu at (209.6, 43.6)
- added RGB11: WS2812B, RGB:ws2812B_6028, B.Cu at (228.6, 43.6)
- added RGB12: WS2812B, RGB:ws2812B_6028, B.Cu at (247.7, 43.6)
- added RGB13: WS2812B, RGB:ws2812B_6028, B.Cu at (266.7, 43.6)
- added RGB14: WS2812B, RGB:ws2812B_6028, B.Cu at (295.3, 43.6)
- added RGB15: WS2812B, RGB:ws2812B_6028, B.Cu at (42.9, 62.6)
- added RGB16: WS2812B, RGB:ws2812B_6028, B.Cu at (66.7, 62.6)
- added RGB17: WS2812B, RGB:ws2812B_6028, B.Cu at (85.7, 62.6)
- added RGB18: WS2812B, RGB:ws2812B_6028, B.Cu at (104.8, 62.6)
- added RGB19: WS2812B, RGB:ws2812B_6028, B.Cu at (123.8, 62.6)
- added RGB2: WS2812B, RGB:ws2812B_6028, B.Cu at (57.1, 32.6)
- added RGB20: WS2812B, RGB:ws2812B_6028, B.Cu at (142.9, 62.6)
- added RGB21: WS2812B, RGB:ws2812B_6028, B.Cu at (161.9, 62.6)
- added RGB22: WS2812B, RGB:ws2812B_6028, B.Cu at (181.0, 62.6)
- added RGB23: WS2812B, RGB:ws2812B_6028, B.Cu at (200.0, 62.6)
- added RGB24: WS2812B, RGB:ws2812B_6028, B.Cu at (219.1, 62.6)
- added RGB25: WS2812B, RGB:ws2812B_6028, B.Cu at (238.1, 62.6)
- added RGB26: WS2812B, RGB:ws2812B_6028, B.Cu at (257.2, 62.6)
- added RGB27: WS2812B, RGB:ws2812B_6028, B.Cu at (276.2, 62.6)
- added RGB28: WS2812B, RGB:ws2812B_6028, B.Cu at (302.4, 72.2)
- added RGB29: WS2812B, RGB:ws2812B_6028, B.Cu at (45.2, 81.7)
- added RGB3: WS2812B, RGB:ws2812B_6028, B.Cu at (76.2, 43.6)
- added RGB30: WS2812B, RGB:ws2812B_6028, B.Cu at (71.4, 81.7)
- added RGB31: WS2812B, RGB:ws2812B_6028, B.Cu at (90.5, 81.7)
- added RGB32: WS2812B, RGB:ws2812B_6028, B.Cu at (109.5, 81.7)
- added RGB33: WS2812B, RGB:ws2812B_6028, B.Cu at (128.6, 81.7)
- added RGB34: WS2812B, RGB:ws2812B_6028, B.Cu at (147.6, 81.7)
- added RGB35: WS2812B, RGB:ws2812B_6028, B.Cu at (166.7, 81.7)
- added RGB36: WS2812B, RGB:ws2812B_6028, B.Cu at (185.7, 81.7)
- added RGB37: WS2812B, RGB:ws2812B_6028, B.Cu at (204.8, 81.7)
- added RGB38: WS2812B, RGB:ws2812B_6028, B.Cu at (223.8, 81.7)
- added RGB39: WS2812B, RGB:ws2812B_6028, B.Cu at (242.9, 81.7)
- added RGB4: WS2812B, RGB:ws2812B_6028, B.Cu at (95.2, 43.6)
- added RGB40: WS2812B, RGB:ws2812B_6028, B.Cu at (261.9, 81.7)
- added RGB41: WS2812B, RGB:ws2812B_6028, B.Cu at (281.0, 81.7)
- added RGB42: WS2812B, RGB:ws2812B_6028, B.Cu at (40.5, 100.8)
- added RGB43: WS2812B, RGB:ws2812B_6028, B.Cu at (61.9, 100.8)
- added RGB44: WS2812B, RGB:ws2812B_6028, B.Cu at (81.0, 100.8)
- added RGB45: WS2812B, RGB:ws2812B_6028, B.Cu at (100.0, 100.8)
- added RGB46: WS2812B, RGB:ws2812B_6028, B.Cu at (119.1, 100.8)
- added RGB47: WS2812B, RGB:ws2812B_6028, B.Cu at (138.1, 100.8)
- added RGB48: WS2812B, RGB:ws2812B_6028, B.Cu at (157.2, 100.8)
- added RGB49: WS2812B, RGB:ws2812B_6028, B.Cu at (176.2, 100.8)
- added RGB5: WS2812B, RGB:ws2812B_6028, B.Cu at (114.3, 43.6)
- added RGB50: WS2812B, RGB:ws2812B_6028, B.Cu at (195.3, 100.8)
- added RGB51: WS2812B, RGB:ws2812B_6028, B.Cu at (214.3, 100.8)
- added RGB52: WS2812B, RGB:ws2812B_6028, B.Cu at (233.4, 100.8)
- added RGB53: WS2812B, RGB:ws2812B_6028, B.Cu at (252.4, 100.8)
- added RGB54: WS2812B, RGB:ws2812B_6028, B.Cu at (288.1, 100.8)
- added RGB55: WS2812B, RGB:ws2812B_6028, B.Cu at (40.5, 119.8)
- added RGB56: WS2812B, RGB:ws2812B_6028, B.Cu at (64.3, 119.8)
- added RGB57: WS2812B, RGB:ws2812B_6028, B.Cu at (88.1, 119.8)
- added RGB58: WS2812B, RGB:ws2812B_6028, B.Cu at (159.5, 119.8)
- added RGB59: WS2812B, RGB:ws2812B_6028, B.Cu at (231.0, 119.8)
- added RGB6: WS2812B, RGB:ws2812B_6028, B.Cu at (133.3, 43.6)
- added RGB60: WS2812B, RGB:ws2812B_6028, B.Cu at (254.8, 119.8)
- added RGB61: WS2812B, RGB:ws2812B_6028, B.Cu at (278.6, 119.8)
- added RGB62: WS2812B, RGB:ws2812B_6028, B.Cu at (302.4, 119.8)
- added RGB7: WS2812B, RGB:ws2812B_6028, B.Cu at (152.4, 43.6)
- added RGB8: WS2812B, RGB:ws2812B_6028, B.Cu at (171.4, 43.6)
- added RGB9: WS2812B, RGB:ws2812B_6028, B.Cu at (190.5, 43.6)
- added RGBC1: 100n, Capacitor_SMD:C_0402_1005Metric, B.Cu at (40.8, 35.6)
- added RGBC10: 100n, Capacitor_SMD:C_0402_1005Metric, B.Cu at (214.6, 44.4)
- added RGBC11: 100n, Capacitor_SMD:C_0402_1005Metric, B.Cu at (233.7, 44.4)
- added RGBC12: 100n, Capacitor_SMD:C_0402_1005Metric, B.Cu at (252.7, 44.4)
- added RGBC13: 100n, Capacitor_SMD:C_0402_1005Metric, B.Cu at (271.8, 44.4)
- added RGBC14: 100n, Capacitor_SMD:C_0402_1005Metric, B.Cu at (300.4, 44.4)
- added RGBC15: 100n, Capacitor_SMD:C_0402_1005Metric, B.Cu at (47.9, 63.4)
- added RGBC16: 100n, Capacitor_SMD:C_0402_1005Metric, B.Cu at (71.8, 63.4)
- added RGBC17: 100n, Capacitor_SMD:C_0402_1005Metric, B.Cu at (90.8, 63.4)
- added RGBC18: 100n, Capacitor_SMD:C_0402_1005Metric, B.Cu at (109.9, 63.4)
- added RGBC19: 100n, Capacitor_SMD:C_0402_1005Metric, B.Cu at (128.9, 63.4)
- added RGBC2: 100n, Capacitor_SMD:C_0402_1005Metric, B.Cu at (62.2, 31.9)
- added RGBC20: 100n, Capacitor_SMD:C_0402_1005Metric, B.Cu at (148.0, 63.4)
- added RGBC21: 100n, Capacitor_SMD:C_0402_1005Metric, B.Cu at (167.0, 63.4)
- added RGBC22: 100n, Capacitor_SMD:C_0402_1005Metric, B.Cu at (186.1, 63.4)
- added RGBC23: 100n, Capacitor_SMD:C_0402_1005Metric, B.Cu at (205.1, 63.4)
- added RGBC24: 100n, Capacitor_SMD:C_0402_1005Metric, B.Cu at (224.2, 63.4)
- added RGBC25: 100n, Capacitor_SMD:C_0402_1005Metric, B.Cu at (243.2, 63.4)
- added RGBC26: 100n, Capacitor_SMD:C_0402_1005Metric, B.Cu at (262.3, 63.4)
- added RGBC27: 100n, Capacitor_SMD:C_0402_1005Metric, B.Cu at (281.3, 63.4)
- added RGBC28: 100n, Capacitor_SMD:C_0402_1005Metric, B.Cu at (307.5, 72.9)
- added RGBC29: 100n, Capacitor_SMD:C_0402_1005Metric, B.Cu at (50.3, 82.5)
- added RGBC3: 100n, Capacitor_SMD:C_0402_1005Metric, B.Cu at (81.3, 44.4)
- added RGBC30: 100n, Capacitor_SMD:C_0402_1005Metric, B.Cu at (76.5, 82.5)
- added RGBC31: 100n, Capacitor_SMD:C_0402_1005Metric, B.Cu at (95.6, 82.5)
- added RGBC32: 100n, Capacitor_SMD:C_0402_1005Metric, B.Cu at (114.6, 82.5)
- added RGBC33: 100n, Capacitor_SMD:C_0402_1005Metric, B.Cu at (133.7, 82.5)
- added RGBC34: 100n, Capacitor_SMD:C_0402_1005Metric, B.Cu at (152.7, 82.5)
- added RGBC35: 100n, Capacitor_SMD:C_0402_1005Metric, B.Cu at (171.8, 82.5)
- added RGBC36: 100n, Capacitor_SMD:C_0402_1005Metric, B.Cu at (190.8, 82.5)
- added RGBC37: 100n, Capacitor_SMD:C_0402_1005Metric, B.Cu at (209.9, 82.5)
- added RGBC38: 100n, Capacitor_SMD:C_0402_1005Metric, B.Cu at (228.9, 82.5)
- added RGBC39: 100n, Capacitor_SMD:C_0402_1005Metric, B.Cu at (248.0, 82.5)
- added RGBC4: 100n, Capacitor_SMD:C_0402_1005Metric, B.Cu at (100.3, 44.4)
- added RGBC40: 100n, Capacitor_SMD:C_0402_1005Metric, B.Cu at (267.0, 82.5)
- added RGBC41: 100n, Capacitor_SMD:C_0402_1005Metric, B.Cu at (286.1, 82.5)
- added RGBC42: 100n, Capacitor_SMD:C_0402_1005Metric, B.Cu at (45.6, 101.5)
- added RGBC43: 100n, Capacitor_SMD:C_0402_1005Metric, B.Cu at (67.0, 101.5)
- added RGBC44: 100n, Capacitor_SMD:C_0402_1005Metric, B.Cu at (86.0, 101.5)
- added RGBC45: 100n, Capacitor_SMD:C_0402_1005Metric, B.Cu at (105.1, 101.5)
- added RGBC46: 100n, Capacitor_SMD:C_0402_1005Metric, B.Cu at (124.1, 101.5)
- added RGBC47: 100n, Capacitor_SMD:C_0402_1005Metric, B.Cu at (143.2, 101.5)
- added RGBC48: 100n, Capacitor_SMD:C_0402_1005Metric, B.Cu at (162.2, 101.5)
- added RGBC49: 100n, Capacitor_SMD:C_0402_1005Metric, B.Cu at (181.3, 101.5)
- added RGBC5: 100n, Capacitor_SMD:C_0402_1005Metric, B.Cu at (119.4, 44.4)
- added RGBC50: 100n, Capacitor_SMD:C_0402_1005Metric, B.Cu at (200.3, 101.5)
- added RGBC51: 100n, Capacitor_SMD:C_0402_1005Metric, B.Cu at (219.4, 101.5)
- added RGBC52: 100n, Capacitor_SMD:C_0402_1005Metric, B.Cu at (238.4, 101.5)
- added RGBC53: 100n, Capacitor_SMD:C_0402_1005Metric, B.Cu at (257.5, 101.5)
- added RGBC54: 100n, Capacitor_SMD:C_0402_1005Metric, B.Cu at (293.2, 101.5)
- added RGBC55: 100n, Capacitor_SMD:C_0402_1005Metric, B.Cu at (45.6, 120.5)
- added RGBC56: 100n, Capacitor_SMD:C_0402_1005Metric, B.Cu at (69.4, 120.5)
- added RGBC57: 100n, Capacitor_SMD:C_0402_1005Metric, B.Cu at (93.2, 120.5)
- added RGBC58: 100n, Capacitor_SMD:C_0402_1005Metric, B.Cu at (164.6, 120.5)
- added RGBC59: 100n, Capacitor_SMD:C_0402_1005Metric, B.Cu at (236.1, 120.5)
- added RGBC6: 100n, Capacitor_SMD:C_0402_1005Metric, B.Cu at (138.4, 44.4)
- added RGBC60: 100n, Capacitor_SMD:C_0402_1005Metric, B.Cu at (259.9, 120.5)
- added RGBC61: 100n, Capacitor_SMD:C_0402_1005Metric, B.Cu at (283.7, 120.5)
- added RGBC62: 100n, Capacitor_SMD:C_0402_1005Metric, B.Cu at (307.5, 120.5)
- added RGBC7: 100n, Capacitor_SMD:C_0402_1005Metric, B.Cu at (157.5, 44.4)
- added RGBC8: 100n, Capacitor_SMD:C_0402_1005Metric, B.Cu at (176.5, 44.4)
- added RGBC9: 100n, Capacitor_SMD:C_0402_1005Metric, B.Cu at (195.6, 44.4)
- C1, C4: value 10u -> 1u
- D1, D10, D11, D12, D13, D14, D15, D16, D17, D18, D19, D2, D20, D21, D22, D23, D24, D25, D26, D27, D28, D29, D3, D30, D31, D32, D33, D34, D35, D36, D37, D38, D39, D4, D40, D41, D42, D43, D44, D45, D46, D47, D48, D49, D5, D50, D51, D52, D53, D54, D55, D56, D57, D58, D59, D6, D60, D61, D62, D7, D8, D9: footprint Diode_SMD:D_SOD-123 -> Diode_SMD:D_SOD-323
- S1, S10, S11, S12, S13, S16, S17, S18, S19, S2, S20, S21, S22, S23, S24, S25, S26, S27, S3, S30, S31, S32, S33, S34, S35, S36, S37, S38, S39, S4, S40, S41, S43, S44, S45, S46, S47, S48, S49, S5, S50, S51, S52, S53, S6, S7, S8, S9: footprint PCM_Switch_Keyboard_Hotswap_Kailh:SW_Hotswap_Kailh_MX_1.00u -> PCM_Switch_Keyboard_Hotswap_Kailh:SW_Hotswap_Kailh_MX_Plated_1.00u
- S14: footprint PCM_Switch_Keyboard_Hotswap_Kailh:SW_Hotswap_Kailh_MX_2.00u -> PCM_Switch_Keyboard_Hotswap_Kailh:SW_Hotswap_Kailh_MX_Plated_2.00u
- S15: footprint PCM_Switch_Keyboard_Hotswap_Kailh:SW_Hotswap_Kailh_MX_1.50u -> PCM_Switch_Keyboard_Hotswap_Kailh:SW_Hotswap_Kailh_MX_Plated_1.50u
- S28: footprint PCM_Switch_Keyboard_Hotswap_Kailh:SW_Hotswap_Kailh_MX_ISOEnter -> PCM_Switch_Keyboard_Hotswap_Kailh:SW_Hotswap_Kailh_MX_Plated_ISOEnter
- S29: footprint PCM_Switch_Keyboard_Hotswap_Kailh:SW_Hotswap_Kailh_MX_1.75u -> PCM_Switch_Keyboard_Hotswap_Kailh:SW_Hotswap_Kailh_MX_Plated_1.75u
- S42, S55, S56, S57, S59, S60, S61, S62: footprint PCM_Switch_Keyboard_Hotswap_Kailh:SW_Hotswap_Kailh_MX_1.25u -> PCM_Switch_Keyboard_Hotswap_Kailh:SW_Hotswap_Kailh_MX_Plated_1.25u
- S54: footprint PCM_Switch_Keyboard_Hotswap_Kailh:SW_Hotswap_Kailh_MX_2.75u -> PCM_Switch_Keyboard_Hotswap_Kailh:SW_Hotswap_Kailh_MX_Plated_2.75u
- S58: footprint PCM_Switch_Keyboard_Hotswap_Kailh:SW_Hotswap_Kailh_MX_6.25u -> PCM_Switch_Keyboard_Hotswap_Kailh:SW_Hotswap_Kailh_MX_Plated_6.25u
- U1: value TLV1117-33 -> ME6211C33M5; footprint Package_TO_SOT_SMD:SOT-223 -> Package_TO_SOT_SMD:SOT-23-5
- U2: value W25Q128JVS -> W25Q16JVSS; footprint Package_SO:SOIC-8_5.23x5.23mm_P1.27mm -> Package_SON:Winbond_USON-8-1EP_3x2mm_P0.5mm_EP0.2x1.6mm
- U3: footprint Package_DFN_QFN:QFN-56-1EP_7x7mm_P0.4mm_EP3.2x3.2mm -> Package_DFN_QFN:QFN-56-1EP_7x7mm_P0.4mm_EP3.2x3.2mm_ThermalVias
- moved C16 19.7 mm to (118.1, 113.6)
- moved C5 16.7 mm to (120.8, 109.0), turned to 0 degrees
- moved C3 14.8 mm to (133.7, 117.8), turned to -90 degrees
- moved C1 13.7 mm to (114.8, 107.8), turned to -90 degrees
- moved C9 13.3 mm to (130.6, 118.2)
- moved C7 11.1 mm to (118.8, 111.3), turned to 90 degrees
- moved U1 10.3 mm to (115.8, 110.5), turned to 0 degrees
- moved C15 10.3 mm to (130.3, 106.6), turned to 90 degrees
- moved D14 10.2 mm to (300.4, 41.1)
- moved D20 10.2 mm to (148.0, 60.2)
- moved D25 10.2 mm to (243.2, 60.2)
- moved D27 10.2 mm to (281.3, 60.2)
- moved D35 10.2 mm to (171.8, 79.2)
- moved D51 10.2 mm to (219.4, 98.3)
- moved D54 10.2 mm to (293.2, 98.3)
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Connections:
- J1 pad S1: unconnected-(J1-SHIELD-PadS1)_3 -> GND
- S1 pad 1: Net-(D1-A) -> col_0
- S1 pad 2: col_0 -> Net-(D1-A)
- S10 pad 1: Net-(D10-A) -> col_9
- S10 pad 2: col_9 -> Net-(D10-A)
- S11 pad 1: Net-(D11-A) -> col_10
- S11 pad 2: col_10 -> Net-(D11-A)
- S12 pad 1: Net-(D12-A) -> col_11
- S12 pad 2: col_11 -> Net-(D12-A)
- S13 pad 1: Net-(D13-A) -> col_12
- S13 pad 2: col_12 -> Net-(D13-A)
- S14 pad 1: Net-(D14-A) -> col_13
- S14 pad 2: col_13 -> Net-(D14-A)
- S15 pad 1: Net-(D15-A) -> col_0
- S15 pad 2: col_0 -> Net-(D15-A)
- S16 pad 1: Net-(D16-A) -> col_1
- S16 pad 2: col_1 -> Net-(D16-A)
- S17 pad 1: Net-(D17-A) -> col_2
- S17 pad 2: col_2 -> Net-(D17-A)
- S18 pad 1: Net-(D18-A) -> col_3
- S18 pad 2: col_3 -> Net-(D18-A)
- S19 pad 1: Net-(D19-A) -> col_4
- S19 pad 2: col_4 -> Net-(D19-A)
- S2 pad 1: Net-(D2-A) -> col_1
- S2 pad 2: col_1 -> Net-(D2-A)
- S20 pad 1: Net-(D20-A) -> col_5
- S20 pad 2: col_5 -> Net-(D20-A)
- S21 pad 1: Net-(D21-A) -> col_6
- S21 pad 2: col_6 -> Net-(D21-A)
- S22 pad 1: Net-(D22-A) -> col_7
- S22 pad 2: col_7 -> Net-(D22-A)
- S23 pad 1: Net-(D23-A) -> col_8
- S23 pad 2: col_8 -> Net-(D23-A)
- S24 pad 1: Net-(D24-A) -> col_9
- S24 pad 2: col_9 -> Net-(D24-A)
- S25 pad 1: Net-(D25-A) -> col_10
- S25 pad 2: col_10 -> Net-(D25-A)
- S26 pad 1: Net-(D26-A) -> col_11
- S26 pad 2: col_11 -> Net-(D26-A)
- S27 pad 1: Net-(D27-A) -> col_12
- S27 pad 2: col_12 -> Net-(D27-A)
- S28 pad 1: Net-(D28-A) -> col_13
- S28 pad 2: col_13 -> Net-(D28-A)
- S29 pad 1: Net-(D29-A) -> col_0
- S29 pad 2: col_0 -> Net-(D29-A)
- S3 pad 1: Net-(D3-A) -> col_2
- S3 pad 2: col_2 -> Net-(D3-A)
- S30 pad 1: Net-(D30-A) -> col_1
- S30 pad 2: col_1 -> Net-(D30-A)
- S31 pad 1: Net-(D31-A) -> col_2
- S31 pad 2: col_2 -> Net-(D31-A)
- S32 pad 1: Net-(D32-A) -> col_3
- S32 pad 2: col_3 -> Net-(D32-A)
- S33 pad 1: Net-(D33-A) -> col_4
- S33 pad 2: col_4 -> Net-(D33-A)
- S34 pad 1: Net-(D34-A) -> col_5
- S34 pad 2: col_5 -> Net-(D34-A)
- S35 pad 1: Net-(D35-A) -> col_6
- S35 pad 2: col_6 -> Net-(D35-A)
- S36 pad 1: Net-(D36-A) -> col_7
- S36 pad 2: col_7 -> Net-(D36-A)
- S37 pad 1: Net-(D37-A) -> col_8
- S37 pad 2: col_8 -> Net-(D37-A)
- S38 pad 1: Net-(D38-A) -> col_9
- S38 pad 2: col_9 -> Net-(D38-A)
- S39 pad 1: Net-(D39-A) -> col_10
- S39 pad 2: col_10 -> Net-(D39-A)
- S4 pad 1: Net-(D4-A) -> col_3
- S4 pad 2: col_3 -> Net-(D4-A)
- S40 pad 1: Net-(D40-A) -> col_11
- S40 pad 2: col_11 -> Net-(D40-A)
- S41 pad 1: Net-(D41-A) -> col_12
- S41 pad 2: col_12 -> Net-(D41-A)
- S42 pad 1: Net-(D42-A) -> col_0
- S42 pad 2: col_0 -> Net-(D42-A)
- S43 pad 1: Net-(D43-A) -> col_1
- S43 pad 2: col_1 -> Net-(D43-A)
- S44 pad 1: Net-(D44-A) -> col_2
- S44 pad 2: col_2 -> Net-(D44-A)
- S45 pad 1: Net-(D45-A) -> col_3
- S45 pad 2: col_3 -> Net-(D45-A)
- S46 pad 1: Net-(D46-A) -> col_4
- S46 pad 2: col_4 -> Net-(D46-A)
- S47 pad 1: Net-(D47-A) -> col_5
- S47 pad 2: col_5 -> Net-(D47-A)
- S48 pad 1: Net-(D48-A) -> col_6
- S48 pad 2: col_6 -> Net-(D48-A)
- S49 pad 1: Net-(D49-A) -> col_7
- S49 pad 2: col_7 -> Net-(D49-A)
- S5 pad 1: Net-(D5-A) -> col_4
- S5 pad 2: col_4 -> Net-(D5-A)
- S50 pad 1: Net-(D50-A) -> col_8
- S50 pad 2: col_8 -> Net-(D50-A)
- S51 pad 1: Net-(D51-A) -> col_9
- S51 pad 2: col_9 -> Net-(D51-A)
- S52 pad 1: Net-(D52-A) -> col_10
- S52 pad 2: col_10 -> Net-(D52-A)
- S53 pad 1: Net-(D53-A) -> col_11
- S53 pad 2: col_11 -> Net-(D53-A)
- S54 pad 1: Net-(D54-A) -> col_13
- S54 pad 2: col_13 -> Net-(D54-A)
- S55 pad 1: Net-(D55-A) -> col_0
- S55 pad 2: col_0 -> Net-(D55-A)
- S56 pad 1: Net-(D56-A) -> col_1
- S56 pad 2: col_1 -> Net-(D56-A)
- S57 pad 1: Net-(D57-A) -> col_2
- S57 pad 2: col_2 -> Net-(D57-A)
- S58 pad 1: Net-(D58-A) -> col_6
- S58 pad 2: col_6 -> Net-(D58-A)
- S59 pad 1: Net-(D59-A) -> col_10
- S59 pad 2: col_10 -> Net-(D59-A)
- S6 pad 1: Net-(D6-A) -> col_5
- S6 pad 2: col_5 -> Net-(D6-A)
- S60 pad 1: Net-(D60-A) -> col_11
- S60 pad 2: col_11 -> Net-(D60-A)
- S61 pad 1: Net-(D61-A) -> col_12
- S61 pad 2: col_12 -> Net-(D61-A)
- S62 pad 1: Net-(D62-A) -> col_13
- S62 pad 2: col_13 -> Net-(D62-A)
- S7 pad 1: Net-(D7-A) -> col_6
- S7 pad 2: col_6 -> Net-(D7-A)
- S8 pad 1: Net-(D8-A) -> col_7
- S8 pad 2: col_7 -> Net-(D8-A)
- S9 pad 1: Net-(D9-A) -> col_8
- S9 pad 2: col_8 -> Net-(D9-A)
- U1 pad 1: GND -> VBUS
- U1 pad 2: +3V3 -> VBUS
- U1 pad 3: VBUS -> GND
- U1 pad 4: (no net) -> unconnected-(U1-NC-Pad4)
- U3 pad 11: col_8 -> col_7
- U3 pad 12: col_9 -> col_13
- U3 pad 13: col_10 -> col_12
- U3 pad 15: col_12 -> col_10
- U3 pad 16: col_13 -> col_6
- U3 pad 17: row_0 -> unconnected-(U3-GPIO14-Pad17)
- U3 pad 18: row_1 -> unconnected-(U3-GPIO15-Pad18)
- U3 pad 2: col_0 -> col_4
- U3 pad 27: row_2 -> unconnected-(U3-GPIO16-Pad27)
- U3 pad 28: row_3 -> unconnected-(U3-GPIO17-Pad28)
- U3 pad 29: row_4 -> unconnected-(U3-GPIO18-Pad29)
- U3 pad 3: col_1 -> col_3
- U3 pad 34: unconnected-(U3-GPIO22-Pad34) -> row_4
- U3 pad 35: unconnected-(U3-GPIO23-Pad35) -> DIN
- U3 pad 36: unconnected-(U3-GPIO24-Pad36) -> row_3
- U3 pad 37: unconnected-(U3-GPIO25-Pad37) -> row_2
- U3 pad 38: unconnected-(U3-GPIO26_ADC0-Pad38) -> row_1
- U3 pad 39: unconnected-(U3-GPIO27_ADC1-Pad39) -> row_0
- U3 pad 5: col_3 -> col_1
- U3 pad 6: col_4 -> col_0
- U3 pad 8: col_6 -> col_9
- U3 pad 9: col_7 -> col_8
Routing:
- net VBUS: track 140.7 -> 1725.6 mm, vias 2 -> 4
- net Net-(RGB54-DOUT): track 0.00 -> 291.1 mm, vias 0 -> 2
- net Net-(RGB28-DOUT): track 0.00 -> 279.3 mm
- net Net-(RGB14-DOUT): track 0.00 -> 278.4 mm
- net Net-(RGB41-DOUT): track 0.00 -> 278.1 mm
- net DIN: track 0.00 -> 172.4 mm, vias 0 -> 2
- net GND: track 57.7 -> 184.1 mm, vias 14 -> 136
- net Net-(RGB57-DOUT): track 0.00 -> 68.1 mm
- net Net-(RGB58-DOUT): track 0.00 -> 67.6 mm
- net row_0: track 343.9 -> 401.5 mm, vias 2 -> 4
- net row_1: track 293.1 -> 333.5 mm
- net Net-(RGB53-DOUT): track 0.00 -> 30.9 mm
- net col_10: track 213.6 -> 185.3 mm, vias 6 -> 0
- net col_12: track 265.4 -> 239.3 mm, vias 5 -> 0
- net Net-(RGB27-DOUT): track 0.00 -> 25.3 mm
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- added copper zone on B.Cu, net GND
- removed copper zone on B.Cu, net (none)
Other:
- outline, holes or cut-outs redrawn
