File: PCB_Rev2/ISO/PH60_Rev2.kicad_pcb (KiCad board)
At the start: 2 copper layers, 285.8 x 95.2 mm, 280 parts, among them J1 USB_C_Receptacle_USB2.0_16P, J2 Conn_01x02, U1 ME6211C33M5, U2 W25Q16JVSS, U3 RP2040, Y1 Crystal_GND24

Commit message: Change LDO to XC6206
It must be work...
Parts:
- removed C1, C4: 1u, Capacitor_SMD:C_0402_1005Metric
- added C17: 1u, Capacitor_SMD:C_0402_1005Metric, B.Cu at (114.4, 107.4)
- added C18: 1u, Capacitor_SMD:C_0402_1005Metric, B.Cu at (115.8, 112.6)
- U1: value ME6211C33M5 -> XC6206PxxxMR; footprint Package_TO_SOT_SMD:SOT-23-5 -> Package_TO_SOT_SMD:SOT-23-3
- moved U1 1.71 mm to (114.3, 109.8), turned to 180 degrees
Connections:
- U1 pad 1: VBUS -> GND
- U1 pad 2: VBUS -> +3V3
- U1 pad 3: GND -> VBUS
Routing:
- net VBUS: track 1725.6 -> 1718.2 mm
- net GND: track 184.1 -> 185.7 mm, vias 136 -> 135
- net /USB_D+: track 150.3 -> 149.5 mm
- net /USB_D-: track 154.4 -> 153.7 mm

Commit message: Adjust margin to line distance.
Parts:
- moved C8 2.30 mm to (120.4, 116.0)
- moved C11 1.42 mm to (122.7, 117.7), turned to 180 degrees
- moved C10 0.73 mm to (122.7, 116.7)
- moved C13 0.35 mm to (124.8, 118.3), turned to 180 degrees
Routing:
- net +1V1: track 22.4 -> 24.6 mm
- net GND: track 185.7 -> 187.4 mm, vias 135 -> 134
- net +3V3: track 79.7 -> 78.4 mm
- net row_2: track 348.5 -> 347.9 mm
- net row_1: track 333.5 -> 333.0 mm
- net row_0: track 401.5 -> 400.9 mm
- net DIN: track 172.7 -> 172.1 mm
- net row_3: track 309.0 -> 308.5 mm
- net VBUS: track 1718.2 -> 1718.7 mm

Commit message: Project structure improvement.
Routing:
- net GND: track 187.4 -> 189.3 mm, vias 134 -> 136
