File: PCB_Rev2/Multi/matrix.kicad_sch (KiCad schematic)
At the start: 128 parts

Commit message: Wiring and Placing Improvement
Parts:
- S55: footprint PCM_Switch_Keyboard_Hotswap_Kailh:SW_Hotswap_Kailh_MX_Plated_1.75u_90deg -> PCM_Switch_Keyboard_Hotswap_Kailh:SW_Hotswap_Kailh_MX_Plated_2.75u_90deg
- S56: footprint PCM_Switch_Keyboard_Hotswap_Kailh:SW_Hotswap_Kailh_MX_Plated_2.75u_90deg -> PCM_Switch_Keyboard_Hotswap_Kailh:SW_Hotswap_Kailh_MX_Plated_1.00u
Other:
- moved on the sheet: S28, S41
Changed lines of the file:
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@@
 	)
 	(junction
+		(at 358.14 104.14)
+		(diameter 0)
+		(color 0 0 0 0)
+	)
+	(junction
 		(at 180.34 104.14)
 		(diameter 0)
@@
 	)
 	(junction
-		(at 383.54 82.55)
-		(diameter 0)
-		(color 0 0 0 0)
-	)
-	(junction
 		(at 347.98 135.89)
 		(diameter 0)
@@
 	)
 	(junction
+		(at 383.54 82.55)
+		(diameter 0)
+		(color 0 0 0 0)
+	)
+	(junction
 		(at 93.98 71.12)
 		(diameter 0)
@@
 	)
 	(junction
-		(at 358.14 104.14)
-		(diameter 0)
-		(color 0 0 0 0)
-	)
-	(junction
 		(at 78.74 60.96)
 		(diameter 0)
@@
 	(wire
 		(pts
-			(xy 358.14 82.55) (xy 358.14 104.14)
-		)
-		(stroke
-			(width 0)
-			(type default)
-		)
-	)
-	(wire
-		(pts
 			(xy 322.58 92.71) (xy 347.98 92.71)
 		)
@@
 	(wire
 		(pts
+			(xy 358.14 104.14) (xy 358.14 125.73)
+		)
+		(stroke
+			(width 0)
+			(type default)
+		)
+	)
+	(wire
+		(pts
 			(xy 154.94 82.55) (xy 154.94 104.14)
 		)
@@
 	(wire
 		(pts
-			(xy 383.54 82.55) (xy 383.54 104.14)
+			(xy 383.54 60.96) (xy 383.54 82.55)
 		)
 		(stroke
@@
 	(wire
 		(pts
-			(xy 383.54 60.96) (xy 383.54 82.55)
-		)
-		(stroke
-			(width 0)
-			(type default)
-		)
-	)
-	(wire
-		(pts
 			(xy 220.98 113.03) (xy 220.98 114.3)
 		)
@@
 	(wire
 		(pts
+			(xy 358.14 82.55) (xy 358.14 104.14)
+		)
+		(stroke
+			(width 0)
+			(type default)
+		)
+	)
+	(wire
+		(pts
 			(xy 93.98 125.73) (xy 93.98 127)
 		)
@@
 	(wire
 		(pts
-			(xy 119.38 104.14) (xy 119.38 105.41)
+			(xy 383.54 82.55) (xy 383.54 104.14)
 		)
 		(stroke
@@
 	(wire
 		(pts
-			(xy 154.94 52.07) (xy 154.94 60.96)
+			(xy 119.38 104.14) (xy 119.38 105.41)
 		)
 		(stroke
@@
 	(wire
 		(pts
-			(xy 68.58 71.12) (xy 93.98 71.12)
+			(xy 154.94 52.07) (xy 154.94 60.96)
 		)
 		(stroke
@@
 	(wire
 		(pts
-			(xy 195.58 157.48) (xy 297.18 157.48)
+			(xy 68.58 71.12) (xy 93.98 71.12)
 		)
 		(stroke
@@
 	(wire
 		(pts
-			(xy 297.18 82.55) (xy 297.18 83.82)
+			(xy 195.58 157.48) (xy 297.18 157.48)
 		)
 		(stroke
@@
 	(wire
 		(pts
-			(xy 93.98 156.21) (xy 93.98 157.48)
+			(xy 297.18 82.55) (xy 297.18 83.82)
 		)
 		(stroke
@@
 	(wire
 		(pts
-			(xy 256.54 52.07) (xy 256.54 60.96)
+			(xy 93.98 156.21) (xy 93.98 157.48)
 		)
 		(stroke
@@
 	(wire
 		(pts
-			(xy 170.18 71.12) (xy 195.58 71.12)
+			(xy 256.54 52.07) (xy 256.54 60.96)
 		)
 		(stroke
@@
 	(wire
 		(pts
-			(xy 358.14 104.14) (xy 358.14 125.73)
+			(xy 170.18 71.12) (xy 195.58 71.12)
 		)
 		(stroke
@@
 		(lib_id "Switch:SW_Push")
 		(at 378.46 82.55 0)
-		(mirror x)
 		(unit 1)
 		(exclude_from_sim no)
@@
 		(fields_autoplaced yes)
 		(property "Reference" "S28"
-			(at 378.46 77.47 0)
+			(at 378.46 74.93 0)
 			(effects
 				(font
@@
 		)
 		(property "Value" "MX1A"
-			(at 378.46 80.01 0)
+			(at 378.46 77.47 0)
 			(effects
 				(font
@@
 		)
 		(property "Footprint" "PCM_Switch_Keyboard_Hotswap_Kailh:SW_Hotswap_Kailh_MX_Plated_1.50u_90deg"
-			(at 378.46 87.63 0)
+			(at 378.46 77.47 0)
 			(effects
 				(font
@@
 		)
 		(property "Datasheet" "~"
-			(at 378.46 87.63 0)
+			(at 378.46 77.47 0)
 			(effects
 				(font
@@
 			)
 		)
-		(property "Footprint" "PCM_Switch_Keyboard_Hotswap_Kailh:SW_Hotswap_Kailh_MX_Plated_1.75u_90deg"
+		(property "Footprint" "PCM_Switch_Keyboard_Hotswap_Kailh:SW_Hotswap_Kailh_MX_Plated_2.75u_90deg"
 			(at 353.06 130.81 0)
 			(effects
@@
 		(lib_id "Switch:SW_Push")
 		(at 353.06 104.14 0)
-		(mirror x)
 		(unit 1)
 		(exclude_from_sim no)
@@
 		(fields_autoplaced yes)
 		(property "Reference" "S41"
-			(at 353.06 99.06 0)
+			(at 353.06 96.52 0)
 			(effects
 				(font
@@
 		)
 		(property "Value" "MX1A"
-			(at 353.06 101.6 0)
+			(at 353.06 99.06 0)
 			(effects
 				(font
@@
 		)
 		(property "Footprint" "PCM_Switch_Keyboard_Hotswap_Kailh:SW_Hotswap_Kailh_MX_Plated_2.25u_90deg"
-			(at 353.06 109.22 0)
+			(at 353.06 99.06 0)
 			(effects
 				(font
@@
 		)
 		(property "Datasheet" "~"
-			(at 353.06 109.22 0)
+			(at 353.06 99.06 0)
 			(effects
 				(font
@@
 			)
 		)
-		(property "Footprint" "PCM_Switch_Keyboard_Hotswap_Kailh:SW_Hotswap_Kailh_MX_Plated_2.75u_90deg"
+		(property "Footprint" "PCM_Switch_Keyboard_Hotswap_Kailh:SW_Hotswap_Kailh_MX_Plated_1.00u"
 			(at 378.46 130.81 0)
 			(effects
