File: PCB_Rev2/Multi/matrix.kicad_sch (KiCad schematic)
At the start: 141 parts

Commit message: Wiring Improvement
Parts:
- renumbered S62-2 to S61-2, S63-2 to S62-2
Connections:
- net col_10: now also S61-2.2
- net col_11: now also S62-2.2; no longer S61-2.2
- net col_12: no longer S62-2.2
- net at D60.2 (A), S60.2: now also S62-2.1; no longer S61-2.1
- net at D61.2 (A), S61.2: no longer S62-2.1
- net at D59.2 (A), S59.1: now also S61-2.1
Other:
- moved on the sheet: S61-2, S62-2
Changed lines of the file:
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@@
 	(paper "A3")
 	(junction
-		(at 322.58 148.59)
+		(at 322.58 157.48)
 		(diameter 0)
 		(color 0 0 0 0)
 	)
 	(junction
-		(at 322.58 157.48)
+		(at 358.14 124.46)
 		(diameter 0)
 		(color 0 0 0 0)
 	)
 	(junction
-		(at 358.14 124.46)
+		(at 68.58 148.59)
 		(diameter 0)
 		(color 0 0 0 0)
 	)
 	(junction
-		(at 68.58 148.59)
+		(at 322.58 147.32)
 		(diameter 0)
 		(color 0 0 0 0)
@@
 	)
 	(junction
+		(at 332.74 147.32)
+		(diameter 0)
+		(color 0 0 0 0)
+	)
+	(junction
 		(at 180.34 60.96)
 		(diameter 0)
@@
 	)
 	(junction
-		(at 358.14 147.32)
-		(diameter 0)
-		(color 0 0 0 0)
-	)
-	(junction
 		(at 104.14 125.73)
 		(diameter 0)
@@
 	)
 	(junction
-		(at 347.98 148.59)
-		(diameter 0)
-		(color 0 0 0 0)
-	)
-	(junction
 		(at 281.94 104.14)
 		(diameter 0)
@@
 	)
 	(junction
+		(at 307.34 147.32)
+		(diameter 0)
+		(color 0 0 0 0)
+	)
+	(junction
 		(at 271.78 71.12)
 		(diameter 0)
@@
 	)
 	(junction
-		(at 332.74 147.32)
-		(diameter 0)
-		(color 0 0 0 0)
-	)
-	(junction
 		(at 68.58 92.71)
 		(diameter 0)
@@
 	)
 	(junction
+		(at 297.18 147.32)
+		(diameter 0)
+		(color 0 0 0 0)
+	)
+	(junction
 		(at 93.98 71.12)
 		(diameter 0)
@@
 	(wire
 		(pts
+			(xy 306.07 165.1) (xy 307.34 165.1)
+		)
+		(stroke
+			(width 0)
+			(type default)
+		)
+	)
+	(wire
+		(pts
 			(xy 154.94 60.96) (xy 154.94 82.55)
 		)
@@
 	(wire
 		(pts
-			(xy 358.14 147.32) (xy 358.14 165.1)
+			(xy 78.74 147.32) (xy 78.74 165.1)
 		)
 		(stroke
@@
 	(wire
 		(pts
-			(xy 78.74 147.32) (xy 78.74 165.1)
+			(xy 53.34 124.46) (xy 53.34 125.73)
 		)
 		(stroke
@@
 	(wire
 		(pts
-			(xy 53.34 124.46) (xy 53.34 125.73)
+			(xy 297.18 69.85) (xy 297.18 71.12)
 		)
 		(stroke
@@
 	(wire
 		(pts
-			(xy 297.18 69.85) (xy 297.18 71.12)
+			(xy 195.58 147.32) (xy 195.58 148.59)
 		)
 		(stroke
@@
 	(wire
 		(pts
-			(xy 195.58 147.32) (xy 195.58 148.59)
+			(xy 321.31 147.32) (xy 322.58 147.32)
 		)
 		(stroke
@@
 	(wire
 		(pts
-			(xy 346.71 165.1) (xy 346.71 148.59)
-		)
-		(stroke
-			(width 0)
-			(type default)
-		)
-	)
-	(wire
-		(pts
 			(xy 195.58 134.62) (xy 195.58 135.89)
 		)
@@
 	(wire
 		(pts
+			(xy 321.31 165.1) (xy 321.31 147.32)
+		)
+		(stroke
+			(width 0)
+			(type default)
+		)
+	)
+	(wire
+		(pts
 			(xy 246.38 69.85) (xy 246.38 71.12)
 		)
@@
 	(wire
 		(pts
-			(xy 331.47 165.1) (xy 332.74 165.1)
+			(xy 322.58 156.21) (xy 322.58 157.48)
 		)
 		(stroke
@@
 	(wire
 		(pts
-			(xy 322.58 156.21) (xy 322.58 157.48)
+			(xy 204.47 165.1) (xy 205.74 165.1)
 		)
 		(stroke
@@
 	(wire
 		(pts
-			(xy 204.47 165.1) (xy 205.74 165.1)
+			(xy 144.78 104.14) (xy 144.78 105.41)
 		)
 		(stroke
@@
 	(wire
 		(pts
-			(xy 144.78 104.14) (xy 144.78 105.41)
+			(xy 297.18 147.32) (xy 295.91 147.32)
 		)
 		(stroke
@@
 	(wire
 		(pts
+			(xy 295.91 147.32) (xy 295.91 165.1)
+		)
+		(stroke
+			(width 0)
+			(type default)
+		)
+	)
+	(wire
+		(pts
 			(xy 271.78 113.03) (xy 271.78 114.3)
 		)
@@
 	(wire
 		(pts
+			(xy 332.74 165.1) (xy 331.47 165.1)
+		)
+		(stroke
+			(width 0)
+			(type default)
+		)
+	)
+	(wire
+		(pts
 			(xy 372.11 165.1) (xy 372.11 148.59)
 		)
@@
 	(wire
 		(pts
-			(xy 346.71 148.59) (xy 347.98 148.59)
-		)
-		(stroke
-			(width 0)
-			(type default)
-		)
-	)
-	(wire
-		(pts
 			(xy 384.81 81.28) (xy 373.38 81.28)
 		)
@@
 	(wire
 		(pts
-			(xy 332.74 147.32) (xy 332.74 165.1)
-		)
-		(stroke
-			(width 0)
-			(type default)
-		)
-	)
-	(wire
-		(pts
 			(xy 281.94 60.96) (xy 281.94 82.55)
 		)
@@
 	(wire
 		(pts
+			(xy 307.34 147.32) (xy 307.34 165.1)
+		)
+		(stroke
+			(width 0)
+			(type default)
+		)
+	)
+	(wire
+		(pts
 			(xy 180.34 60.96) (xy 180.34 82.55)
 		)
@@
 	(wire
 		(pts
-			(xy 321.31 148.59) (xy 322.58 148.59)
-		)
-		(stroke
-			(width 0)
-			(type default)
-		)
-	)
-	(wire
-		(pts
 			(xy 170.18 91.44) (xy 170.18 92.71)
 		)
@@
 	(wire
 		(pts
+			(xy 332.74 147.32) (xy 332.74 165.1)
+		)
+		(stroke
+			(width 0)
+			(type default)
+		)
+	)
+	(wire
+		(pts
 			(xy 31.75 102.87) (xy 31.75 104.14)
 		)
@@
 	(wire
 		(pts
-			(xy 321.31 165.1) (xy 321.31 148.59)
-		)
-		(stroke
-			(width 0)
-			(type default)
-		)
-	)
-	(wire
-		(pts
 			(xy 53.34 125.73) (xy 53.34 147.32)
 		)
@@
 		)
 	)
-	(wire
-		(pts
-			(xy 356.87 165.1) (xy 358.14 165.1)
-		)
-		(stroke
-			(width 0)
-			(type default)
-		)
-	)
 	(global_label "row_0"
 		(shape input)
@@
 	(symbol
 		(lib_id "Switch:SW_Push")
-		(at 326.39 165.1 0)
+		(at 300.99 165.1 0)
 		(mirror x)
 		(unit 1)
@@
 		(dnp no)
 		(fields_autoplaced yes)
-		(property "Reference" "S62-2"
-			(at 326.39 160.02 0)
+		(property "Reference" "S61-2"
+			(at 300.99 160.02 0)
 			(effects
 				(font
@@
 		)
 		(property "Value" "MX1A"
-			(at 326.39 162.56 0)
+			(at 300.99 162.56 0)
 			(effects
 				(font
@@
 		)
 		(property "Footprint" "PCM_Switch_Keyboard_Hotswap_Kailh:SW_Hotswap_Kailh_MX_Plated_1.50u"
-			(at 326.39 170.18 0)
+			(at 300.99 170.18 0)
 			(effects
 				(font
@@
 		)
 		(property "Datasheet" "~"
-			(at 326.39 170.18 0)
+			(at 300.99 170.18 0)
 			(effects
 				(font
@@
 		)
 		(property "Description" "Push button switch, generic, two pins"
-			(at 326.39 165.1 0)
+			(at 300.99 165.1 0)
 			(effects
 				(font
@@
 			(project "PH60_Rev2"
 				(path "/dca0f898-8fdb-4522-a51d-f4f4238906e7/dc5cd3b2-ef82-41de-b720-71645d542746"
-					(reference "S62-2")
+					(reference "S61-2")
 					(unit 1)
 				)
@@
 	(symbol
 		(lib_id "Switch:SW_Push")
-		(at 351.79 165.1 0)
+		(at 326.39 165.1 0)
 		(mirror x)
 		(unit 1)
@@
 		(dnp no)
 		(fields_autoplaced yes)
-		(property "Reference" "S63-2"
-			(at 351.79 160.02 0)
+		(property "Reference" "S62-2"
+			(at 326.39 160.02 0)
 			(effects
 				(font
@@
 		)
 		(property "Value" "MX1A"
-			(at 351.79 162.56 0)
+			(at 326.39 162.56 0)
 			(effects
 				(font
@@
 		)
 		(property "Footprint" "PCM_Switch_Keyboard_Hotswap_Kailh:SW_Hotswap_Kailh_MX_Plated_1.00u"
-			(at 351.79 170.18 0)
+			(at 326.39 170.18 0)
 			(effects
 				(font
@@
 		)
 		(property "Datasheet" "~"
-			(at 351.79 170.18 0)
+			(at 326.39 170.18 0)
 			(effects
 				(font
@@
 		)
 		(property "Description" "Push button switch, generic, two pins"
-			(at 351.79 165.1 0)
+			(at 326.39 165.1 0)
 			(effects
 				(font
@@
 			(project "PH60_Rev2"
 				(path "/dca0f898-8fdb-4522-a51d-f4f4238906e7/dc5cd3b2-ef82-41de-b720-71645d542746"
-					(reference "S63-2")
+					(reference "S62-2")
 					(unit 1)
 				)

Commit message: Wiring Rearrangement
Parts:
- renumbered S41-2 to S28-2, S28-2 to S41-2
Connections:
- net col_12: now also S41-2.2; no longer S28-2.1
- net col_13: now also S28-2.1; no longer S41-2.2
- net at D28.2 (A), S28.1: now also S28-2.2; no longer S41-2.1
- net at D41.2 (A), S41.1: now also S41-2.1; no longer S28-2.2
Other:
- moved on the sheet: S28-2, S41-2
Changed lines of the file:
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@@
 	)
 	(junction
+		(at 347.98 104.14)
+		(diameter 0)
+		(color 0 0 0 0)
+	)
+	(junction
 		(at 322.58 114.3)
 		(diameter 0)
@@
 	)
 	(junction
+		(at 358.14 102.87)
+		(diameter 0)
+		(color 0 0 0 0)
+	)
+	(junction
 		(at 104.14 104.14)
 		(diameter 0)
@@
 	)
 	(junction
+		(at 373.38 82.55)
+		(diameter 0)
+		(color 0 0 0 0)
+	)
+	(junction
 		(at 93.98 92.71)
 		(diameter 0)
@@
 	)
 	(junction
-		(at 358.14 102.87)
-		(diameter 0)
-		(color 0 0 0 0)
-	)
-	(junction
 		(at 154.94 60.96)
 		(diameter 0)
@@
 	)
 	(junction
-		(at 373.38 82.55)
-		(diameter 0)
-		(color 0 0 0 0)
-	)
-	(junction
 		(at 144.78 135.89)
 		(diameter 0)
@@
 	)
 	(junction
-		(at 347.98 104.14)
-		(diameter 0)
-		(color 0 0 0 0)
-	)
-	(junction
 		(at 205.74 82.55)
 		(diameter 0)
@@
 	(wire
 		(pts
-			(xy 358.14 102.87) (xy 394.97 102.87)
-		)
-		(stroke
-			(width 0)
-			(type default)
-		)
-	)
-	(wire
-		(pts
 			(xy 220.98 135.89) (xy 246.38 135.89)
 		)
@@
 	(wire
 		(pts
+			(xy 394.97 101.6) (xy 394.97 102.87)
+		)
+		(stroke
+			(width 0)
+			(type default)
+		)
+	)
+	(wire
+		(pts
 			(xy 104.14 60.96) (xy 104.14 82.55)
 		)
@@
 	(wire
 		(pts
-			(xy 384.81 101.6) (xy 347.98 101.6)
-		)
-		(stroke
-			(width 0)
-			(type default)
-		)
-	)
-	(wire
-		(pts
 			(xy 144.78 125.73) (xy 144.78 127)
 		)
@@
 	(wire
 		(pts
+			(xy 373.38 81.28) (xy 373.38 82.55)
+		)
+		(stroke
+			(width 0)
+			(type default)
+		)
+	)
+	(wire
+		(pts
 			(xy 154.94 82.55) (xy 154.94 104.14)
 		)
@@
 	(wire
 		(pts
-			(xy 347.98 101.6) (xy 347.98 104.14)
-		)
-		(stroke
-			(width 0)
-			(type default)
-		)
-	)
-	(wire
-		(pts
 			(xy 41.91 102.87) (xy 53.34 102.87)
 		)
@@
 	(wire
 		(pts
-			(xy 394.97 101.6) (xy 394.97 102.87)
-		)
-		(stroke
-			(width 0)
-			(type default)
-		)
-	)
-	(wire
-		(pts
 			(xy 321.31 165.1) (xy 321.31 147.32)
 		)
@@
 	(wire
 		(pts
+			(xy 358.14 102.87) (xy 358.14 104.14)
+		)
+		(stroke
+			(width 0)
+			(type default)
+		)
+	)
+	(wire
+		(pts
 			(xy 195.58 60.96) (xy 195.58 62.23)
 		)
@@
 	(wire
 		(pts
+			(xy 394.97 82.55) (xy 383.54 82.55)
+		)
+		(stroke
+			(width 0)
+			(type default)
+		)
+	)
+	(wire
+		(pts
 			(xy 347.98 82.55) (xy 347.98 83.82)
 		)
@@
 	(wire
 		(pts
+			(xy 394.97 81.28) (xy 394.97 82.55)
+		)
+		(stroke
+			(width 0)
+			(type default)
+		)
+	)
+	(wire
+		(pts
 			(xy 373.38 91.44) (xy 373.38 92.71)
 		)
@@
 	(wire
 		(pts
-			(xy 372.11 165.1) (xy 372.11 148.59)
+			(xy 358.14 102.87) (xy 394.97 102.87)
 		)
 		(stroke
@@
 	(wire
 		(pts
-			(xy 347.98 123.19) (xy 347.98 125.73)
+			(xy 372.11 165.1) (xy 372.11 148.59)
 		)
 		(stroke
@@
 	(wire
 		(pts
-			(xy 394.97 81.28) (xy 394.97 82.55)
+			(xy 347.98 123.19) (xy 347.98 125.73)
 		)
 		(stroke
@@
 	(wire
 		(pts
-			(xy 384.81 81.28) (xy 373.38 81.28)
-		)
-		(stroke
-			(width 0)
-			(type default)
-		)
-	)
-	(wire
-		(pts
 			(xy 93.98 157.48) (xy 195.58 157.48)
 		)
@@
 	(wire
 		(pts
+			(xy 347.98 101.6) (xy 347.98 104.14)
+		)
+		(stroke
+			(width 0)
+			(type default)
+		)
+	)
+	(wire
+		(pts
 			(xy 220.98 92.71) (xy 246.38 92.71)
 		)
@@
 	(wire
 		(pts
-			(xy 358.14 102.87) (xy 358.14 104.14)
-		)
-		(stroke
-			(width 0)
-			(type default)
-		)
-	)
-	(wire
-		(pts
 			(xy 195.58 157.48) (xy 297.18 157.48)
 		)
@@
 	(wire
 		(pts
-			(xy 194.31 165.1) (xy 194.31 148.59)
+			(xy 384.81 81.28) (xy 373.38 81.28)
 		)
 		(stroke
@@
 	(wire
 		(pts
-			(xy 31.75 124.46) (xy 31.75 125.73)
+			(xy 194.31 165.1) (xy 194.31 148.59)
 		)
 		(stroke
@@
 	(wire
 		(pts
-			(xy 256.54 104.14) (xy 256.54 125.73)
+			(xy 384.81 101.6) (xy 347.98 101.6)
 		)
 		(stroke
@@
 	(wire
 		(pts
-			(xy 93.98 147.32) (xy 93.98 148.59)
+			(xy 31.75 124.46) (xy 31.75 125.73)
 		)
 		(stroke
@@
 	(wire
 		(pts
-			(xy 104.14 52.07) (xy 104.14 60.96)
+			(xy 256.54 104.14) (xy 256.54 125.73)
 		)
 		(stroke
@@
 	(wire
 		(pts
-			(xy 297.18 147.32) (xy 297.18 148.59)
+			(xy 93.98 147.32) (xy 93.98 148.59)
 		)
 		(stroke
@@
 	(wire
 		(pts
-			(xy 93.98 92.71) (xy 119.38 92.71)
+			(xy 104.14 52.07) (xy 104.14 60.96)
 		)
 		(stroke
@@
 	(wire
 		(pts
-			(xy 347.98 60.96) (xy 347.98 62.23)
+			(xy 297.18 147.32) (xy 297.18 148.59)
 		)
 		(stroke
@@
 	(wire
 		(pts
-			(xy 383.54 82.55) (xy 394.97 82.55)
+			(xy 93.98 92.71) (xy 119.38 92.71)
 		)
 		(stroke
@@
 	(wire
 		(pts
-			(xy 358.14 82.55) (xy 358.14 102.87)
+			(xy 347.98 60.96) (xy 347.98 62.23)
 		)
 		(stroke
@@
 	(wire
 		(pts
-			(xy 373.38 81.28) (xy 373.38 82.55)
+			(xy 358.14 82.55) (xy 358.14 102.87)
 		)
 		(stroke
@@
 	(symbol
 		(lib_id "Switch:SW_Push")
-		(at 389.89 101.6 0)
+		(at 389.89 81.28 0)
 		(mirror y)
 		(unit 1)
@@
 		(dnp no)
 		(fields_autoplaced yes)
-		(property "Reference" "S41-2"
-			(at 389.89 93.98 0)
+		(property "Reference" "S28-2"
+			(at 389.89 73.66 0)
 			(effects
 				(font
@@
 		)
 		(property "Value" "MX1A"
-			(at 389.89 96.52 0)
+			(at 389.89 76.2 0)
 			(effects
 				(font
@@
 		)
 		(property "Footprint" "PCM_Switch_Keyboard_Hotswap_Kailh:SW_Hotswap_Kailh_MX_Plated_1.50u_90deg"
-			(at 389.89 96.52 0)
+			(at 389.89 76.2 0)
 			(effects
 				(font
@@
 		)
 		(property "Datasheet" "~"
-			(at 389.89 96.52 0)
+			(at 389.89 76.2 0)
 			(effects
 				(font
@@
 		)
 		(property "Description" "Push button switch, generic, two pins"
-			(at 389.89 101.6 0)
+			(at 389.89 81.28 0)
 			(effects
 				(font
@@
 			(project "PH60_Rev2"
 				(path "/dca0f898-8fdb-4522-a51d-f4f4238906e7/dc5cd3b2-ef82-41de-b720-71645d542746"
-					(reference "S41-2")
+					(reference "S28-2")
 					(unit 1)
 				)
@@
 	(symbol
 		(lib_id "Switch:SW_Push")
-		(at 389.89 81.28 0)
+		(at 389.89 101.6 0)
 		(mirror x)
 		(unit 1)
@@
 		(dnp no)
 		(fields_autoplaced yes)
-		(property "Reference" "S28-2"
-			(at 389.89 76.2 0)
+		(property "Reference" "S41-2"
+			(at 389.89 96.52 0)
 			(effects
 				(font
@@
 		)
 		(property "Value" "MX1A"
-			(at 389.89 78.74 0)
+			(at 389.89 99.06 0)
 			(effects
 				(font
@@
 		)
 		(property "Footprint" "PCM_Switch_Keyboard_Hotswap_Kailh:SW_Hotswap_Kailh_MX_Plated_2.25u_90deg"
-			(at 389.89 86.36 0)
+			(at 389.89 106.68 0)
 			(effects
 				(font
@@
 		)
 		(property "Datasheet" "~"
-			(at 389.89 86.36 0)
+			(at 389.89 106.68 0)
 			(effects
 				(font
@@
 		)
 		(property "Description" "Push button switch, generic, two pins"
-			(at 389.89 81.28 0)
+			(at 389.89 101.6 0)
 			(effects
 				(font
@@
 			(project "PH60_Rev2"
 				(path "/dca0f898-8fdb-4522-a51d-f4f4238906e7/dc5cd3b2-ef82-41de-b720-71645d542746"
-					(reference "S28-2")
+					(reference "S41-2")
 					(unit 1)
 				)

Commit message: Update PCB Routing
Parts:
- renumbered D42 to D43, D43 to D44, D46 to D47, D47 to D48, D48 to D49, D49 to D50, D50 to D51, D51 to D52, D52 to D53, D55 to D57, D56 to D58, D57 to D59, D58 to D60, D59 to D61, D60 to D62, D61 to D63, D62 to D64, S42 to S43, S43 to S44, S46 to S47, S47 to S48, S48 to S49, S49 to S50, S50 to S51, S51 to S52, S52 to S53, S55 to S57, S56 to S58, S57 to S59, S58 to S60, S59 to S61, S60 to S62, S61 to S63, S62 to S64
Connections:
- net col_12: now also S28-2.1; no longer S41.2
- net col_13: now also S41.2; no longer S28-2.1
- net at D28.2 (A), S28.1: now also S41.1; no longer S28-2.2
- net at D41.2 (A), S41-2.1: now also S28-2.2; no longer S41.1
Other:
- moved on the sheet: S28-2, S41

Commit message: Wiring Fixing
Connections:
- net col_12: now also S28.2; no longer S28-2.1
- net col_13: now also S28-2.1; no longer S28.2
- net at D28.2 (A), S41.1: now also S28-2.2; no longer S28.1
- net at D41.2 (A), S41-2.1: now also S28.1; no longer S28-2.2
Other:
- moved on the sheet: S28, S28-2, S41
Changed lines of the file:
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@@
 	)
 	(junction
-		(at 154.94 104.14)
+		(at 358.14 104.14)
 		(diameter 0)
 		(color 0 0 0 0)
 	)
 	(junction
-		(at 297.18 157.48)
+		(at 154.94 104.14)
 		(diameter 0)
 		(color 0 0 0 0)
 	)
 	(junction
-		(at 104.14 125.73)
+		(at 297.18 157.48)
 		(diameter 0)
 		(color 0 0 0 0)
 	)
 	(junction
-		(at 383.54 147.32)
+		(at 104.14 125.73)
 		(diameter 0)
 		(color 0 0 0 0)
 	)
 	(junction
-		(at 383.54 82.55)
+		(at 383.54 147.32)
 		(diameter 0)
 		(color 0 0 0 0)
@@
 	)
 	(junction
-		(at 373.38 82.55)
-		(diameter 0)
-		(color 0 0 0 0)
-	)
-	(junction
 		(at 93.98 92.71)
 		(diameter 0)
@@
 	)
 	(junction
-		(at 347.98 104.14)
-		(diameter 0)
-		(color 0 0 0 0)
-	)
-	(junction
 		(at 281.94 82.55)
 		(diameter 0)
@@
 	)
 	(junction
-		(at 358.14 104.14)
-		(diameter 0)
-		(color 0 0 0 0)
-	)
-	(junction
 		(at 53.34 102.87)
 		(diameter 0)
@@
 	)
 	(junction
+		(at 347.98 104.14)
+		(diameter 0)
+		(color 0 0 0 0)
+	)
+	(junction
 		(at 220.98 92.71)
 		(diameter 0)
@@
 	)
 	(junction
+		(at 383.54 82.55)
+		(diameter 0)
+		(color 0 0 0 0)
+	)
+	(junction
 		(at 144.78 71.12)
 		(diameter 0)
@@
 	)
 	(junction
+		(at 373.38 82.55)
+		(diameter 0)
+		(color 0 0 0 0)
+	)
+	(junction
 		(at 246.38 92.71)
 		(diameter 0)
@@
 	(wire
 		(pts
+			(xy 373.38 82.55) (xy 373.38 83.82)
+		)
+		(stroke
+			(width 0)
+			(type default)
+		)
+	)
+	(wire
+		(pts
 			(xy 231.14 52.07) (xy 231.14 60.96)
 		)
@@
 	(wire
 		(pts
-			(xy 373.38 82.55) (xy 373.38 83.82)
+			(xy 347.98 69.85) (xy 347.98 71.12)
 		)
 		(stroke
@@
 	(wire
 		(pts
-			(xy 347.98 69.85) (xy 347.98 71.12)
+			(xy 383.54 82.55) (xy 383.54 104.14)
 		)
 		(stroke
@@
 	(wire
 		(pts
-			(xy 373.38 81.28) (xy 373.38 82.55)
-		)
-		(stroke
-			(width 0)
-			(type default)
-		)
-	)
-	(wire
-		(pts
 			(xy 154.94 82.55) (xy 154.94 104.14)
 		)
@@
 	(wire
 		(pts
+			(xy 358.14 104.14) (xy 358.14 124.46)
+		)
+		(stroke
+			(width 0)
+			(type default)
+		)
+	)
+	(wire
+		(pts
 			(xy 307.34 52.07) (xy 307.34 60.96)
 		)
@@
 	(wire
 		(pts
-			(xy 358.14 104.14) (xy 358.14 124.46)
+			(xy 358.14 102.87) (xy 358.14 104.14)
 		)
 		(stroke
@@
 	(wire
 		(pts
+			(xy 394.97 82.55) (xy 383.54 82.55)
+		)
+		(stroke
+			(width 0)
+			(type default)
+		)
+	)
+	(wire
+		(pts
 			(xy 41.91 102.87) (xy 53.34 102.87)
 		)
@@
 	(wire
 		(pts
-			(xy 358.14 102.87) (xy 358.14 104.14)
-		)
-		(stroke
-			(width 0)
-			(type default)
-		)
-	)
-	(wire
-		(pts
 			(xy 195.58 60.96) (xy 195.58 62.23)
 		)
@@
 	(wire
 		(pts
-			(xy 394.97 82.55) (xy 383.54 82.55)
-		)
-		(stroke
-			(width 0)
-			(type default)
-		)
-	)
-	(wire
-		(pts
 			(xy 347.98 82.55) (xy 347.98 83.82)
 		)
@@
 	(wire
 		(pts
-			(xy 394.97 81.28) (xy 394.97 82.55)
-		)
-		(stroke
-			(width 0)
-			(type default)
-		)
-	)
-	(wire
-		(pts
 			(xy 358.14 102.87) (xy 394.97 102.87)
 		)
@@
 	(wire
 		(pts
-			(xy 347.98 104.14) (xy 347.98 105.41)
-		)
-		(stroke
-			(width 0)
-			(type default)
-		)
-	)
-	(wire
-		(pts
 			(xy 195.58 91.44) (xy 195.58 92.71)
 		)
@@
 	(wire
 		(pts
-			(xy 383.54 60.96) (xy 383.54 82.55)
-		)
-		(stroke
-			(width 0)
-			(type default)
-		)
-	)
-	(wire
-		(pts
 			(xy 220.98 113.03) (xy 220.98 114.3)
 		)
@@
 	(wire
 		(pts
+			(xy 373.38 81.28) (xy 373.38 82.55)
+		)
+		(stroke
+			(width 0)
+			(type default)
+		)
+	)
+	(wire
+		(pts
 			(xy 43.18 134.62) (xy 43.18 135.89)
 		)
@@
 	(wire
 		(pts
+			(xy 394.97 81.28) (xy 394.97 82.55)
+		)
+		(stroke
+			(width 0)
+			(type default)
+		)
+	)
+	(wire
+		(pts
 			(xy 256.54 60.96) (xy 256.54 82.55)
 		)
@@
 	(wire
 		(pts
+			(xy 384.81 81.28) (xy 373.38 81.28)
+		)
+		(stroke
+			(width 0)
+			(type default)
+		)
+	)
+	(wire
+		(pts
 			(xy 373.38 104.14) (xy 373.38 105.41)
 		)
@@
 	(wire
 		(pts
+			(xy 347.98 104.14) (xy 347.98 105.41)
+		)
+		(stroke
+			(width 0)
+			(type default)
+		)
+	)
+	(wire
+		(pts
 			(xy 93.98 114.3) (xy 119.38 114.3)
 		)
@@
 	(wire
 		(pts
-			(xy 373.38 81.28) (xy 384.81 81.28)
-		)
-		(stroke
-			(width 0)
-			(type default)
-		)
-	)
-	(wire
-		(pts
 			(xy 297.18 147.32) (xy 297.18 148.59)
 		)
@@
 	(wire
 		(pts
-			(xy 383.54 82.55) (xy 383.54 104.14)
+			(xy 271.78 104.14) (xy 271.78 105.41)
 		)
 		(stroke
@@
 	(wire
 		(pts
-			(xy 271.78 104.14) (xy 271.78 105.41)
+			(xy 53.34 104.14) (xy 53.34 124.46)
 		)
 		(stroke
@@
 	(wire
 		(pts
-			(xy 53.34 104.14) (xy 53.34 124.46)
+			(xy 383.54 60.96) (xy 383.54 82.55)
 		)
 		(stroke
@@
 	(symbol
 		(lib_id "Switch:SW_Push")
-		(at 378.46 82.55 0)
+		(at 353.06 104.14 0)
 		(mirror x)
 		(unit 1)
@@
 		(fields_autoplaced yes)
 		(property "Reference" "S28"
-			(at 378.46 77.47 0)
+			(at 353.06 99.06 0)
 			(effects
 				(font
@@
 		)
 		(property "Value" "MX1A"
-			(at 378.46 80.01 0)
+			(at 353.06 101.6 0)
 			(effects
 				(font
@@
 		)
 		(property "Footprint" "PCM_Switch_Keyboard_Hotswap_Kailh:SW_Hotswap_Kailh_MX_Plated_ISOEnter_90deg"
-			(at 378.46 87.63 0)
+			(at 353.06 109.22 0)
 			(effects
 				(font
@@
 		)
 		(property "Datasheet" "~"
-			(at 378.46 87.63 0)
+			(at 353.06 109.22 0)
 			(effects
 				(font
@@
 		)
 		(property "Description" "Push button switch, generic, two pins"
-			(at 378.46 82.55 0)
+			(at 353.06 104.14 0)
 			(effects
 				(font
@@
 	(symbol
 		(lib_id "Switch:SW_Push")
-		(at 353.06 104.14 0)
+		(at 389.89 81.28 0)
 		(mirror y)
 		(unit 1)
@@
 		(fields_autoplaced yes)
 		(property "Reference" "S28-2"
-			(at 353.06 96.52 0)
+			(at 389.89 73.66 0)
 			(effects
 				(font
@@
 		)
 		(property "Value" "MX1A"
-			(at 353.06 99.06 0)
+			(at 389.89 76.2 0)
 			(effects
 				(font
@@
 		)
 		(property "Footprint" "PCM_Switch_Keyboard_Hotswap_Kailh:SW_Hotswap_Kailh_MX_Plated_1.50u_90deg"
-			(at 353.06 99.06 0)
+			(at 389.89 76.2 0)
 			(effects
 				(font
@@
 		)
 		(property "Datasheet" "~"
-			(at 353.06 99.06 0)
+			(at 389.89 76.2 0)
 			(effects
 				(font
@@
 		)
 		(property "Description" "Push button switch, generic, two pins"
-			(at 353.06 104.14 0)
+			(at 389.89 81.28 0)
 			(effects
 				(font
@@
 	(symbol
 		(lib_id "Switch:SW_Push")
-		(at 389.89 81.28 0)
+		(at 378.46 82.55 0)
 		(mirror x)
 		(unit 1)
@@
 		(fields_autoplaced yes)
 		(property "Reference" "S41"
-			(at 389.89 76.2 0)
+			(at 378.46 77.47 0)
 			(effects
 				(font
@@
 		)
 		(property "Value" "MX1A"
-			(at 389.89 78.74 0)
+			(at 378.46 80.01 0)
 			(effects
 				(font
@@
 		)
 		(property "Footprint" "PCM_Switch_Keyboard_Hotswap_Kailh:SW_Hotswap_Kailh_MX_Plated_1.00u"
-			(at 389.89 86.36 0)
+			(at 378.46 87.63 0)
 			(effects
 				(font
@@
 		)
 		(property "Datasheet" "~"
-			(at 389.89 86.36 0)
+			(at 378.46 87.63 0)
 			(effects
 				(font
@@
 		)
 		(property "Description" "Push button switch, generic, two pins"
-			(at 389.89 81.28 0)
+			(at 378.46 82.55 0)
 			(effects
 				(font
