File: PCB_Rev2/Slim/PH60_Rev2.kicad_pcb (KiCad board)
At the start: 2 copper layers, 285 x 94.6 mm, 212 parts, among them J1 USB_C_Receptacle_USB2.0_16P, J2 Conn_01x02, U2 W25Q128JVS, U3 RP2040, U4 XC6206PxxxMR, Y1 Crystal_GND24

Commit message: Route RGB light.
Parts:
- moved D65 11.6 mm to (50.6, 66.5)
- moved R6 0.97 mm to (37.3, 68.0), turned to 0 degrees
- moved R7 0.95 mm to (37.4, 65.4), turned to 0 degrees
- turned D57 to 90 degrees
- turned D58 to 90 degrees
- turned D59 to 90 degrees
- turned D62 to 90 degrees
- turned D63 to 90 degrees
- turned D64 to 90 degrees
Routing:
- net VBUS: track 137.5 -> 1129.4 mm, vias 3 -> 54
- net row_0: track 0.00 -> 325.9 mm
- net row_1: track 0.00 -> 325.1 mm
- net row_2: track 0.00 -> 304.8 mm
- net row_3: track 0.00 -> 286.9 mm
- net row_4: track 0.00 -> 265.2 mm
- net GND: track 70.2 -> 86.5 mm, vias 80 -> 82
- net Net-(D64-A): track 0.00 -> 7.29 mm
- net Net-(D62-A): track 0.00 -> 7.29 mm
- net Net-(D54-A): track 0.00 -> 7.29 mm
- net Net-(D28-A): track 0.00 -> 7.29 mm
- net Net-(D11-A): track 0.00 -> 7.29 mm
- net Net-(D61-A): track 0.00 -> 7.29 mm
- net Net-(D50-A): track 0.00 -> 7.29 mm
- net Net-(D38-A): track 0.00 -> 7.29 mm
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
Commit message: [WIP] Route all lights
Parts:
- moved R7 0.35 mm to (37.7, 65.5)
Routing:
- net row_0: track 325.9 -> 599.1 mm, vias 0 -> 2
- net row_1: track 325.1 -> 578.4 mm, vias 0 -> 2
- net row_2: track 304.8 -> 518.6 mm
- net row_3: track 286.9 -> 405.1 mm, vias 0 -> 2
- net VBUS: track 1129.4 -> 1207.2 mm, vias 54 -> 58
- net Net-(RGB57-DOUT): track 0.00 -> 69.4 mm
- net Net-(RGB56-DOUT): track 0.00 -> 68.7 mm, vias 0 -> 2
- net Net-(RGB14-DOUT): track 0.00 -> 37.4 mm
- net Net-(RGB53-DOUT): track 0.00 -> 37.1 mm
- net Net-(RGB42-DOUT): track 0.00 -> 33.2 mm
- net row_4: track 265.2 -> 298.3 mm
- net Net-(RGB41-DOUT): track 0.00 -> 32.0 mm, vias 0 -> 2
- net Net-(RGB40-DOUT): track 0.00 -> 28.5 mm
- net Net-(RGB52-DOUT): track 0.00 -> 28.2 mm
- net Net-(RGB28-DOUT): track 0.00 -> 27.4 mm, vias 0 -> 2
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
Commit message: Almost route done.
Routing:
- net VBUS: track 1207.2 -> 1430.2 mm, vias 58 -> 66
- net GND: track 89.3 -> 92.3 mm
- net row_1: track 578.4 -> 577.4 mm
- net row_2: track 518.6 -> 518.0 mm
- net col_3: track 114.4 -> 115.0 mm
