File: PCB_Rev2/Slim/PH60_Rev2.kicad_pcb (KiCad board)
At the start: 2 copper layers, 285 x 94.6 mm, 212 parts, among them J1 USB_C_Receptacle_USB2.0_16P, J2 Conn_01x02, U2 W25Q128JVS, U3 RP2040, U4 XC6206PxxxMR, Y1 Crystal_GND24

Commit message: Change RGB footprint
Parts:
- RGB1, RGB10, RGB11, RGB12, RGB13, RGB14, RGB15, RGB16, RGB17, RGB18, RGB19, RGB2, RGB20, RGB21, RGB22, RGB23, RGB24, RGB25, RGB26, RGB27, RGB28, RGB29, RGB3, RGB30, RGB31, RGB32, RGB33, RGB34, RGB35, RGB36, RGB37, RGB38, RGB39, RGB4, RGB40, RGB41, RGB42, RGB43, RGB44, RGB45, RGB46, RGB47, RGB48, RGB49, RGB5, RGB50, RGB51, RGB52, RGB53, RGB54, RGB55, RGB56, RGB57, RGB58, RGB59, RGB6, RGB60, RGB61, RGB7, RGB8, RGB9: footprint RGB:ws2812B_6028 -> RGB:ws2812B_6028_FIX
Routing:
- net GND: vias 82 -> 88

Commit message: Add mounting hole.
Parts:
- added F1: 500ma, Fuse:Fuse_0402_1005Metric, B.Cu at (43.0, 64.9)
- added H1: MountingHole, MountingHole:MountingHole_2.2mm_M2, F.Cu at (54.8, 57.1)
- added H2: MountingHole, MountingHole:MountingHole_2.2mm_M2, F.Cu at (52.4, 114.3)
- added H3: MountingHole, MountingHole:MountingHole_2.2mm_M2, F.Cu at (171.4, 57.1)
- added H4: MountingHole, MountingHole:MountingHole_2.2mm_M2, F.Cu at (166.7, 95.2)
- added H5: MountingHole, MountingHole:MountingHole_2.2mm_M2, F.Cu at (288.1, 57.1)
- added H6: MountingHole, MountingHole:MountingHole_2.2mm_M2, F.Cu at (290.5, 114.3)
- moved C12 0.63 mm to (136.9, 118.9), turned to -90 degrees
Connections:
- J1 pad A4: VBUS -> Net-(F1-Pad1)
- J1 pad A9: VBUS -> Net-(F1-Pad1)
- J1 pad B4: VBUS -> Net-(F1-Pad1)
- J1 pad B9: VBUS -> Net-(F1-Pad1)
- RGB1 pad 4: DIN -> RGB_IN
- U3 pad 32: DIN -> unconnected-(U3-GPIO21-Pad32)
- U3 pad 34: unconnected-(U3-GPIO22-Pad34) -> RGB_IN
Routing:
- net RGB_IN: track 0.00 -> 171.8 mm, vias 0 -> 2
- net col_6: track 100.8 -> 128.0 mm, vias 1 -> 2
- net Net-(F1-Pad1): track 0.00 -> 14.4 mm
- net VBUS: track 1430.2 -> 1418.9 mm
- net row_0: track 599.2 -> 598.3 mm
- net row_1: track 577.4 -> 576.7 mm
- net row_2: track 518.0 -> 517.3 mm
- net row_3: track 405.1 -> 404.6 mm
- net GND: track 92.3 -> 92.2 mm, vias 88 -> 156
