File: PCB_Rev2/Slim/PH60_Rev2.kicad_pcb (KiCad board)
At the start: 2 copper layers, 285 x 94.6 mm, 219 parts, among them J1 USB_C_Receptacle_USB2.0_16P, J2 Conn_01x02, U2 W25Q128JVS, U3 RP2040, U4 XC6206PxxxMR, Y1 Crystal_GND24

Commit message: Hole Update.
Parts:
- R3, R4: value 27.4 -> 1R
- moved J2 6.22 mm to (124.0, 113.0), turned to -90 degrees
- moved C4 3.34 mm to (122.9, 106.5)
- moved C1 2.91 mm to (120.2, 109.5)
- moved U4 2.39 mm to (120.1, 107.1)
- moved C5 0.72 mm to (125.5, 108.8), turned to 90 degrees
Routing:
- net GND: track 83.0 -> 68.9 mm, vias 156 -> 165
- net Net-(RGB53-DOUT): track 43.4 -> 57.0 mm
- net col_12: track 313.5 -> 302.9 mm
- net VBUS: track 1487.4 -> 1477.3 mm, vias 67 -> 65
- net /~{USB_BOOT}: track 1.74 -> 9.60 mm
- net row_4: track 333.5 -> 330.4 mm
- net row_3: track 421.6 -> 423.9 mm
- net Net-(RGB52-DOUT): track 51.5 -> 53.3 mm
- net +3V3: track 65.8 -> 67.4 mm, vias 4 -> 5
- net /USB_D+: track 131.5 -> 130.4 mm
- net col_13: track 254.7 -> 255.7 mm
- net row_0: track 614.0 -> 615.0 mm
- net /USB_D-: track 131.8 -> 130.9 mm
- net Net-(RGB40-DOUT): track 32.6 -> 33.5 mm
- net RGB_IN: track 175.2 -> 176.0 mm
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Other:
- outline, holes or cut-outs redrawn
