File: PCB_Rev2/Slim/RGB.kicad_sch (KiCad schematic)
At the start: 61 parts

Commit message: Change RGB footprint
Parts:
- RGB1, RGB10, RGB11, RGB12, RGB13, RGB14, RGB15, RGB16, RGB17, RGB18, RGB19, RGB2, RGB20, RGB21, RGB22, RGB23, RGB24, RGB25, RGB26, RGB27, RGB28, RGB29, RGB3, RGB30, RGB31, RGB32, RGB33, RGB34, RGB35, RGB36, RGB37, RGB38, RGB39, RGB4, RGB40, RGB41, RGB42, RGB43, RGB44, RGB45, RGB46, RGB47, RGB48, RGB49, RGB5, RGB50, RGB51, RGB52, RGB53, RGB54, RGB55, RGB56, RGB57, RGB58, RGB59, RGB6, RGB60, RGB61, RGB7, RGB8, RGB9: footprint RGB:ws2812B_6028 -> RGB:SK6812-MINI-E
Changed lines of the file:
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@@
 			)
 		)
-		(property "Footprint" "RGB:ws2812B_6028"
+		(property "Footprint" "RGB:SK6812-MINI-E"
 			(at 128.27 77.47 0)
 			(effects
@@
 			)
 		)
-		(property "Footprint" "RGB:ws2812B_6028"
+		(property "Footprint" "RGB:SK6812-MINI-E"
 			(at 62.23 120.65 0)
 			(effects
@@
 			)
 		)
-		(property "Footprint" "RGB:ws2812B_6028"
+		(property "Footprint" "RGB:SK6812-MINI-E"
 			(at 196.85 133.35 0)
 			(effects
@@
 			)
 		)
-		(property "Footprint" "RGB:ws2812B_6028"
+		(property "Footprint" "RGB:SK6812-MINI-E"
 			(at 153.67 64.77 0)
 			(effects
@@
 			)
 		)
-		(property "Footprint" "RGB:ws2812B_6028"
+		(property "Footprint" "RGB:SK6812-MINI-E"
 			(at 290.83 64.77 0)
 			(effects
@@
 			)
 		)
-		(property "Footprint" "RGB:ws2812B_6028"
+		(property "Footprint" "RGB:SK6812-MINI-E"
 			(at 265.43 77.47 0)
 			(effects
@@
 			)
 		)
-		(property "Footprint" "RGB:ws2812B_6028"
+		(property "Footprint" "RGB:SK6812-MINI-E"
 			(at 219.71 77.47 0)
 			(effects
@@
 			)
 		)
-		(property "Footprint" "RGB:ws2812B_6028"
+		(property "Footprint" "RGB:SK6812-MINI-E"
 			(at 267.97 120.65 0)
 			(effects
@@
 			)
 		)
-		(property "Footprint" "RGB:ws2812B_6028"
+		(property "Footprint" "RGB:SK6812-MINI-E"
 			(at 288.29 77.47 0)
 			(effects
@@
 			)
 		)
-		(property "Footprint" "RGB:ws2812B_6028"
+		(property "Footprint" "RGB:SK6812-MINI-E"
 			(at 199.39 64.77 0)
 			(effects
@@
 			)
 		)
-		(property "Footprint" "RGB:ws2812B_6028"
+		(property "Footprint" "RGB:SK6812-MINI-E"
 			(at 176.53 64.77 0)
 			(effects
@@
 			)
 		)
-		(property "Footprint" "RGB:ws2812B_6028"
+		(property "Footprint" "RGB:SK6812-MINI-E"
 			(at 130.81 120.65 0)
 			(effects
@@
 			)
 		)
-		(property "Footprint" "RGB:ws2812B_6028"
+		(property "Footprint" "RGB:SK6812-MINI-E"
 			(at 313.69 64.77 0)
 			(effects
@@
 			)
 		)
-		(property "Footprint" "RGB:ws2812B_6028"
+		(property "Footprint" "RGB:SK6812-MINI-E"
 			(at 356.87 133.35 0)
 			(effects
@@
 			)
 		)
-		(property "Footprint" "RGB:ws2812B_6028"
+		(property "Footprint" "RGB:SK6812-MINI-E"
 			(at 151.13 133.35 0)
 			(effects
@@
 			)
 		)
-		(property "Footprint" "RGB:ws2812B_6028"
+		(property "Footprint" "RGB:SK6812-MINI-E"
 			(at 128.27 133.35 0)
 			(effects
@@
 			)
 		)
-		(property "Footprint" "RGB:ws2812B_6028"
+		(property "Footprint" "RGB:SK6812-MINI-E"
 			(at 288.29 133.35 0)
 			(effects
@@
 			)
 		)
-		(property "Footprint" "RGB:ws2812B_6028"
+		(property "Footprint" "RGB:SK6812-MINI-E"
 			(at 151.13 77.47 0)
 			(effects
@@
 			)
 		)
-		(property "Footprint" "RGB:ws2812B_6028"
+		(property "Footprint" "RGB:SK6812-MINI-E"
 			(at 311.15 133.35 0)
 			(effects
@@
 			)
 		)
-		(property "Footprint" "RGB:ws2812B_6028"
+		(property "Footprint" "RGB:SK6812-MINI-E"
 			(at 356.87 77.47 0)
 			(effects
@@
 			)
 		)
-		(property "Footprint" "RGB:ws2812B_6028"
+		(property "Footprint" "RGB:SK6812-MINI-E"
 			(at 59.69 77.47 0)
 			(effects
@@
 			)
 		)
-		(property "Footprint" "RGB:ws2812B_6028"
+		(property "Footprint" "RGB:SK6812-MINI-E"
 			(at 265.43 133.35 0)
 			(effects
@@
 			)
 		)
-		(property "Footprint" "RGB:ws2812B_6028"
+		(property "Footprint" "RGB:SK6812-MINI-E"
 			(at 242.57 133.35 0)
 			(effects
@@
 			)
 		)
-		(property "Footprint" "RGB:ws2812B_6028"
+		(property "Footprint" "RGB:SK6812-MINI-E"
 			(at 222.25 120.65 0)
 			(effects
@@
 			)
 		)
-		(property "Footprint" "RGB:ws2812B_6028"
+		(property "Footprint" "RGB:SK6812-MINI-E"
 			(at 85.09 64.77 0)
 			(effects
@@
 			)
 		)
-		(property "Footprint" "RGB:ws2812B_6028"
+		(property "Footprint" "RGB:SK6812-MINI-E"
 			(at 379.73 133.35 0)
 			(effects
@@
 			)
 		)
-		(property "Footprint" "RGB:ws2812B_6028"
+		(property "Footprint" "RGB:SK6812-MINI-E"
 			(at 359.41 64.77 0)
 			(effects
@@
 			)
 		)
-		(property "Footprint" "RGB:ws2812B_6028"
+		(property "Footprint" "RGB:SK6812-MINI-E"
 			(at 379.73 77.47 0)
 			(effects
@@
 			)
 		)
-		(property "Footprint" "RGB:ws2812B_6028"
+		(property "Footprint" "RGB:SK6812-MINI-E"
 			(at 39.37 120.65 0)
 			(effects
@@
 			)
 		)
-		(property "Footprint" "RGB:ws2812B_6028"
+		(property "Footprint" "RGB:SK6812-MINI-E"
 			(at 153.67 120.65 0)
 			(effects
@@
 			)
 		)
-		(property "Footprint" "RGB:ws2812B_6028"
+		(property "Footprint" "RGB:SK6812-MINI-E"
 			(at 105.41 133.35 0)
 			(effects
@@
 			)
 		)
-		(property "Footprint" "RGB:ws2812B_6028"
+		(property "Footprint" "RGB:SK6812-MINI-E"
 			(at 85.09 120.65 0)
 			(effects
@@
 			)
 		)
-		(property "Footprint" "RGB:ws2812B_6028"
+		(property "Footprint" "RGB:SK6812-MINI-E"
 			(at 196.85 77.47 0)
 			(effects
@@
 			)
 		)
-		(property "Footprint" "RGB:ws2812B_6028"
+		(property "Footprint" "RGB:SK6812-MINI-E"
 			(at 82.55 77.47 0)
 			(effects
@@
 			)
 		)
-		(property "Footprint" "RGB:ws2812B_6028"
+		(property "Footprint" "RGB:SK6812-MINI-E"
 			(at 334.01 133.35 0)
 			(effects
@@
 			)
 		)
-		(property "Footprint" "RGB:ws2812B_6028"
+		(property "Footprint" "RGB:SK6812-MINI-E"
 			(at 336.55 64.77 0)
 			(effects
@@
 			)
 		)
-		(property "Footprint" "RGB:ws2812B_6028"
+		(property "Footprint" "RGB:SK6812-MINI-E"
 			(at 245.11 64.77 0)
 			(effects
@@
 			)
 		)
-		(property "Footprint" "RGB:ws2812B_6028"
+		(property "Footprint" "RGB:SK6812-MINI-E"
 			(at 39.37 64.77 0)
 			(effects
@@
 			)
 		)
-		(property "Footprint" "RGB:ws2812B_6028"
+		(property "Footprint" "RGB:SK6812-MINI-E"
 			(at 173.99 77.47 0)
 			(effects
@@
 			)
 		)
-		(property "Footprint" "RGB:ws2812B_6028"
+		(property "Footprint" "RGB:SK6812-MINI-E"
 			(at 336.55 120.65 0)
 			(effects
@@
 			)
 		)
-		(property "Footprint" "RGB:ws2812B_6028"
+		(property "Footprint" "RGB:SK6812-MINI-E"
 			(at 107.95 64.77 0)
 			(effects
@@
 			)
 		)
-		(property "Footprint" "RGB:ws2812B_6028"
+		(property "Footprint" "RGB:SK6812-MINI-E"
 			(at 219.71 133.35 0)
 			(effects
@@
 			)
 		)
-		(property "Footprint" "RGB:ws2812B_6028"
+		(property "Footprint" "RGB:SK6812-MINI-E"
 			(at 105.41 77.47 0)
 			(effects
@@
 			)
 		)
-		(property "Footprint" "RGB:ws2812B_6028"
+		(property "Footprint" "RGB:SK6812-MINI-E"
 			(at 176.53 120.65 0)
 			(effects
@@
 			)
 		)
-		(property "Footprint" "RGB:ws2812B_6028"
+		(property "Footprint" "RGB:SK6812-MINI-E"
 			(at 242.57 77.47 0)
 			(effects
@@
 			)
 		)
-		(property "Footprint" "RGB:ws2812B_6028"
+		(property "Footprint" "RGB:SK6812-MINI-E"
 			(at 267.97 64.77 0)
 			(effects
@@
 			)
 		)
-		(property "Footprint" "RGB:ws2812B_6028"
+		(property "Footprint" "RGB:SK6812-MINI-E"
 			(at 359.41 120.65 0)
 			(effects
@@
 			)
 		)
-		(property "Footprint" "RGB:ws2812B_6028"
+		(property "Footprint" "RGB:SK6812-MINI-E"
 			(at 311.15 77.47 0)
 			(effects
@@
 			)
 		)
-		(property "Footprint" "RGB:ws2812B_6028"
+		(property "Footprint" "RGB:SK6812-MINI-E"
 			(at 107.95 120.65 0)
 			(effects
@@
 			)
 		)
-		(property "Footprint" "RGB:ws2812B_6028"
+		(property "Footprint" "RGB:SK6812-MINI-E"
 			(at 313.69 120.65 0)
 			(effects
@@
 			)
 		)
-		(property "Footprint" "RGB:ws2812B_6028"
+		(property "Footprint" "RGB:SK6812-MINI-E"
 			(at 199.39 120.65 0)
 			(effects
@@
 			)
 		)
-		(property "Footprint" "RGB:ws2812B_6028"
+		(property "Footprint" "RGB:SK6812-MINI-E"
 			(at 130.81 64.77 0)
 			(effects
@@
 			)
 		)
-		(property "Footprint" "RGB:ws2812B_6028"
+		(property "Footprint" "RGB:SK6812-MINI-E"
 			(at 222.25 64.77 0)
 			(effects
@@
 			)
 		)
-		(property "Footprint" "RGB:ws2812B_6028"
+		(property "Footprint" "RGB:SK6812-MINI-E"
 			(at 36.83 77.47 0)
 			(effects
@@
 			)
 		)
-		(property "Footprint" "RGB:ws2812B_6028"
+		(property "Footprint" "RGB:SK6812-MINI-E"
 			(at 245.11 120.65 0)
 			(effects
@@
 			)
 		)
-		(property "Footprint" "RGB:ws2812B_6028"
+		(property "Footprint" "RGB:SK6812-MINI-E"
 			(at 382.27 120.65 0)
 			(effects
@@
 			)
 		)
-		(property "Footprint" "RGB:ws2812B_6028"
+		(property "Footprint" "RGB:SK6812-MINI-E"
 			(at 62.23 64.77 0)
 			(effects
@@
 			)
 		)
-		(property "Footprint" "RGB:ws2812B_6028"
+		(property "Footprint" "RGB:SK6812-MINI-E"
 			(at 382.27 64.77 0)
 			(effects
@@
 			)
 		)
-		(property "Footprint" "RGB:ws2812B_6028"
+		(property "Footprint" "RGB:SK6812-MINI-E"
 			(at 290.83 120.65 0)
 			(effects
@@
 			)
 		)
-		(property "Footprint" "RGB:ws2812B_6028"
+		(property "Footprint" "RGB:SK6812-MINI-E"
 			(at 173.99 133.35 0)
 			(effects
@@
 			)
 		)
-		(property "Footprint" "RGB:ws2812B_6028"
+		(property "Footprint" "RGB:SK6812-MINI-E"
 			(at 334.01 77.47 0)
 			(effects

Commit message: Add mounting hole.
Parts:
- RGB1, RGB10, RGB11, RGB12, RGB13, RGB14, RGB15, RGB16, RGB17, RGB18, RGB19, RGB2, RGB20, RGB21, RGB22, RGB23, RGB24, RGB25, RGB26, RGB27, RGB28, RGB29, RGB3, RGB30, RGB31, RGB32, RGB33, RGB34, RGB35, RGB36, RGB37, RGB38, RGB39, RGB4, RGB40, RGB41, RGB42, RGB43, RGB44, RGB45, RGB46, RGB47, RGB48, RGB49, RGB5, RGB50, RGB51, RGB52, RGB53, RGB54, RGB55, RGB56, RGB57, RGB58, RGB59, RGB6, RGB60, RGB61, RGB7, RGB8, RGB9: footprint RGB:SK6812-MINI-E -> RGB:ws2812B_6028_FIX
Connections:
- net DIN renamed RGB_IN
Changed lines of the file:
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@@
 		)
 	)
-	(global_label "DIN"
+	(global_label "RGB_IN"
 		(shape input)
 		(at 30.48 57.15 180)
@@
 		)
 		(property "Intersheetrefs" "${INTERSHEET_REFS}"
-			(at 24.2895 57.15 0)
+			(at 20.7819 57.15 0)
 			(effects
 				(font
@@
 			)
 		)
-		(property "Footprint" "RGB:SK6812-MINI-E"
+		(property "Footprint" "RGB:ws2812B_6028_FIX"
 			(at 128.27 77.47 0)
 			(effects
@@
 			)
 		)
-		(property "Footprint" "RGB:SK6812-MINI-E"
+		(property "Footprint" "RGB:ws2812B_6028_FIX"
 			(at 62.23 120.65 0)
 			(effects
@@
 			)
 		)
-		(property "Footprint" "RGB:SK6812-MINI-E"
+		(property "Footprint" "RGB:ws2812B_6028_FIX"
 			(at 196.85 133.35 0)
 			(effects
@@
 			)
 		)
-		(property "Footprint" "RGB:SK6812-MINI-E"
+		(property "Footprint" "RGB:ws2812B_6028_FIX"
 			(at 153.67 64.77 0)
 			(effects
@@
 			)
 		)
-		(property "Footprint" "RGB:SK6812-MINI-E"
+		(property "Footprint" "RGB:ws2812B_6028_FIX"
 			(at 290.83 64.77 0)
 			(effects
@@
 			)
 		)
-		(property "Footprint" "RGB:SK6812-MINI-E"
+		(property "Footprint" "RGB:ws2812B_6028_FIX"
 			(at 265.43 77.47 0)
 			(effects
@@
 			)
 		)
-		(property "Footprint" "RGB:SK6812-MINI-E"
+		(property "Footprint" "RGB:ws2812B_6028_FIX"
 			(at 219.71 77.47 0)
 			(effects
@@
 			)
 		)
-		(property "Footprint" "RGB:SK6812-MINI-E"
+		(property "Footprint" "RGB:ws2812B_6028_FIX"
 			(at 267.97 120.65 0)
 			(effects
@@
 			)
 		)
-		(property "Footprint" "RGB:SK6812-MINI-E"
+		(property "Footprint" "RGB:ws2812B_6028_FIX"
 			(at 288.29 77.47 0)
 			(effects
@@
 			)
 		)
-		(property "Footprint" "RGB:SK6812-MINI-E"
+		(property "Footprint" "RGB:ws2812B_6028_FIX"
 			(at 199.39 64.77 0)
 			(effects
@@
 			)
 		)
-		(property "Footprint" "RGB:SK6812-MINI-E"
+		(property "Footprint" "RGB:ws2812B_6028_FIX"
 			(at 176.53 64.77 0)
 			(effects
@@
 			)
 		)
-		(property "Footprint" "RGB:SK6812-MINI-E"
+		(property "Footprint" "RGB:ws2812B_6028_FIX"
 			(at 130.81 120.65 0)
 			(effects
@@
 			)
 		)
-		(property "Footprint" "RGB:SK6812-MINI-E"
+		(property "Footprint" "RGB:ws2812B_6028_FIX"
 			(at 313.69 64.77 0)
 			(effects
@@
 			)
 		)
-		(property "Footprint" "RGB:SK6812-MINI-E"
+		(property "Footprint" "RGB:ws2812B_6028_FIX"
 			(at 356.87 133.35 0)
 			(effects
@@
 			)
 		)
-		(property "Footprint" "RGB:SK6812-MINI-E"
+		(property "Footprint" "RGB:ws2812B_6028_FIX"
 			(at 151.13 133.35 0)
 			(effects
@@
 			)
 		)
-		(property "Footprint" "RGB:SK6812-MINI-E"
+		(property "Footprint" "RGB:ws2812B_6028_FIX"
 			(at 128.27 133.35 0)
 			(effects
@@
 			)
 		)
-		(property "Footprint" "RGB:SK6812-MINI-E"
+		(property "Footprint" "RGB:ws2812B_6028_FIX"
 			(at 288.29 133.35 0)
 			(effects
@@
 			)
 		)
-		(property "Footprint" "RGB:SK6812-MINI-E"
+		(property "Footprint" "RGB:ws2812B_6028_FIX"
 			(at 151.13 77.47 0)
 			(effects
@@
 			)
 		)
-		(property "Footprint" "RGB:SK6812-MINI-E"
+		(property "Footprint" "RGB:ws2812B_6028_FIX"
 			(at 311.15 133.35 0)
 			(effects
@@
 			)
 		)
-		(property "Footprint" "RGB:SK6812-MINI-E"
+		(property "Footprint" "RGB:ws2812B_6028_FIX"
 			(at 356.87 77.47 0)
 			(effects
@@
 			)
 		)
-		(property "Footprint" "RGB:SK6812-MINI-E"
+		(property "Footprint" "RGB:ws2812B_6028_FIX"
 			(at 59.69 77.47 0)
 			(effects
@@
 			)
 		)
-		(property "Footprint" "RGB:SK6812-MINI-E"
+		(property "Footprint" "RGB:ws2812B_6028_FIX"
 			(at 265.43 133.35 0)
 			(effects
@@
 			)
 		)
-		(property "Footprint" "RGB:SK6812-MINI-E"
+		(property "Footprint" "RGB:ws2812B_6028_FIX"
 			(at 242.57 133.35 0)
 			(effects
@@
 			)
 		)
-		(property "Footprint" "RGB:SK6812-MINI-E"
+		(property "Footprint" "RGB:ws2812B_6028_FIX"
 			(at 222.25 120.65 0)
 			(effects
@@
 			)
 		)
-		(property "Footprint" "RGB:SK6812-MINI-E"
+		(property "Footprint" "RGB:ws2812B_6028_FIX"
 			(at 85.09 64.77 0)
 			(effects
@@
 			)
 		)
-		(property "Footprint" "RGB:SK6812-MINI-E"
+		(property "Footprint" "RGB:ws2812B_6028_FIX"
 			(at 379.73 133.35 0)
 			(effects
@@
 			)
 		)
-		(property "Footprint" "RGB:SK6812-MINI-E"
+		(property "Footprint" "RGB:ws2812B_6028_FIX"
 			(at 359.41 64.77 0)
 			(effects
@@
 			)
 		)
-		(property "Footprint" "RGB:SK6812-MINI-E"
+		(property "Footprint" "RGB:ws2812B_6028_FIX"
 			(at 379.73 77.47 0)
 			(effects
@@
 			)
 		)
-		(property "Footprint" "RGB:SK6812-MINI-E"
+		(property "Footprint" "RGB:ws2812B_6028_FIX"
 			(at 39.37 120.65 0)
 			(effects
@@
 			)
 		)
-		(property "Footprint" "RGB:SK6812-MINI-E"
+		(property "Footprint" "RGB:ws2812B_6028_FIX"
 			(at 153.67 120.65 0)
 			(effects
@@
 			)
 		)
-		(property "Footprint" "RGB:SK6812-MINI-E"
+		(property "Footprint" "RGB:ws2812B_6028_FIX"
 			(at 105.41 133.35 0)
 			(effects
@@
 			)
 		)
-		(property "Footprint" "RGB:SK6812-MINI-E"
+		(property "Footprint" "RGB:ws2812B_6028_FIX"
 			(at 85.09 120.65 0)
 			(effects
@@
 			)
 		)
-		(property "Footprint" "RGB:SK6812-MINI-E"
+		(property "Footprint" "RGB:ws2812B_6028_FIX"
 			(at 196.85 77.47 0)
 			(effects
@@
 			)
 		)
-		(property "Footprint" "RGB:SK6812-MINI-E"
+		(property "Footprint" "RGB:ws2812B_6028_FIX"
 			(at 82.55 77.47 0)
 			(effects
@@
 			)
 		)
-		(property "Footprint" "RGB:SK6812-MINI-E"
+		(property "Footprint" "RGB:ws2812B_6028_FIX"
 			(at 334.01 133.35 0)
 			(effects
@@
 			)
 		)
-		(property "Footprint" "RGB:SK6812-MINI-E"
+		(property "Footprint" "RGB:ws2812B_6028_FIX"
 			(at 336.55 64.77 0)
 			(effects
@@
 			)
 		)
-		(property "Footprint" "RGB:SK6812-MINI-E"
+		(property "Footprint" "RGB:ws2812B_6028_FIX"
 			(at 245.11 64.77 0)
 			(effects
@@
 			)
 		)
-		(property "Footprint" "RGB:SK6812-MINI-E"
+		(property "Footprint" "RGB:ws2812B_6028_FIX"
 			(at 39.37 64.77 0)
 			(effects
@@
 			)
 		)
-		(property "Footprint" "RGB:SK6812-MINI-E"
+		(property "Footprint" "RGB:ws2812B_6028_FIX"
 			(at 173.99 77.47 0)
 			(effects
@@
 			)
 		)
-		(property "Footprint" "RGB:SK6812-MINI-E"
+		(property "Footprint" "RGB:ws2812B_6028_FIX"
 			(at 336.55 120.65 0)
 			(effects
@@
 			)
 		)
-		(property "Footprint" "RGB:SK6812-MINI-E"
+		(property "Footprint" "RGB:ws2812B_6028_FIX"
 			(at 107.95 64.77 0)
 			(effects
@@
 			)
 		)
-		(property "Footprint" "RGB:SK6812-MINI-E"
+		(property "Footprint" "RGB:ws2812B_6028_FIX"
 			(at 219.71 133.35 0)
 			(effects
@@
 			)
 		)
-		(property "Footprint" "RGB:SK6812-MINI-E"
+		(property "Footprint" "RGB:ws2812B_6028_FIX"
 			(at 105.41 77.47 0)
 			(effects
@@
 			)
 		)
-		(property "Footprint" "RGB:SK6812-MINI-E"
+		(property "Footprint" "RGB:ws2812B_6028_FIX"
 			(at 176.53 120.65 0)
 			(effects
@@
 			)
 		)
-		(property "Footprint" "RGB:SK6812-MINI-E"
+		(property "Footprint" "RGB:ws2812B_6028_FIX"
 			(at 242.57 77.47 0)
 			(effects
@@
 			)
 		)
-		(property "Footprint" "RGB:SK6812-MINI-E"
+		(property "Footprint" "RGB:ws2812B_6028_FIX"
 			(at 267.97 64.77 0)
 			(effects
@@
 			)
 		)
-		(property "Footprint" "RGB:SK6812-MINI-E"
+		(property "Footprint" "RGB:ws2812B_6028_FIX"
 			(at 359.41 120.65 0)
 			(effects
@@
 			)
 		)
-		(property "Footprint" "RGB:SK6812-MINI-E"
+		(property "Footprint" "RGB:ws2812B_6028_FIX"
 			(at 311.15 77.47 0)
 			(effects
@@
 			)
 		)
-		(property "Footprint" "RGB:SK6812-MINI-E"
+		(property "Footprint" "RGB:ws2812B_6028_FIX"
 			(at 107.95 120.65 0)
 			(effects
@@
 			)
 		)
-		(property "Footprint" "RGB:SK6812-MINI-E"
+		(property "Footprint" "RGB:ws2812B_6028_FIX"
 			(at 313.69 120.65 0)
 			(effects
@@
 			)
 		)
-		(property "Footprint" "RGB:SK6812-MINI-E"
+		(property "Footprint" "RGB:ws2812B_6028_FIX"
 			(at 199.39 120.65 0)
 			(effects
@@
 			)
 		)
-		(property "Footprint" "RGB:SK6812-MINI-E"
+		(property "Footprint" "RGB:ws2812B_6028_FIX"
 			(at 130.81 64.77 0)
 			(effects
@@
 			)
 		)
-		(property "Footprint" "RGB:SK6812-MINI-E"
+		(property "Footprint" "RGB:ws2812B_6028_FIX"
 			(at 222.25 64.77 0)
 			(effects
@@
 			)
 		)
-		(property "Footprint" "RGB:SK6812-MINI-E"
+		(property "Footprint" "RGB:ws2812B_6028_FIX"
 			(at 36.83 77.47 0)
 			(effects
@@
 			)
 		)
-		(property "Footprint" "RGB:SK6812-MINI-E"
+		(property "Footprint" "RGB:ws2812B_6028_FIX"
 			(at 245.11 120.65 0)
 			(effects
@@
 			)
 		)
-		(property "Footprint" "RGB:SK6812-MINI-E"
+		(property "Footprint" "RGB:ws2812B_6028_FIX"
 			(at 382.27 120.65 0)
 			(effects
@@
 			)
 		)
-		(property "Footprint" "RGB:SK6812-MINI-E"
+		(property "Footprint" "RGB:ws2812B_6028_FIX"
 			(at 62.23 64.77 0)
 			(effects
@@
 			)
 		)
-		(property "Footprint" "RGB:SK6812-MINI-E"
+		(property "Footprint" "RGB:ws2812B_6028_FIX"
 			(at 382.27 64.77 0)
 			(effects
@@
 			)
 		)
-		(property "Footprint" "RGB:SK6812-MINI-E"
+		(property "Footprint" "RGB:ws2812B_6028_FIX"
 			(at 290.83 120.65 0)
 			(effects
@@
 			)
 		)
-		(property "Footprint" "RGB:SK6812-MINI-E"
+		(property "Footprint" "RGB:ws2812B_6028_FIX"
 			(at 173.99 133.35 0)
 			(effects
@@
 			)
 		)
-		(property "Footprint" "RGB:SK6812-MINI-E"
+		(property "Footprint" "RGB:ws2812B_6028_FIX"
 			(at 334.01 77.47 0)
 			(effects
