File: PCB_Rev3/ANSI/PH60_Rev3.kicad_pcb (KiCad board)
At the start: 2 copper layers, 285.8 x 95.2 mm, 216 parts, among them J1 USB_C_Receptacle_USB2.0_16P, J2 Conn_01x02, U1 XC6206PxxxMR, U2 W25Q16JVSS, U3 RP2040, Y1 Crystal_GND24

Commit message: Add wireless part
Parts:
- removed C10, C17, C18, C8: 1u, Capacitor_SMD:C_0402_1005Metric
- removed C11, C12, C13, C14, C15, C16, C5, C6, C7, C9: 100n, Capacitor_SMD:C_0402_1005Metric
- removed C2, C3: 20p, Capacitor_SMD:C_0402_1005Metric
- removed R1, R5: 1k, Resistor_SMD:R_0402_1005Metric
- removed R3, R4: 27.4, Resistor_SMD:R_0402_1005Metric
- removed U1: XC6206PxxxMR, Package_TO_SOT_SMD:SOT-23-3
- removed U2: W25Q16JVSS, Package_SON:Winbond_USON-8-1EP_3x2mm_P0.5mm_EP0.2x1.6mm
- removed U3: RP2040, Package_DFN_QFN:QFN-56-1EP_7x7mm_P0.4mm_EP3.2x3.2mm_ThermalVias
- removed Y1: Crystal_GND24, Crystal:Crystal_SMD_3225-4Pin_3.2x2.5mm
Routing:
- net VBUS: track 1508.8 -> 0.00 mm, vias 7 -> 0
- net row_0: track 541.9 -> 0.00 mm, vias 2 -> 0
- net row_1: track 512.3 -> 0.00 mm
- net row_2: track 484.6 -> 0.00 mm, vias 2 -> 0
- net row_3: track 347.7 -> 0.00 mm, vias 2 -> 0
- net Net-(RGB53-DOUT): track 307.8 -> 0.00 mm, vias 4 -> 0
- net col_12: track 302.2 -> 0.00 mm, vias 3 -> 0
- net Net-(RGB14-DOUT): track 294.5 -> 0.00 mm, vias 2 -> 0
- net Net-(RGB28-DOUT): track 292.9 -> 0.00 mm, vias 2 -> 0
- net Net-(RGB41-DOUT): track 285.9 -> 0.00 mm, vias 4 -> 0
- net row_4: track 262.9 -> 0.00 mm, vias 4 -> 0
- net col_13: track 249.8 -> 0.00 mm, vias 3 -> 0
- net col_11: track 238.7 -> 0.00 mm, vias 3 -> 0
- net col_0: track 226.0 -> 0.00 mm, vias 2 -> 0
- net DIN: track 197.0 -> 0.00 mm, vias 4 -> 0
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
Commit message: Finish board design
Parts:
- added AE1: Antenna_Shield, PH60:ANT-2.4G-1.6MM-MINI, B.Cu at (336.5, 92.5)
- added BT1: Battery, Connector_Molex:Molex_PicoBlade_53261-0271_1x02-1MP_P1.25mm_Horizontal, B.Cu at (123.7, 33.0)
- added C1: 100n, Capacitor_SMD:C_0402_1005Metric, B.Cu at (192.5, 151.6)
- added C10: 1u, Capacitor_SMD:C_0402_1005Metric, B.Cu at (190.6, 138.7)
- added C11: 1u, Capacitor_SMD:C_0402_1005Metric, B.Cu at (189.6, 138.7)
- added C12: 20p, Capacitor_SMD:C_0402_1005Metric, B.Cu at (200.4, 153.5)
- added C13: 20p, Capacitor_SMD:C_0402_1005Metric, B.Cu at (197.8, 151.1)
- added C14: 4.7u, Capacitor_SMD:C_0402_1005Metric, B.Cu at (132.3, 146.2)
- added C15: 10u, Capacitor_SMD:C_0402_1005Metric, B.Cu at (119.8, 147.1)
- added C16: 100n, Capacitor_SMD:C_0402_1005Metric, B.Cu at (200.6, 136.5)
- added C17: 10u, Capacitor_SMD:C_0402_1005Metric, B.Cu at (149.8, 151.4)
- added C18: 22u, Capacitor_SMD:C_0402_1005Metric, B.Cu at (153.5, 151.6)
- added C19: 1u, Capacitor_SMD:C_0402_1005Metric, B.Cu at (333.4, 97.9)
- added C2: 100n, Capacitor_SMD:C_0402_1005Metric, B.Cu at (196.5, 137.4)
- added C20: 0.1u, Capacitor_SMD:C_0402_1005Metric, B.Cu at (326.0, 96.0)
- added C21: 2u2, Capacitor_SMD:C_0402_1005Metric, B.Cu at (326.0, 93.9)
- added C22: 2u2, Capacitor_SMD:C_0402_1005Metric, B.Cu at (329.2, 101.0)
- added C23: 2u2, Capacitor_SMD:C_0402_1005Metric, B.Cu at (333.2, 102.7)
- added C3: 100n, Capacitor_SMD:C_0402_1005Metric, B.Cu at (191.5, 138.7)
- added C4: 100n, Capacitor_SMD:C_0402_1005Metric, B.Cu at (200.7, 141.3)
- added C5: 100n, Capacitor_SMD:C_0402_1005Metric, B.Cu at (193.5, 151.6)
- added C6: 100n, Capacitor_SMD:C_0402_1005Metric, B.Cu at (200.7, 146.1)
- added C7: 100n, Capacitor_SMD:C_0402_1005Metric, B.Cu at (187.6, 146.1)
- added C8: 100n, Capacitor_SMD:C_0402_1005Metric, B.Cu at (194.5, 137.4)
- added C9: 100n, Capacitor_SMD:C_0402_1005Metric, B.Cu at (195.5, 137.4)
- added D1: PRTR5V0U2X, Package_TO_SOT_SMD:SOT-143, B.Cu at (47.4, 47.9)
- added F1: 1000ma, Fuse:Fuse_0805_2012Metric, B.Cu at (50.7, 46.5)
- added J4: Conn_01x02_Pin, Connector_PinHeader_1.27mm:PinHeader_1x02_P1.27mm_Vertical, F.Cu at (124.3, 33.0)
- added J5: Conn_01x04_Pin, Connector_PinHeader_2.00mm:PinHeader_1x04_P2.00mm_Vertical, B.Cu at (329.2, 84.1)
- added J6: Conn_01x02, Connector_PinHeader_2.54mm:PinHeader_1x02_P2.54mm_Vertical, B.Cu at (340.5, 105.9)
- added J7: Conn_01x02, Connector_PinHeader_2.54mm:PinHeader_1x02_P2.54mm_Vertical, B.Cu at (332.0, 108.6)
- added L1: 2.2uH, Inductor_SMD:L_Changjiang_FNR252012S, B.Cu at (126.2, 141.7)
- added L2: 2.2uH, Inductor_SMD:L_Changjiang_FNR252012S, B.Cu at (146.0, 147.3)
- added L3: 22uH, Inductor_SMD:L_Changjiang_FNR252012S, B.Cu at (325.1, 100.5)
- added R10: 33k, PCM_Resistor_SMD_AKL:R_0402_1005Metric, B.Cu at (151.2, 143.6)
- added R11: 10k, PCM_Resistor_SMD_AKL:R_0402_1005Metric, B.Cu at (154.4, 145.1)
- added R12: 100k, PCM_Resistor_SMD_AKL:R_0402_1005Metric, B.Cu at (148.9, 143.4)
- added R3: 1R, PCM_Resistor_SMD_AKL:R_0402_1005Metric, B.Cu at (193.6, 138.7)
- added R4: 1R, PCM_Resistor_SMD_AKL:R_0402_1005Metric, B.Cu at (192.5, 138.7)
- added R5: 1k, PCM_Resistor_SMD_AKL:R_0402_1005Metric, B.Cu at (194.9, 153.5)
- added R6: 442k, PCM_Resistor_SMD_AKL:R_0402_1005Metric, B.Cu at (123.1, 145.7)
- added R7: 100k, PCM_Resistor_SMD_AKL:R_0402_1005Metric, B.Cu at (122.9, 148.6)
- added R8: 1k, PCM_Resistor_SMD_AKL:R_0402_1005Metric, B.Cu at (199.4, 133.9)
- added R9: 1k, PCM_Resistor_SMD_AKL:R_0402_1005Metric, B.Cu at (154.9, 148.8)
- added SW1: SW_SPDT_321, PCM_marbastlib-various:SW_MSK12C02-HB, B.Cu at (30.7, 33.4)
- added U1: TLV62569DBV, Package_TO_SOT_SMD:SOT-23-5, B.Cu at (128.1, 146.8)
- added U2: RP2040, Package_DFN_QFN:QFN-56-1EP_7x7mm_P0.4mm_EP3.2x3.2mm_ThermalVias, B.Cu at (194.3, 145.1)
- added U3: W25Q16JVSS, Package_SON:Winbond_USON-8-1EP_3x2mm_P0.5mm_EP0.2x1.6mm, B.Cu at (198.9, 137.7)
- added U4: ETA6093, Package_TO_SOT_SMD:SOT-23-5, B.Cu at (150.0, 147.2)
- added U5: CH582F, PH60:QFN28_4X4_FIX, B.Cu at (329.8, 95.1)
- added Y1: Crystal_GND24, Crystal:Crystal_SMD_3225-4Pin_3.2x2.5mm, B.Cu at (197.7, 153.5)
- added Y2: X322532MOB4SI, Crystal:Crystal_SMD_3225-4Pin_3.2x2.5mm, B.Cu at (334.0, 91.3)
- added Y3: XKXGI-SUA-32.768K, Crystal:Crystal_SMD_3215-2Pin_3.2x1.5mm, B.Cu at (322.6, 96.3)
- R1: renamed from R6; footprint Resistor_SMD:R_0402_1005Metric -> PCM_Resistor_SMD_AKL:R_0402_1005Metric
- R2: renamed from R7; footprint Resistor_SMD:R_0402_1005Metric -> PCM_Resistor_SMD_AKL:R_0402_1005Metric
- RGB1, RGB10, RGB11, RGB12, RGB13, RGB14, RGB15, RGB16, RGB17, RGB18, RGB19, RGB2, RGB20, RGB21, RGB22, RGB23, RGB24, RGB25, RGB26, RGB27, RGB28, RGB29, RGB3, RGB30, RGB31, RGB32, RGB33, RGB34, RGB35, RGB36, RGB37, RGB38, RGB39, RGB4, RGB40, RGB41, RGB42, RGB43, RGB44, RGB45, RGB46, RGB47, RGB48, RGB49, RGB5, RGB50, RGB51, RGB52, RGB53, RGB54, RGB55, RGB56, RGB57, RGB58, RGB59, RGB6, RGB60, RGB61, RGB7, RGB8, RGB9: footprint PH60:WS2812B_Reverse -> PH60:ws2812b_6028
- moved J2 88.9 mm to (198.8, 128.5)
- moved R2 0.18 mm to (49.2, 40.1)
- moved R1 0.11 mm to (47.1, 40.1)
- renumbered D9 to D10, D10 to D11, D11 to D12, D12 to D13, D13 to D14, D14 to D15, D15 to D16, D16 to D17, D17 to D18, D18 to D19, D1 to D2, D19 to D20, D20 to D21, D21 to D22, D22 to D23, D23 to D24, D24 to D25, D25 to D26, D26 to D27, D27 to D28, D28 to D29, D2 to D3, D29 to D30, D30 to D31, D31 to D32, D32 to D33, D33 to D34, D34 to D35, D35 to D36, D36 to D37, D37 to D38, D38 to D39, D3 to D4, D39 to D40, D40 to D41, D41 to D42, D42 to D43, D43 to D44, D44 to D45, D45 to D46, D46 to D47, D47 to D48, D48 to D49, D4 to D5, D49 to D50, D50 to D51, D51 to D52, D52 to D53, D53 to D54, D54 to D55, D55 to D56, D56 to D57, D57 to D58, D58 to D59, D5 to D6, D59 to D60, D60 to D61, D61 to D62, D6 to D7, D7 to D8, D8 to D9
Connections:
- J1 pad A4: VBUS -> VBUS_UP
- J1 pad A9: VBUS -> VBUS_UP
- J1 pad B4: VBUS -> VBUS_UP
- J1 pad B9: VBUS -> VBUS_UP
- J2 pad 1: /~{USB_BOOT} -> Net-(J2-Pin_1)
Other:
- board text removed: "PH60-REV3-ANSI-RPI_Ver"
- board text removed: "PROTOTYPE_01"
- board text removed: "Team PHDesign"

Commit message: Add files via upload
Parts:
- moved AE1 193.7 mm to (144.9, 120.8), turned to 0 degrees
- moved C23 191.2 mm to (142.6, 118.1), turned to 0 degrees
- moved C21 191.2 mm to (135.6, 110.6), turned to 180 degrees
- moved C20 191.1 mm to (135.6, 111.6), turned to 0 degrees
- moved C19 191.1 mm to (143.1, 114.1)
- moved U5 190.4 mm to (140.1, 111.1)
- moved C22 189.4 mm to (140.6, 118.1), turned to 180 degrees
- moved Y2 188.5 mm to (146.6, 111.1), turned to 180 degrees
- moved Y3 187.9 mm to (135.6, 114.6), turned to 180 degrees
- moved L3 185.7 mm to (140.1, 116.1), turned to 180 degrees
- moved J5 179.9 mm to (169.6, 167.1)
- moved J6 179.9 mm to (180.9, 188.9)
- moved J7 179.9 mm to (172.3, 191.5)
- moved C18 107.7 mm to (125.6, 47.6), turned to -90 degrees
- moved C17 106.5 mm to (115.6, 50.6), turned to 0 degrees
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
Commit message: Regroup
Parts:
- removed J6: Conn_01x02, Connector_PinHeader_2.54mm:PinHeader_1x02_P2.54mm_Vertical
- removed U3: W25Q16JVSS, Package_SON:Winbond_USON-8-1EP_3x2mm_P0.5mm_EP0.2x1.6mm
- added U6: W25Q16JVSS, Package_SON:Winbond_USON-8-1EP_3x2mm_P0.5mm_EP0.2x1.6mm, B.Cu at (115.9, 111.2)
- J2: moved to F.Cu
- J7: value Conn_01x02 -> Conn_01x03_Pin; footprint Connector_PinHeader_2.54mm:PinHeader_1x02_P2.54mm_Vertical -> Connector_PinSocket_1.27mm:PinSocket_1x03_P1.27mm_Vertical; moved to F.Cu
- moved J2 104.8 mm to (116.4, 106.9)
- moved J7 89.3 mm to (193.4, 104.7), turned to -90 degrees
- moved R10 87.1 mm to (56.0, 81.5)
- moved R12 87.1 mm to (58.5, 81.5)
- moved J5 61.6 mm to (185.0, 107.5)
- moved AE1 52.0 mm to (196.4, 113.4), turned to 90 degrees
- moved C19 48.3 mm to (191.3, 111.7), turned to 180 degrees
- moved C22 48.1 mm to (188.5, 114.7), turned to -90 degrees
- moved Y3 47.9 mm to (183.5, 115.2), turned to 135 degrees
- moved U5 46.6 mm to (186.7, 111.2)
- moved Y2 46.1 mm to (192.6, 108.3)
- moved C21 45.6 mm to (181.1, 109.6)
- moved C20 43.2 mm to (178.8, 111.9)
- moved L3 41.2 mm to (181.1, 111.7), turned to 90 degrees
- moved C23 36.9 mm to (178.8, 110.9), turned to 180 degrees
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Connections:
- D1 pad 2: /USB_D+ -> USB_D+
- D1 pad 3: /USB_D- -> USB_D-
- J1 pad A6: /USB_D+ -> USB_D+
- J1 pad A7: /USB_D- -> USB_D-
- J1 pad B6: /USB_D+ -> USB_D+
- J1 pad B7: /USB_D- -> USB_D-
- J2 pad 1: Net-(J2-Pin_1) -> RPI_BOOTSEL
- J5 pad 3: /wireless/RX1 -> /wireless/TX1
- J5 pad 4: /wireless/TX1 -> /wireless/RX1
- J7 pad 1: GND -> BOOT
- J7 pad 2: RST -> GND
- R8 pad 1: Net-(J2-Pin_1) -> RPI_BOOTSEL
- R8 pad 2: /QSPI_SS -> RPI_BOOTSEL
- U2 pad 26: unconnected-(U2-RUN-Pad26) -> RPI_RUN
- U2 pad 56: /QSPI_SS -> RPI_BOOTSEL
- U5 pad 12: WCH_D+ -> USB_D+
- U5 pad 13: WCH_D- -> USB_D-
- U5 pad 27: unconnected-(U5-PA13/SCK0/PWM5/AIN3-Pad27) -> RPI_RUN
- U5 pad 28: unconnected-(U5-PA12/SCS/PWM4/AIN2-Pad28) -> RPI_BOOTSEL
Routing:
- net +3V3: track 0.00 -> 59.9 mm, vias 0 -> 3
- net GND: track 0.00 -> 42.6 mm, vias 0 -> 9
- net VDCIA: track 0.00 -> 28.0 mm
- net +1V1: track 0.00 -> 22.9 mm
- net RPI_BOOTSEL: track 0.00 -> 13.6 mm, vias 0 -> 1
- net BOOT: track 0.00 -> 9.75 mm
- net /QSPI_SD1: track 0.00 -> 8.46 mm
- net /QSPI_SD2: track 0.00 -> 7.67 mm
- net RST: track 0.00 -> 7.44 mm
- net /wireless/RX1: track 0.00 -> 6.87 mm
- net X32MI: track 0.00 -> 6.00 mm
- net /XIN: track 0.00 -> 5.99 mm
- net X32MO: track 0.00 -> 5.52 mm
- net Net-(U1-FB): track 0.00 -> 5.23 mm
- net VBUS: track 0.00 -> 5.11 mm
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