File: PCB_Rev3/ANSI/PH60_Rev3.kicad_pcb (KiCad board)
At the start: 2 copper layers, 285 x 94.6 mm, 251 parts, among them J1 USB_C_Receptacle_USB2.0_16P, J2 Conn_01x02, J3 Conn_01x02_Pin, J4 Conn_01x02_Pin, J5 Conn_01x04_Pin, J6 Conn_01x02_Pin, J7 Conn_01x03_Pin, SW1 SW_SPDT_321, U1 TLV62569DBV, U2 RP2040, U4 ETA6093, U5 CH582F, U6 W25Q16JVSS, Y1 Crystal_GND24, Y2 X322532MOB4SI, Y3 XKXGI-SUA-32.768K

Commit message: Antenna update
Parts:
- added AE1: Antenna_Shield, PH60:ANT-2.4G-1.6MM-MINI-Reversed, B.Cu at (121.5, 120.2)
- added J8: Conn_01x02_Pin, Connector_PinHeader_2.00mm:PinHeader_1x02_P2.00mm_Vertical, F.Cu at (128.3, 121.1)
Connections:
- U2 pad 40: unconnected-(U2-GPIO28_ADC2-Pad40) -> /RPI_TX
- U2 pad 41: unconnected-(U2-GPIO29_ADC3-Pad41) -> /RPI_RX
Routing:
- net /RPI_TX: track 0.00 -> 11.1 mm
- net Net-(AE1-A): track 0.00 -> 7.06 mm
- net /RPI_RX: track 0.00 -> 6.50 mm
- net DIN: track 170.3 -> 173.7 mm
- net row_1: track 350.2 -> 352.8 mm
- net row_3: track 298.1 -> 297.1 mm
- net row_2: track 321.1 -> 320.2 mm
- net RPI_RUN: track 43.0 -> 43.8 mm
- net row_4: track 519.1 -> 518.3 mm
- net row_0: track 378.7 -> 379.5 mm
- net GND: vias 400 -> 446
Other:
- outline, holes or cut-outs redrawn

Commit message: Add files via upload
Parts:
- moved SW1 2.31 mm to (33.0, 71.6)
Routing:
- net +BATT: track 257.0 -> 258.4 mm, vias 2 -> 5
- net VBUS: vias 22 -> 19
- net GND: vias 446 -> 453
