File: PCB_Rev3/ANSI/PH60_Rev3.kicad_pcb (KiCad board)
At the start: 2 copper layers, 285 x 94.6 mm, 258 parts, among them J1 USB_C_Receptacle_USB2.0_16P, J2 Conn_01x02, J3 Conn_01x02_Pin, J4 Conn_01x02_Pin, J5 Conn_01x04_Pin, J6 Conn_01x02_Pin, J7 Conn_01x03_Pin, J8 Conn_01x02_Pin, SW1 SW_SPDT_321, U1 TLV62569DBV, U2 RP2040, U4 ETA6093, U5 CH582F, U6 W25Q16JVSS, Y1 Crystal_GND24, Y2 X322532MOB4SI, Y3 XKXGI-SUA-32.768K

Commit message: 四次drc
gnd过孔精简，3v3添加0F调试电容
Parts:
- added C29: 0u, Capacitor_SMD:C_0402_1005Metric, B.Cu at (123.8, 110.2)
Routing:
- net RPI_BOOTSEL: track 29.8 -> 30.7 mm
- net /RGB/rgb3: track 26.6 -> 27.4 mm
- net VBUS_SW: track 1324.2 -> 1324.8 mm
- net row_1: track 349.9 -> 350.5 mm, vias 4 -> 2
- net Net-(RGB15-DOUT): track 19.2 -> 19.7 mm
- net GND: vias 416 -> 374

Commit message: Routing update
Parts:
- removed J7: Conn_01x03_Pin, Connector_PinSocket_1.27mm:PinSocket_1x03_P1.27mm_Vertical
- added J9: Conn_01x02_Pin, Connector_PinHeader_2.00mm:PinHeader_1x02_P2.00mm_Vertical, F.Cu at (114.8, 106.4)
- J4: footprint Connector_PinHeader_2.00mm:PinHeader_1x02_P2.00mm_Vertical -> Connector_PinHeader_1.27mm:PinHeader_1x02_P1.27mm_Vertical
- moved C16 1.62 mm to (126.0, 112.8), turned to 180 degrees
- moved R7 1.19 mm to (118.8, 109.5)
- moved R6 1.11 mm to (120.0, 109.5)
- moved Y2 0.62 mm to (113.3, 110.0)
- moved C15 0.59 mm to (123.7, 108.6)
- moved C29 0.25 mm to (123.7, 110.5)
Connections:
- U5 pad 16: RST -> unconnected-(U5-PB23/RST/TMR0_/TXD2_/PWM11-Pad16)
Routing:
- net RST: track 8.52 -> 0.00 mm, vias 1 -> 0
- net +3V3: track 100.5 -> 93.0 mm, vias 7 -> 9
- net GND: track 71.2 -> 75.3 mm, vias 374 -> 376
- net RPI_BOOTSEL: track 30.7 -> 31.4 mm
- net col_4: track 92.7 -> 93.3 mm
- added copper zone on B.Cu, net +3V3
Other:
- outline, holes or cut-outs redrawn
