File: PCB_Rev3/ANSI/RGB.kicad_sch (KiCad schematic)
At the start: 64 parts

Commit message: REV3 与 REV3_A 合并
Parts:
- renumbered C24 to C22, C25 to C23, C26 to C24
Changed lines of the file:
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@@
 		(dnp no)
 		(fields_autoplaced yes)
-		(property "Reference" "C26"
+		(property "Reference" "C24"
 			(at 237.49 116.8399 0)
 			(effects
@@
 			(project "PH60_Rev3"
 				(path "/dca0f898-8fdb-4522-a51d-f4f4238906e7/c0337f82-e68f-485d-b406-18ae8e593971"
-					(reference "C26")
+					(reference "C24")
 					(unit 1)
 				)
@@
 		(dnp no)
 		(fields_autoplaced yes)
-		(property "Reference" "C25"
+		(property "Reference" "C23"
 			(at 223.52 116.8399 0)
 			(effects
@@
 			(project "PH60_Rev3"
 				(path "/dca0f898-8fdb-4522-a51d-f4f4238906e7/c0337f82-e68f-485d-b406-18ae8e593971"
-					(reference "C25")
+					(reference "C23")
 					(unit 1)
 				)
@@
 		(dnp no)
 		(fields_autoplaced yes)
-		(property "Reference" "C24"
+		(property "Reference" "C22"
 			(at 208.28 116.8399 0)
 			(effects
@@
 			(project ""
 				(path "/dca0f898-8fdb-4522-a51d-f4f4238906e7/c0337f82-e68f-485d-b406-18ae8e593971"
-					(reference "C24")
-					(unit 1)
-				)
+					(reference "C22")
+					(unit 1)
+				)
