File: PCB_Rev3/ANSI/wireless.kicad_sch (KiCad schematic)
At the start: 37 parts, among them J11 Conn_01x02_Pin, J3 Conn_01x02_Pin, J4 Conn_01x02_Pin, J5 Conn_01x02_Pin, J6 Conn_01x04_Pin, J7 USB_HS, J9 Conn_01x04_Pin, SW2 SW_SPDT_321, U4 CH582F, U5 TLV62569DBV, U6 ETA6093, Y2 X322532MOB4SI, Y3 XKXGI-SUA-32.768K

Commit message: Finish board design
Parts:
- removed BT1: Battery, Connector_Molex:Molex_PicoBlade_53261-0271_1x02-1MP_P1.25mm_Horizontal, symbol Device:Battery
- removed C22: 4.7u, Capacitor_SMD:C_0402_1005Metric, symbol Device:C
- removed C23, C24: 10u, Capacitor_SMD:C_0402_1005Metric, symbol Device:C
- removed C25: 22u, Capacitor_SMD:C_0402_1005Metric, symbol Device:C
- removed D62: LED, PCM_Diode_SMD_AKL:D_0402_1005Metric, symbol Device:LED
- removed J11: Conn_01x02_Pin, Connector_PinHeader_1.27mm:PinHeader_1x02_P1.27mm_Vertical, symbol Connector:Conn_01x02_Pin
- removed J3, J4, J5: Conn_01x02_Pin, part:TS-1088-AR02016, symbol Connector:Conn_01x02_Pin
- removed J7: USB_HS, part:USB-C_16P_HandSolder, symbol Connector:USB_C_Receptacle_USB2.0_14P
- removed J9: Conn_01x04_Pin, Connector_PinHeader_2.00mm:PinHeader_1x04_P2.00mm_Vertical, symbol Connector:Conn_01x04_Pin
- removed L1, L3: 2.2uH, Inductor_SMD:L_Changjiang_FNR252012S, symbol Device:L
- removed R10: 442k, PCM_Resistor_SMD_AKL:R_0402_1005Metric, symbol Device:R
- removed R11, R13: 100k, PCM_Resistor_SMD_AKL:R_0402_1005Metric, symbol Device:R
- removed R12: 33k, PCM_Resistor_SMD_AKL:R_0402_1005Metric, symbol Device:R
- removed R14: 1k, PCM_Resistor_SMD_AKL:R_0402_1005Metric, symbol Device:R
- removed R15: 10k, PCM_Resistor_SMD_AKL:R_0402_1005Metric, symbol Device:R
- removed R2: 1K, PCM_Resistor_SMD_AKL:R_0402_1005Metric, symbol Device:R
- removed R8, R9: 5.1k, PCM_Resistor_SMD_AKL:R_0402_1005Metric, symbol Device:R
- removed SW2: SW_SPDT_321, PCM_marbastlib-various:SW_MSK12C02-HB, symbol Switch:SW_SPDT_321
- removed U4: CH582F, QFN28_4X4, symbol CHXXX:CH582F
- removed U5: TLV62569DBV, Package_TO_SOT_SMD:SOT-23-5, symbol Regulator_Switching:TLV62569DBV
- removed U6: ETA6093, Package_TO_SOT_SMD:SOT-23-5, symbol eta6093:ETA6093
- added J6, J7: Conn_01x02, Connector_PinHeader_2.54mm:PinHeader_1x02_P2.54mm_Vertical, symbol Connector_Generic:Conn_01x02
- added U5: CH582F, CHXXX:QFN28_4X4, symbol WCH:CH582F
- AE1: footprint part:ANT-2.4G-1.6MM-MINI -> PH60:ANT-2.4G-1.6MM-MINI
- renumbered C1 to C19, C4 to C20, C19 to C22, C20 to C23, J6 to J5, L2 to L3
Connections:
- net VBUS is gone; now on net SWDIO: J5.1 (Pin_1)
- net +3V3: now also U5.5 (VIO33/VDD33)
- net BOOT: now also J6.2 (Pin_2), U5.17 (PB22/TMR3/RXD2_)
- net CHRG: now also U5.24 (PA5/TXD3/AIN1)
- net GND: now also J6.1 (Pin_1), J7.1 (Pin_1), U5.0 (GND); no longer J5.2 (Pin_2)
- net RST: now also J7.2 (Pin_2), U5.16 (PB23/RST/TMR0_/TXD2_/PWM11)
- net RX1: now also U5.6 (PA8/RXD1/AIN12)
- net SWDIO: now also U5.9 (PB14/TIO/DSR_/MOSI_/PWM10)
- net SWTCK: now also J5.2 (Pin_2), U5.8 (PB15/TCK/MISO_/DTR_)
- net TX1: now also U5.7 (PA9/TMR0/TXD1/AIN13)
- net VDCIA: now also U5.22 (VDCIA), U5.3 (VDCID)
- net VSW: now also U5.4 (VSW)
- net WCH_D+: now also U5.12 (PB11/UD+/TMR2_)
- net WCH_D-: now also U5.13 (PB10/UD-/TMR1_)
- net X32KI: now also U5.2 (PA10/X32KI/TMR1)
- net X32KO: now also U5.1 (PA11/X32KO/TMR2)
- net X32MI: now also U5.19 (X32MI)
- net X32MO: now also U5.18 (X32MO)
- net batt_level: now also U5.23 (PA4/RXD3/AIN0)
- net at C19.2: now also U5.20 (VINTA)
- net at AE1.1 (A): now also U5.21 (ANT)
- new net RPI_D+: U5.10 (PB13/U2D+/SCK0_/SCL/TXD1_)
- new net RPI_D-: U5.11 (PB12/U2D-/SCS_/SDA/RXD1_)
- no-connect marks 7 -> 6
Other:
- note added: "UART&SWD"
- note added: "ch582F"
- note removed: "Batt status"
- note removed: "Charge & Boost"
- note removed: "LED"
- note removed: "SWD"
- note removed: "UART"
- note removed: "USB_OUT"
- note removed: "main"
- note removed: "power"
- moved on the sheet: AE1, C19, C20, C21, C22, C23, J5, L3, Y2, Y3

Commit message: Regroup
Parts:
- removed J6, J7: Conn_01x02, Connector_PinHeader_2.54mm:PinHeader_1x02_P2.54mm_Vertical, symbol Connector_Generic:Conn_01x02
- added J7: Conn_01x03_Pin, Connector_PinSocket_1.27mm:PinSocket_1x03_P1.27mm_Vertical, symbol Connector:Conn_01x03_Pin
- U5: footprint CHXXX:QFN28_4X4 -> PH60:QFN28_4X4_FIX
Connections:
- net BOOT: now also J7.1 (Pin_1)
- net GND: now also J7.2 (Pin_2)
- net RST: now also J7.3 (Pin_3)
- net RX1: now also J5.4 (Pin_4); no longer J5.3 (Pin_3)
- net TX1: now also J5.3 (Pin_3); no longer J5.4 (Pin_4)
- net RPI_RUN: now reaches U5.27 (PA13/SCK0/PWM5/AIN3)
- net RPI_BOOTSEL: now reaches U5.28 (PA12/SCS/PWM4/AIN2)
- net WCH_D+ renamed USB_D+
- net WCH_D- renamed USB_D-
- no-connect marks 6 -> 4
Other:
- moved on the sheet: C21

Commit message: Antenna update
Parts:
- AE1: footprint PH60:ANT-2.4G-1.6MM-MINI -> PH60:ANT-2.4G-1.6MM-MINI-Reversed
Other:
- moved on the sheet: AE1
Changed lines of the file:
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@@
+	(wire
+		(pts
+			(xy 143.51 24.13) (xy 143.51 25.4)
+		)
+		(stroke
+			(width 0)
+			(type default)
+		)
+	)
 	(wire
 		(pts
@@
 	(wire
 		(pts
-			(xy 140.97 25.4) (xy 140.97 39.37)
+			(xy 140.97 24.13) (xy 140.97 39.37)
 		)
 		(stroke
@@
 	(symbol
 		(lib_id "Device:Antenna_Shield")
-		(at 140.97 20.32 0)
+		(at 140.97 19.05 0)
 		(unit 1)
 		(exclude_from_sim no)
@@
 		(dnp no)
 		(property "Reference" "AE1"
-			(at 144.78 18.4149 0)
+			(at 144.78 17.1449 0)
 			(effects
 				(font
@@
 		)
 		(property "Value" "Antenna_Shield"
-			(at 144.78 20.9549 0)
+			(at 144.78 19.6849 0)
 			(effects
 				(font
@@
 			)
 		)
-		(property "Footprint" "PH60:ANT-2.4G-1.6MM-MINI"
-			(at 140.97 17.78 0)
+		(property "Footprint" "PH60:ANT-2.4G-1.6MM-MINI-Reversed"
+			(at 140.97 16.51 0)
 			(effects
 				(font
@@
 		)
 		(property "Datasheet" "~"
-			(at 140.97 17.78 0)
+			(at 140.97 16.51 0)
 			(effects
 				(font
@@
 		)
 		(property "Description" "Antenna with extra pin for shielding"
-			(at 140.97 20.32 0)
-			(effects
-				(font
+			(at 140.97 19.05 0)
+			(effects
+				(font

Commit message: Routing update
Parts:
- removed J7: Conn_01x03_Pin, Connector_PinSocket_1.27mm:PinSocket_1x03_P1.27mm_Vertical, symbol Connector:Conn_01x03_Pin
- added J9: Conn_01x02_Pin, Connector_PinHeader_2.00mm:PinHeader_1x02_P2.00mm_Vertical, symbol Connector:Conn_01x02_Pin
Connections:
- net BOOT: now also J9.1 (Pin_1)
- net GND: now also J9.2 (Pin_2)
- net RST: no longer names the net of U5.16 (PB23/RST/TMR0_/TXD2_/PWM11)
- no-connect marks 4 -> 5

Commit message: REV3 与 REV3_A 合并
Parts:
- renumbered C19 to C25, C20 to C26, C21 to C27, C22 to C28, C23 to C29, J9 to J7, J5 to J8
Changed lines of the file:
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@@
 		(on_board yes)
 		(dnp no)
-		(property "Reference" "C22"
+		(property "Reference" "C28"
 			(at 76.2 140.9699 0)
 			(effects
@@
 			(project "PH60_Rev3"
 				(path "/dca0f898-8fdb-4522-a51d-f4f4238906e7/cfb76ba3-57e3-4364-b5e7-d3e68b86cce5"
-					(reference "C22")
+					(reference "C28")
 					(unit 1)
 				)
@@
 		(dnp no)
 		(fields_autoplaced yes)
-		(property "Reference" "J9"
+		(property "Reference" "J7"
 			(at 35.56 27.3049 90)
 			(effects
@@
 			(project ""
 				(path "/dca0f898-8fdb-4522-a51d-f4f4238906e7/cfb76ba3-57e3-4364-b5e7-d3e68b86cce5"
-					(reference "J9")
+					(reference "J7")
 					(unit 1)
 				)
@@
 		(dnp no)
 		(fields_autoplaced yes)
-		(property "Reference" "C20"
+		(property "Reference" "C26"
 			(at 96.52 62.23 90)
 			(effects
@@
 			(project "PH60_Rev3"
 				(path "/dca0f898-8fdb-4522-a51d-f4f4238906e7/cfb76ba3-57e3-4364-b5e7-d3e68b86cce5"
-					(reference "C20")
+					(reference "C26")
 					(unit 1)
 				)
@@
 		(on_board yes)
 		(dnp no)
-		(property "Reference" "C19"
+		(property "Reference" "C25"
 			(at 147.32 26.67 0)
 			(effects
@@
 			(project "PH60_Rev3"
 				(path "/dca0f898-8fdb-4522-a51d-f4f4238906e7/cfb76ba3-57e3-4364-b5e7-d3e68b86cce5"
-					(reference "C19")
+					(reference "C25")
 					(unit 1)
 				)
@@
 		(dnp no)
 		(fields_autoplaced yes)
-		(property "Reference" "C23"
+		(property "Reference" "C29"
 			(at 97.79 140.9699 0)
 			(effects
@@
 			(project "PH60_Rev3"
 				(path "/dca0f898-8fdb-4522-a51d-f4f4238906e7/cfb76ba3-57e3-4364-b5e7-d3e68b86cce5"
-					(reference "C23")
+					(reference "C29")
 					(unit 1)
 				)
@@
 		(dnp no)
 		(fields_autoplaced yes)
-		(property "Reference" "J5"
+		(property "Reference" "J8"
 			(at 85.725 101.6 0)
 			(effects
@@
 			(project "PH60_Rev3"
 				(path "/dca0f898-8fdb-4522-a51d-f4f4238906e7/cfb76ba3-57e3-4364-b5e7-d3e68b86cce5"
-					(reference "J5")
+					(reference "J8")
 					(unit 1)
 				)
@@
 		(dnp no)
 		(fields_autoplaced yes)
-		(property "Reference" "C21"
+		(property "Reference" "C27"
 			(at 160.02 116.84 90)
 			(effects
@@
 			(project "PH60_Rev3"
 				(path "/dca0f898-8fdb-4522-a51d-f4f4238906e7/cfb76ba3-57e3-4364-b5e7-d3e68b86cce5"
-					(reference "C21")
+					(reference "C27")
 					(unit 1)
 				)
